File: src/hardware/camera.kicad_sch (KiCad schematic)
At the start: 0 parts

Commit message: Removed Camera because currently not viable
Parts:
- added C102, C103, C104: 100nF, symbol Device:C
- added R52: 10kΩ, Resistor_SMD:R_0603_1608Metric, symbol Device:R
- added U36: HM01B0-MWA, Project:BGA16N50X40P4X4_227X213X81, symbol HM01B0-MWA:HM01B0-MWA
- added U38: TXS0108ERKSR, Project:VQFN20_RKS_TEX, symbol TXS0108ERKSR:TXS0108ERKSR
Connections:
- new net: R52.1, U38.10 (OE)
- new net: C102.2, U36.D3 (DVDD)
- new net +1V8: C103.2, U36.D4 (IOVDD), U38.2 (VCCA)
- new net +3V0: C104.2, U36.D1 (AVDD)
- new net +3V3: U38.19 (VCCB)
- new net CAM1D0: U38.20 (B1)
- new net CAM1D01V8: U36.B4 (D0/SDO), U38.1 (A1)
- new net CAM1D1: U38.18 (B2)
- new net CAM1D11V8: U36.B3 (D1), U38.3 (A2)
- new net CAM1D2: U38.17 (B3)
- new net CAM1D21V8: U36.A4 (D2), U38.4 (A3)
- new net CAM1D3: U38.16 (B4)
- new net CAM1D31V8: U36.A3 (D3), U38.5 (A4)
- new net CAM1FVLD1V8: U36.C2 (FVLD)
- new net CAM1INT1V8: U36.A2 (INT)
- new net CAM1LVLD1V8: U36.B1 (LVLD)
- new net CAM2D0: U38.15 (B5)
- new net CAM2D01V8: U38.6 (A5)
- new net CAM2D1: U38.14 (B6)
- new net CAM2D11V8: U38.7 (A6)
- new net CAM2D2: U38.13 (B7)
- new net CAM2D21V8: U38.8 (A7)
- new net CAM2D3: U38.12 (B8)
- new net CAM2D31V8: U38.9 (A8)
- new net CAMTRIG: U36.C1 (TRIG)
- new net GND: C102.1, C103.1, C104.1, R52.2, U36.D2 (GND), U38.11 (GND), U38.21 (GND)
- new net SCL1V8: U36.B2 (SCL)
- new net SDA1V8: U36.A1 (SDA)
