File: src/hardware/microcontroller.kicad_sch (KiCad schematic)
At the start: 40 parts, among them Y1 32.768kHz, Y2 32MHz

Commit message: Cleanup
Parts:
- C1: Additional Requirements X6T -> (none); Class (none) -> X6T
- C10, C12, C4, C5, C7, C8: Additional Requirements X7R -> (none); Class (none) -> X7R
- C11: Additional Requirements C0G -> (none); Class (none) -> C0G
- C3: Additional Requirements X6S -> (none); Class (none) -> X6S
- C6: Additional Requirements NP0, High Q -> (none); Class (none) -> NP0
- C9: Additional Requirements NP0 -> (none); Class (none) -> NP0
- C? (x2): Additional Requirements C0G/NP0 -> (none); Class (none) -> C0G/NP0
- C?: Additional Requirements X5R -> (none); Class (none) -> X5R
- FB1: Additional Requirements 120Ω at 100MHz, 500mΩ Max -> (none); Resistance (none) -> 120Ω at 100MHz, 500mΩ Max
- L1: Additional Requirements 650mΩ -> (none); Resistance (none) -> 650mΩ
- Y1, Y2: Additional Requirements Cl = 6~9pF -> (none); Cl (none) -> 6~9pF

Commit message: Added Accelerometer Clock; Cleanup & Fixes
Parts:
- R? (x6): value 10k -> 10kΩ
- R?: value 200k -> 200kΩ
Connections:
- net ACCCLK is gone; now on net SCL: U?.9 (P1.08/CLK16M/EXTREF)
- net LCDCMD is gone; now on net AIN: U?.18 (P2.07/TRACEDATA(0)/SWO)
- net LCDCS is gone; now on net AIN: U?.21 (P2.10/TRACEDATA(3))
- net LORACS is gone; now on net AIN: U?.16 (P2.05)
- net MISO is gone; now on net AIN: U?.20 (P2.09/TRACEDATA(2))
- net MOSI is gone; now on net AIN: U?.19 (P2.08/TRACEDATA(1))
- net MSDCS is gone; now on net AIN: U?.15 (P2.04)
- net AIN: now also U?.11 (P2.00), U?.12 (P2.01), U?.13 (P2.02), U?.14 (P2.03); no longer U?.27 (P0.02), U?.28 (P0.03/GRTCPWM), U?.37 (P1.09/ASO(2)/RADIO(0))
- net SCL: no longer U?.12 (P2.01)
- net SCL2: now also U?.28 (P0.03/GRTCPWM); no longer U?.14 (P2.03)
- net SDA: now also U?.37 (P1.09/ASO(2)/RADIO(0)); no longer U?.11 (P2.00)
- net SDA2: now also U?.27 (P0.02); no longer U?.13 (P2.02)

Commit message: Cleanup & Fixes; Added footprints; Removed Light sensors
Parts:
- removed TP?: TestPoint_2Pole, symbol Connector:TestPoint_2Pole
- removed Y1: 32.768kHz, symbol Device:Crystal_GND24
- removed Y2: 32MHz, symbol Device:Crystal
- added TP1: TestPoint_2Pole, TestPoint:TestPoint_2Pads_Pitch2.54mm_Drill0.8mm, symbol Connector:TestPoint_2Pole
- added Y1: ABS07-32.768KHZ-7-T, Project:XTAL_ABS07-32.768KHZ-7-T, symbol ABS07-32.768KHZ-7-T:ABS07-32.768KHZ-7-T
- added Y2: ECS-320-8-37B-CKY-TR, Project:XTAL_ECS-160-9-37-CKM-TR, symbol ECS-320-8-37B-CKY-TR:ECS-320-8-37B-CKY-TR
- ANT1: renamed from ANT?; footprint W3102:IND_W3102 -> Project:WS2816C-1313-4P
- C1: renamed from C6; footprint (none) -> Capacitor_SMD:C_0603_1608Metric
- C10: renamed from C1; footprint (none) -> Capacitor_SMD:C_0603_1608Metric
- C11: renamed from C8; footprint (none) -> Capacitor_SMD:C_0603_1608Metric
- C12: renamed from C5; footprint (none) -> Capacitor_SMD:C_0603_1608Metric
- C13: renamed from C7; footprint (none) -> Capacitor_SMD:C_0603_1608Metric
- C14: renamed from C12; footprint (none) -> Capacitor_SMD:C_0603_1608Metric
- C15: renamed from C4; footprint (none) -> Capacitor_SMD:C_0603_1608Metric
- C16: renamed from C2; footprint (none) -> Capacitor_SMD:C_0603_1608Metric
- C17, C5, C8, C9: renamed from C?; footprint (none) -> Capacitor_SMD:C_0603_1608Metric
- C2: renamed from C13; footprint (none) -> Capacitor_SMD:C_0603_1608Metric
- C3: renamed from C9; footprint (none) -> Capacitor_SMD:C_0603_1608Metric
- C4: renamed from C11; footprint (none) -> Capacitor_SMD:C_0603_1608Metric
- C6: renamed from C10; footprint (none) -> Capacitor_SMD:C_0603_1608Metric
- C7: renamed from C3; footprint (none) -> Capacitor_SMD:C_0603_1608Metric
- L1: renamed from L2; footprint (none) -> Inductor_SMD:L_0402_1005Metric
- L2: renamed from L3; footprint (none) -> Inductor_SMD:L_0402_1005Metric
- L3: renamed from L4; footprint (none) -> Inductor_SMD:L_0402_1005Metric
- L4, L5: renamed from L?; footprint (none) -> Inductor_SMD:L_0402_1005Metric
- L6: renamed from L1; footprint (none) -> Inductor_SMD:L_0402_1005Metric
- R1: footprint (none) -> Resistor_SMD:R_0603_1608Metric
- R2, R3, R4, R5, R6, R7, R8, R9: renamed from R?; footprint (none) -> Resistor_SMD:R_0603_1608Metric
- U1: renamed from U?; footprint NRF54L15-QFAA-R:QFN40P600X600X90-49N -> Project:QFN40P600X600X90-49N
- U2: renamed from U?; footprint SR4W035_4X6_ANT -> Project:SR4W035_4X6_ANT
- U3: renamed from U?; footprint PCA9306DQER:SON35P140X100X40-8N -> Project:SON35P140X100X40-8N
Connections:
- net GND: now also Y2.2 (GND), Y2.4 (GND)
- net at U1.1 (P1.00/XL1): now also Y1.2
- net at U1.2 (P1.01/XL2): now also Y1.1
- net at U1.25 (SWDIO): now also TP1.2
- net at U1.26 (SWDCLK): now also TP1.1
- net XC1: now reaches U1.34 (XC1)
- net XC1: now also U1.35 (XC2), Y2.1 (IN/OUT), Y2.3 (OUT/IN)
- net AIN renamed GPIO

Commit message: Cleanup & Fixes; Changed GPIO; Added Camera; Added Microphone
Connections:
- net GPIO: no longer U1.41 (P1.13/RADIO(4)/AIN6), U1.42 (P1.14/RADIO(5)/AIN7)
- new net PDMCLK: U1.42 (P1.14/RADIO(5)/AIN7)
- new net PDMDIN: U1.41 (P1.13/RADIO(4)/AIN6)
Changed lines of the file:
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@@
 	(wire
 		(pts
-			(xy 153.67 125.73) (xy 149.86 125.73)
+			(xy 143.51 158.75) (xy 143.51 160.02)
 		)
 		(stroke
@@
 	(wire
 		(pts
-			(xy 149.86 160.02) (xy 143.51 160.02)
-		)
-		(stroke
-			(width 0)
-			(type default)
-		)
-	)
-	(wire
-		(pts
 			(xy 130.81 97.79) (xy 137.16 97.79)
 		)
@@
 	(wire
 		(pts
-			(xy 149.86 127) (xy 143.51 127)
-		)
-		(stroke
-			(width 0)
-			(type default)
-		)
-	)
-	(wire
-		(pts
 			(xy 238.76 39.37) (xy 224.79 39.37)
 		)
@@
 	(wire
 		(pts
+			(xy 60.96 175.26) (xy 62.23 175.26)
+		)
+		(stroke
+			(width 0)
+			(type default)
+		)
+	)
+	(wire
+		(pts
 			(xy 44.45 147.32) (xy 40.64 147.32)
 		)
@@
 	(wire
 		(pts
+			(xy 144.78 139.7) (xy 143.51 139.7)
+		)
+		(stroke
+			(width 0)
+			(type default)
+		)
+	)
+	(wire
+		(pts
 			(xy 82.55 36.83) (xy 82.55 39.37)
 		)
@@
 	(wire
 		(pts
-			(xy 143.51 137.16) (xy 160.02 137.16)
+			(xy 60.96 147.32) (xy 62.23 147.32)
 		)
 		(stroke
@@
 	(wire
 		(pts
+			(xy 144.78 125.73) (xy 143.51 125.73)
+		)
+		(stroke
+			(width 0)
+			(type default)
+		)
+	)
+	(wire
+		(pts
 			(xy 189.23 86.36) (xy 196.85 86.36)
 		)
@@
 	(wire
 		(pts
+			(xy 143.51 125.73) (xy 143.51 127)
+		)
+		(stroke
+			(width 0)
+			(type default)
+		)
+	)
+	(wire
+		(pts
 			(xy 224.79 39.37) (xy 224.79 34.29)
 		)
@@
 	(wire
 		(pts
-			(xy 160.02 139.7) (xy 143.51 139.7)
-		)
-		(stroke
-			(width 0)
-			(type default)
-		)
-	)
-	(wire
-		(pts
 			(xy 143.51 167.64) (xy 160.02 167.64)
 		)
@@
 	(wire
 		(pts
-			(xy 154.94 158.75) (xy 149.86 158.75)
-		)
-		(stroke
-			(width 0)
-			(type default)
-		)
-	)
-	(wire
-		(pts
 			(xy 175.26 86.36) (xy 182.88 86.36)
 		)
@@
 	(wire
 		(pts
-			(xy 149.86 158.75) (xy 149.86 160.02)
+			(xy 144.78 158.75) (xy 143.51 158.75)
 		)
 		(stroke
@@
 	(wire
 		(pts
+			(xy 60.96 144.78) (xy 62.23 144.78)
+		)
+		(stroke
+			(width 0)
+			(type default)
+		)
+	)
+	(wire
+		(pts
 			(xy 58.42 36.83) (xy 55.88 36.83)
 		)
@@
 	(wire
 		(pts
+			(xy 144.78 137.16) (xy 143.51 137.16)
+		)
+		(stroke
+			(width 0)
+			(type default)
+		)
+	)
+	(wire
+		(pts
 			(xy 27.94 124.46) (xy 27.94 129.54)
 		)
@@
 		(pts
 			(xy 38.1 127) (xy 62.23 127)
-		)
-		(stroke
-			(width 0)
-			(type default)
-		)
-	)
-	(wire
-		(pts
-			(xy 149.86 125.73) (xy 149.86 127)
 		)
 		(stroke
@@
 		)
 	)
-	(label "TAMPC"
-		(at 50.8 167.64 0)
-		(effects
-			(font
-				(size 1.27 1.27)
-			)
-			(justify left bottom)
-		)
-	)
 	(label "ANT"
 		(at 30.48 36.83 180)
@@
 		)
 	)
-	(label "GPIO"
-		(at 160.02 139.7 180)
-		(effects
-			(font
-				(size 1.27 1.27)
-			)
-			(justify right bottom)
-		)
-	)
 	(label "PIN48"
 		(at 157.48 86.36 0)
@@
 		)
 	)
-	(label "TAMPC"
-		(at 50.8 172.72 0)
-		(effects
-			(font
-				(size 1.27 1.27)
-			)
-			(justify left bottom)
-		)
-	)
 	(label "XC1"
 		(at 120.65 81.28 180)
@@
 	)
 	(label "GPIO"
-		(at 160.02 137.16 180)
-		(effects
-			(font
-				(size 1.27 1.27)
-			)
-			(justify right bottom)
-		)
-	)
-	(label "GPIO"
 		(at 45.72 139.7 0)
 		(effects
@@
 			)
 			(justify right bottom)
-		)
-	)
-	(label "TAMPC"
-		(at 50.8 165.1 0)
-		(effects
-			(font
-				(size 1.27 1.27)
-			)
-			(justify left bottom)
-		)
-	)
-	(label "TAMPC"
-		(at 50.8 170.18 0)
-		(effects
-			(font
-				(size 1.27 1.27)
-			)
-			(justify left bottom)
 		)
 	)
@@
 	(global_label "SCL2"
 		(shape output)
-		(at 62.23 147.32 180)
+		(at 60.96 147.32 180)
 		(fields_autoplaced yes)
 		(effects
@@
 		)
 		(property "Intersheetrefs" "${INTERSHEET_REFS}"
-			(at 54.5277 147.32 0)
+			(at 53.2577 147.32 0)
 			(effects
 				(font
@@
 	(global_label "SDA2"
 		(shape bidirectional)
-		(at 62.23 144.78 180)
+		(at 60.96 144.78 180)
 		(fields_autoplaced yes)
 		(effects
@@
 		)
 		(property "Intersheetrefs" "${INTERSHEET_REFS}"
-			(at 53.3559 144.78 0)
+			(at 52.0859 144.78 0)
 			(effects
 				(font
@@
 	(global_label "SCL"
 		(shape output)
-		(at 62.23 175.26 180)
+		(at 60.96 175.26 180)
 		(fields_autoplaced yes)
 		(effects
@@
 		)
 		(property "Intersheetrefs" "${INTERSHEET_REFS}"
-			(at 55.7372 175.26 0)
+			(at 54.4672 175.26 0)
 			(effects
 				(font
@@
 	(global_label "SDA"
 		(shape bidirectional)
-		(at 153.67 125.73 0)
+		(at 144.78 125.73 0)
 		(fields_autoplaced yes)
 		(effects
@@
 		)
 		(property "Intersheetrefs" "${INTERSHEET_REFS}"
-			(at 161.3346 125.73 0)
+			(at 152.4446 125.73 0)
 			(effects
 				(font
@@
 	(global_label "SCK"
 		(shape output)
-		(at 154.94 158.75 0)
+		(at 144.78 158.75 0)
 		(fields_autoplaced yes)
 		(effects
@@
 		)
 		(property "Intersheetrefs" "${INTERSHEET_REFS}"
-			(at 161.6747 158.75 0)
+			(at 151.5147 158.75 0)
 			(effects
 				(font
@@
 		)
 	)
+	(global_label "PDMDIN"
+		(shape input)
+		(at 144.78 137.16 0)
+		(fields_autoplaced yes)
+		(effects
+			(font
+				(size 1.27 1.27)
+			)
+			(justify left)
+		)
+		(property "Intersheetrefs" "${INTERSHEET_REFS}"
+			(at 154.9619 137.16 0)
+			(effects
+				(font
+					(size 1.27 1.27)
+				)
+				(justify left)
+				(hide yes)
+			)
+		)
+	)
 	(global_label "BTN1"
 		(shape input)
@@
 				(hide yes)
 			)
+		)
+	)
+	(global_label "PDMCLK"
+		(shape output)
+		(at 144.78 139.7 0)
+		(fields_autoplaced yes)
+		(effects
+			(font
+				(size 1.27 1.27)
+			)
+			(justify left)
+		)
+		(property "Intersheetrefs" "${INTERSHEET_REFS}"
+			(at 155.3247 139.7 0)
+			(effects
+				(font
+					(size 1.27 1.27)
+				)
+				(justify left)
+				(hide yes)
+			)

Commit message: Added Microphone
Parts:
- added R50: 100kΩ, Resistor_SMD:R_0603_1608Metric, symbol Device:R
Connections:
- net GND: now also R50.2
- net PDMDIN renamed PDMDATA
- net PDMDATA: now also R50.1
Changed lines of the file:
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@@
 		)
 	)
+	(global_label "PDMDATA"
+		(shape input)
+		(at 252.73 105.41 180)
+		(fields_autoplaced yes)
+		(effects
+			(font
+				(size 1.27 1.27)
+			)
+			(justify right)
+		)
+		(property "Intersheetrefs" "${INTERSHEET_REFS}"
+			(at 241.3386 105.41 0)
+			(effects
+				(font
+					(size 1.27 1.27)
+				)
+				(justify right)
+				(hide yes)
+			)
+		)
+	)
 	(global_label "SDA2"
 		(shape bidirectional)
@@
 		)
 	)
-	(global_label "PDMDIN"
+	(global_label "PDMDATA"
 		(shape input)
 		(at 144.78 137.16 0)
@@
 		)
 		(property "Intersheetrefs" "${INTERSHEET_REFS}"
-			(at 154.9619 137.16 0)
+			(at 156.1714 137.16 0)
 			(effects
 				(font
@@
 	)
 	(symbol
+		(lib_id "Device:R")
+		(at 256.54 105.41 90)
+		(unit 1)
+		(exclude_from_sim no)
+		(in_bom yes)
+		(on_board yes)
+		(dnp no)
+		(fields_autoplaced yes)
+		(property "Reference" "R50"
+			(at 256.54 99.06 90)
+			(effects
+				(font
+					(size 1.27 1.27)
+				)
+			)
+		)
+		(property "Value" "100kΩ"
+			(at 256.54 101.6 90)
+			(effects
+				(font
+					(size 1.27 1.27)
+				)
+			)
+		)
+		(property "Footprint" "Resistor_SMD:R_0603_1608Metric"
+			(at 256.54 107.188 90)
+			(effects
+				(font
+					(size 1.27 1.27)
+				)
+				(hide yes)
+			)
+		)
+		(property "Datasheet" "~"
+			(at 256.54 105.41 0)
+			(effects
+				(font
+					(size 1.27 1.27)
+				)
+				(hide yes)
+			)
+		)
+		(property "Description" "Resistor"
+			(at 256.54 105.41 0)
+			(effects
+				(font
+					(size 1.27 1.27)
+				)
+				(hide yes)
+			)
+		)
+		(pin "1"
+		)
+		(pin "2"
+		)
+		(instances
+			(project "raywatch"
+				(path "/7b654ee8-2a53-4d39-8b7d-32c7bb3cb0ed/fa39c797-7f88-47af-b50c-765e69cbd658"
+					(reference "R50")
+					(unit 1)
+				)
+			)
+		)
+	)
+	(symbol
 		(lib_id "Device:C")
 		(at 88.9 36.83 90)
@@
 					(unit 1)
 				)
+			)
+		)
+	)
+	(symbol
+		(lib_id "power:GND")
+		(at 260.35 105.41 90)
+		(unit 1)
+		(exclude_from_sim no)
+		(in_bom yes)
+		(on_board yes)
+		(dnp no)
+		(fields_autoplaced yes)
+		(property "Reference" "#PWR0411"
+			(at 266.7 105.41 0)
+			(effects
+				(font
+					(size 1.27 1.27)
+				)
+				(hide yes)
+			)
+		)
+		(property "Value" "GND"
+			(at 264.16 105.4099 90)
+			(effects
+				(font
+					(size 1.27 1.27)
+				)
+				(justify right)
+			)
+		)
+		(property "Footprint" ""
+			(at 260.35 105.41 0)
+			(effects
+				(font
+					(size 1.27 1.27)
+				)
+				(hide yes)
+			)
+		)
+		(property "Datasheet" ""
+			(at 260.35 105.41 0)
+			(effects
+				(font
+					(size 1.27 1.27)
+				)
+				(hide yes)
+			)
+		)
+		(property "Description" "Power symbol creates a global label with name \"GND\" , ground"
+			(at 260.35 105.41 0)
+			(effects
+				(font
+					(size 1.27 1.27)
+				)
+				(hide yes)
+			)
+		)
+		(pin "1"
+		)
+		(instances
+			(project "raywatch"
+				(path "/7b654ee8-2a53-4d39-8b7d-32c7bb3cb0ed/fa39c797-7f88-47af-b50c-765e69cbd658"
+					(reference "#PWR0411")
+					(unit 1)
+				)

Commit message: Removed Camera because currently not viable
Connections:
- net GPIO: now also U1.37 (P1.09/ASO(2)/RADIO(0)); no longer U1.8 (P1.07/ASI(1)/AIN3)
- net SCL: now also U1.28 (P0.03/GRTCPWM); no longer U1.9 (P1.08/CLK16M/EXTREF)
- net SCL2: now also U1.9 (P1.08/CLK16M/EXTREF); no longer U1.28 (P0.03/GRTCPWM)
- net SDA: now also U1.27 (P0.02); no longer U1.37 (P1.09/ASO(2)/RADIO(0))
- net SDA2: now also U1.8 (P1.07/ASI(1)/AIN3); no longer U1.27 (P0.02)
Changed lines of the file:
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@@
-	(wire
-		(pts
-			(xy 60.96 175.26) (xy 62.23 175.26)
-		)
-		(stroke
-			(width 0)
-			(type default)
-		)
-	)
 	(wire
 		(pts
@@
 	(wire
 		(pts
-			(xy 144.78 139.7) (xy 143.51 139.7)
-		)
-		(stroke
-			(width 0)
-			(type default)
-		)
-	)
-	(wire
-		(pts
 			(xy 82.55 36.83) (xy 82.55 39.37)
 		)
@@
 	(wire
 		(pts
-			(xy 60.96 147.32) (xy 62.23 147.32)
-		)
-		(stroke
-			(width 0)
-			(type default)
-		)
-	)
-	(wire
-		(pts
 			(xy 130.81 92.71) (xy 137.16 92.71)
 		)
@@
 	(wire
 		(pts
-			(xy 144.78 125.73) (xy 143.51 125.73)
-		)
-		(stroke
-			(width 0)
-			(type default)
-		)
-	)
-	(wire
-		(pts
 			(xy 189.23 86.36) (xy 196.85 86.36)
 		)
@@
 	(wire
 		(pts
-			(xy 143.51 125.73) (xy 143.51 127)
-		)
-		(stroke
-			(width 0)
-			(type default)
-		)
-	)
-	(wire
-		(pts
 			(xy 224.79 39.37) (xy 224.79 34.29)
 		)
@@
 	(wire
 		(pts
-			(xy 60.96 144.78) (xy 62.23 144.78)
-		)
-		(stroke
-			(width 0)
-			(type default)
-		)
-	)
-	(wire
-		(pts
 			(xy 58.42 36.83) (xy 55.88 36.83)
 		)
@@
 	(wire
 		(pts
-			(xy 144.78 137.16) (xy 143.51 137.16)
-		)
-		(stroke
-			(width 0)
-			(type default)
-		)
-	)
-	(wire
-		(pts
 			(xy 27.94 124.46) (xy 27.94 129.54)
 		)
@@
 	(wire
 		(pts
-			(xy 45.72 172.72) (xy 62.23 172.72)
+			(xy 160.02 127) (xy 143.51 127)
 		)
 		(stroke
@@
 	)
 	(label "GPIO"
-		(at 45.72 172.72 0)
-		(effects
-			(font
-				(size 1.27 1.27)
-			)
-			(justify left bottom)
+		(at 160.02 127 180)
+		(effects
+			(font
+				(size 1.27 1.27)
+			)
+			(justify right bottom)
 		)
 	)
@@
 	(global_label "SCL2"
 		(shape output)
-		(at 60.96 147.32 180)
+		(at 62.23 175.26 180)
 		(fields_autoplaced yes)
 		(effects
@@
 		)
 		(property "Intersheetrefs" "${INTERSHEET_REFS}"
-			(at 53.2577 147.32 0)
+			(at 54.5277 175.26 0)
 			(effects
 				(font
@@
 	(global_label "SDA2"
 		(shape bidirectional)
-		(at 60.96 144.78 180)
+		(at 62.23 172.72 180)
 		(fields_autoplaced yes)
 		(effects
@@
 		)
 		(property "Intersheetrefs" "${INTERSHEET_REFS}"
-			(at 52.0859 144.78 0)
+			(at 53.3559 172.72 0)
 			(effects
 				(font
@@
 	(global_label "SCL"
 		(shape output)
-		(at 60.96 175.26 180)
+		(at 62.23 147.32 180)
 		(fields_autoplaced yes)
 		(effects
@@
 		)
 		(property "Intersheetrefs" "${INTERSHEET_REFS}"
-			(at 54.4672 175.26 0)
+			(at 55.7372 147.32 0)
 			(effects
 				(font
@@
 	(global_label "SDA"
 		(shape bidirectional)
-		(at 144.78 125.73 0)
-		(fields_autoplaced yes)
-		(effects
-			(font
-				(size 1.27 1.27)
-			)
-			(justify left)
-		)
-		(property "Intersheetrefs" "${INTERSHEET_REFS}"
-			(at 152.4446 125.73 0)
-			(effects
-				(font
-					(size 1.27 1.27)
-				)
-				(justify left)
+		(at 62.23 144.78 180)
+		(fields_autoplaced yes)
+		(effects
+			(font
+				(size 1.27 1.27)
+			)
+			(justify right)
+		)
+		(property "Intersheetrefs" "${INTERSHEET_REFS}"
+			(at 54.5654 144.78 0)
+			(effects
+				(font
+					(size 1.27 1.27)
+				)
+				(justify right)
 				(hide yes)
 			)
@@
 	(global_label "PDMDATA"
 		(shape input)
-		(at 144.78 137.16 0)
+		(at 143.51 137.16 0)
 		(fields_autoplaced yes)
 		(effects
@@
 		)
 		(property "Intersheetrefs" "${INTERSHEET_REFS}"
-			(at 156.1714 137.16 0)
+			(at 154.9014 137.16 0)
 			(effects
 				(font
@@
 	(global_label "PDMCLK"
 		(shape output)
-		(at 144.78 139.7 0)
+		(at 143.51 139.7 0)
 		(fields_autoplaced yes)
 		(effects
@@
 		)
 		(property "Intersheetrefs" "${INTERSHEET_REFS}"
-			(at 155.3247 139.7 0)
-			(effects
-				(font
+			(at 154.0547 139.7 0)
+			(effects
+				(font

Commit message: Updated GPIO
Parts:
- C2: now not fitted; now left out of the parts list
Connections:
- net GPIO: no longer U1.18 (P2.07/TRACEDATA(0)/SWO), U1.19 (P2.08/TRACEDATA(1)), U1.20 (P2.09/TRACEDATA(2))
- new net LCDCMD: U1.20 (P2.09/TRACEDATA(2))
- new net MISO: U1.19 (P2.08/TRACEDATA(1))
- new net MOSI: U1.18 (P2.07/TRACEDATA(0)/SWO)
Other:
- moved on the sheet: C12, C14, C16
