File: src/hardware/solar.kicad_sch (KiCad schematic)
At the start: 0 parts

Commit message: Added Solar
Parts:
- added B? (x2): KXOB25-05X3F-TR, CHIP2_KXOB25-05X3F-TR_AAR, symbol KXOB25-05X3F-TR:KXOB25-05X3F-TR
- added C? (x3): 10µF, symbol Device:C
- added L?: 202µH, symbol Device:L
- added R?: 100K, symbol Device:R
- added R?: 400K, symbol Device:R
- added U?: TPS61099YFFT, YFF0006AFAD, symbol TPS61099YFFT:TPS61099YFFT
Connections:
- new net: B?.2, B?.2, C?.1, L?.1, U?.A1 (VIN), U?.C1 (EN)
- new net: R?.1, R?.2, U?.C2 (FB)
- new net: L?.2, U?.B1 (SW)
- new net GND: B?.1, B?.1, C?.2, C?.2, C?.2, R?.2, U?.A2 (GND)
- new net SOLAR: C?.1, C?.1, R?.1, U?.B2 (VOUT)

Commit message: Changed power symboles
Connections:
- net SOLAR renamed VSOLAR
Changed lines of the file:
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@@
-		)
-	)
-	(wire
-		(pts
-			(xy 194.31 95.25) (xy 194.31 97.79)
-		)
-		(stroke
-			(width 0)
-			(type default)
-		)
-	)
-	(global_label "SOLAR"
-		(shape passive)
-		(at 194.31 95.25 90)
-		(fields_autoplaced yes)
-		(effects
-			(font
-				(size 1.27 1.27)
-			)
-			(justify left)
-		)
-		(property "Intersheetrefs" "${INTERSHEET_REFS}"
-			(at 194.31 87.4494 90)
-			(effects
-				(font
-					(size 1.27 1.27)
-				)
-				(justify left)
-				(hide yes)
-			)
 		)
 	)
@@
 					(unit 1)
 				)
+			)
+		)
+	)
+	(symbol
+		(lib_id "power:LINE")
+		(at 194.31 97.79 0)
+		(unit 1)
+		(exclude_from_sim no)
+		(in_bom yes)
+		(on_board yes)
+		(dnp no)
+		(fields_autoplaced yes)
+		(property "Reference" "#PWR0371"
+			(at 194.31 101.6 0)
+			(effects
+				(font
+					(size 1.27 1.27)
+				)
+				(hide yes)
+			)
+		)
+		(property "Value" "VSOLAR"
+			(at 194.31 92.71 0)
+			(effects
+				(font
+					(size 1.27 1.27)
+				)
+			)
+		)
+		(property "Footprint" ""
+			(at 194.31 97.79 0)
+			(effects
+				(font
+					(size 1.27 1.27)
+				)
+				(hide yes)
+			)
+		)
+		(property "Datasheet" ""
+			(at 194.31 97.79 0)
+			(effects
+				(font
+					(size 1.27 1.27)
+				)
+				(hide yes)
+			)
+		)
+		(property "Description" "Power symbol creates a global label with name \"LINE\""
+			(at 194.31 97.79 0)
+			(effects
+				(font
+					(size 1.27 1.27)
+				)
+				(hide yes)
+			)
+		)
+		(pin "1"
+		)
+		(instances
+			(project "raywatch"
+				(path "/7b654ee8-2a53-4d39-8b7d-32c7bb3cb0ed/6e6a70ea-4db2-4b59-a2d7-c468f9b8b5a6/94d294dd-af54-43f7-9e9b-15472c788437"
+					(reference "#PWR0371")
+					(unit 1)
+				)

Commit message: Added battery
Parts:
- L?: value 202µH -> 2.2µH
Changed lines of the file:
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@@
 			)
 		)
-		(property "Value" "202µH"
+		(property "Value" "2.2µH"
 			(at 148.59 77.47 90)
 			(effects

Commit message: Added Accelerometer Clock; Cleanup & Fixes
Parts:
- R?: value 100K -> 100KΩ
- R?: value 400K -> 400KΩ
Changed lines of the file:
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@@
 			)
 		)
-		(property "Value" "100K"
+		(property "Value" "100KΩ"
 			(at 175.26 110.4899 0)
 			(effects
@@
 			)
 		)
-		(property "Value" "400K"
+		(property "Value" "400KΩ"
 			(at 175.26 102.8699 0)
 			(effects

Commit message: Cleanup & Fixes; Added footprints; Removed Light sensors
Parts:
- B1, B2: renamed from B?; footprint CHIP2_KXOB25-05X3F-TR_AAR -> Project:CHIP2_KXOB25-05X3F-TR_AAR
- C68, C69, C70: renamed from C?; footprint (none) -> Capacitor_SMD:C_0603_1608Metric
- L9: renamed from L?; footprint (none) -> Inductor_SMD:L_0402_1005Metric
- R35, R36: renamed from R?; footprint (none) -> Resistor_SMD:R_0603_1608Metric
- U23: renamed from U?; footprint YFF0006AFAD -> Project:YFF0006AFAD
Changed lines of the file:
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@@
 		(on_board yes)
 		(dnp no)
-		(property "Reference" "C?"
+		(fields_autoplaced yes)
+		(property "Reference" "C69"
 			(at 186.69 100.3299 0)
 			(effects
@@
 			)
 		)
-		(property "Footprint" ""
+		(property "Footprint" "Capacitor_SMD:C_0603_1608Metric"
 			(at 183.8452 105.41 0)
 			(effects
@@
 			(project "raywatch"
 				(path "/7b654ee8-2a53-4d39-8b7d-32c7bb3cb0ed/6e6a70ea-4db2-4b59-a2d7-c468f9b8b5a6/94d294dd-af54-43f7-9e9b-15472c788437"
-					(reference "C?")
+					(reference "C69")
 					(unit 1)
 				)
@@
 		(dnp no)
 		(fields_autoplaced yes)
-		(property "Reference" "#PWR0340"
+		(property "Reference" "#PWR0347"
 			(at 194.31 111.76 0)
 			(effects
@@
 			(project "raywatch"
 				(path "/7b654ee8-2a53-4d39-8b7d-32c7bb3cb0ed/6e6a70ea-4db2-4b59-a2d7-c468f9b8b5a6/94d294dd-af54-43f7-9e9b-15472c788437"
-					(reference "#PWR0340")
+					(reference "#PWR0347")
 					(unit 1)
 				)
@@
 		(dnp no)
 		(fields_autoplaced yes)
-		(property "Reference" "#PWR0371"
+		(property "Reference" "#PWR0346"
 			(at 194.31 101.6 0)
 			(effects
@@
 			(project "raywatch"
 				(path "/7b654ee8-2a53-4d39-8b7d-32c7bb3cb0ed/6e6a70ea-4db2-4b59-a2d7-c468f9b8b5a6/94d294dd-af54-43f7-9e9b-15472c788437"
-					(reference "#PWR0371")
+					(reference "#PWR0346")
 					(unit 1)
 				)
@@
 		(dnp no)
 		(fields_autoplaced yes)
-		(property "Reference" "#PWR0338"
+		(property "Reference" "#PWR0344"
 			(at 172.72 119.38 0)
 			(effects
@@
 			(project "raywatch"
 				(path "/7b654ee8-2a53-4d39-8b7d-32c7bb3cb0ed/6e6a70ea-4db2-4b59-a2d7-c468f9b8b5a6/94d294dd-af54-43f7-9e9b-15472c788437"
-					(reference "#PWR0338")
+					(reference "#PWR0344")
 					(unit 1)
 				)
@@
 		(dnp no)
 		(fields_autoplaced yes)
-		(property "Reference" "C?"
+		(property "Reference" "C68"
 			(at 123.19 95.2499 0)
 			(effects
@@
 			)
 		)
-		(property "Footprint" ""
+		(property "Footprint" "Capacitor_SMD:C_0603_1608Metric"
 			(at 126.0348 100.33 0)
 			(effects
@@
 			(project "raywatch"
 				(path "/7b654ee8-2a53-4d39-8b7d-32c7bb3cb0ed/6e6a70ea-4db2-4b59-a2d7-c468f9b8b5a6/94d294dd-af54-43f7-9e9b-15472c788437"
-					(reference "C?")
+					(reference "C68")
 					(unit 1)
 				)
@@
 		(dnp no)
 		(fields_autoplaced yes)
-		(property "Reference" "#PWR0335"
+		(property "Reference" "#PWR0340"
 			(at 95.885 99.06 0)
 			(effects
@@
 			(project "raywatch"
 				(path "/7b654ee8-2a53-4d39-8b7d-32c7bb3cb0ed/6e6a70ea-4db2-4b59-a2d7-c468f9b8b5a6/94d294dd-af54-43f7-9e9b-15472c788437"
-					(reference "#PWR0335")
+					(reference "#PWR0340")
 					(unit 1)
 				)
@@
 		(dnp no)
 		(fields_autoplaced yes)
-		(property "Reference" "R?"
+		(property "Reference" "R36"
 			(at 175.26 107.9499 0)
 			(effects
@@
 			)
 		)
-		(property "Footprint" ""
+		(property "Footprint" "Resistor_SMD:R_0603_1608Metric"
 			(at 170.942 109.22 90)
 			(effects
@@
 			(project "raywatch"
 				(path "/7b654ee8-2a53-4d39-8b7d-32c7bb3cb0ed/6e6a70ea-4db2-4b59-a2d7-c468f9b8b5a6/94d294dd-af54-43f7-9e9b-15472c788437"
-					(reference "R?")
+					(reference "R36")
 					(unit 1)
 				)
@@
 		(dnp no)
 		(fields_autoplaced yes)
-		(property "Reference" "#PWR0339"
+		(property "Reference" "#PWR0345"
 			(at 182.88 111.76 0)
 			(effects
@@
 			(project "raywatch"
 				(path "/7b654ee8-2a53-4d39-8b7d-32c7bb3cb0ed/6e6a70ea-4db2-4b59-a2d7-c468f9b8b5a6/94d294dd-af54-43f7-9e9b-15472c788437"
-					(reference "#PWR0339")
+					(reference "#PWR0345")
 					(unit 1)
 				)
@@
 		(on_board yes)
 		(dnp no)
-		(property "Reference" "U?"
+		(fields_autoplaced yes)
+		(property "Reference" "U23"
 			(at 148.59 82.55 0)
 			(effects
@@
 			)
 		)
-		(property "Footprint" "YFF0006AFAD"
+		(property "Footprint" "Project:YFF0006AFAD"
 			(at 148.59 100.33 0)
 			(effects
@@
 			(project "raywatch"
 				(path "/7b654ee8-2a53-4d39-8b7d-32c7bb3cb0ed/6e6a70ea-4db2-4b59-a2d7-c468f9b8b5a6/94d294dd-af54-43f7-9e9b-15472c788437"
-					(reference "U?")
+					(reference "U23")
 					(unit 1)
 				)
@@
 		(dnp no)
 		(fields_autoplaced yes)
-		(property "Reference" "L?"
+		(property "Reference" "L9"
 			(at 148.59 74.93 90)
 			(effects
@@
 			)
 		)
-		(property "Footprint" ""
+		(property "Footprint" "Inductor_SMD:L_0402_1005Metric"
 			(at 148.59 80.01 0)
 			(effects
@@
 			(project "raywatch"
 				(path "/7b654ee8-2a53-4d39-8b7d-32c7bb3cb0ed/6e6a70ea-4db2-4b59-a2d7-c468f9b8b5a6/94d294dd-af54-43f7-9e9b-15472c788437"
-					(reference "L?")
+					(reference "L9")
 					(unit 1)
 				)
@@
 		(on_board yes)
 		(dnp no)
-		(property "Reference" "C?"
+		(fields_autoplaced yes)
+		(property "Reference" "C70"
 			(at 198.12 100.3299 0)
 			(effects
@@
 			)
 		)
-		(property "Footprint" ""
+		(property "Footprint" "Capacitor_SMD:C_0603_1608Metric"
 			(at 195.2752 105.41 0)
 			(effects
@@
 			(project "raywatch"
 				(path "/7b654ee8-2a53-4d39-8b7d-32c7bb3cb0ed/6e6a70ea-4db2-4b59-a2d7-c468f9b8b5a6/94d294dd-af54-43f7-9e9b-15472c788437"
-					(reference "C?")
+					(reference "C70")
 					(unit 1)
 				)
@@
 		(dnp no)
 		(fields_autoplaced yes)
-		(property "Reference" "B?"
+		(property "Reference" "B2"
 			(at 101.854 100.33 0)
 			(effects
@@
 			)
 		)
-		(property "Footprint" "CHIP2_KXOB25-05X3F-TR_AAR"
+		(property "Footprint" "Project:CHIP2_KXOB25-05X3F-TR_AAR"
 			(at 96.52 110.49 0)
 			(effects
@@
 			(project "raywatch"
 				(path "/7b654ee8-2a53-4d39-8b7d-32c7bb3cb0ed/6e6a70ea-4db2-4b59-a2d7-c468f9b8b5a6/94d294dd-af54-43f7-9e9b-15472c788437"
-					(reference "B?")
+					(reference "B2")
 					(unit 1)
 				)
@@
 		(dnp no)
 		(fields_autoplaced yes)
-		(property "Reference" "R?"
+		(property "Reference" "R35"
 			(at 175.26 100.3299 0)
 			(effects
@@
 			)
 		)
-		(property "Footprint" ""
+		(property "Footprint" "Resistor_SMD:R_0603_1608Metric"
 			(at 170.942 101.6 90)
 			(effects
@@
 			(project "raywatch"
 				(path "/7b654ee8-2a53-4d39-8b7d-32c7bb3cb0ed/6e6a70ea-4db2-4b59-a2d7-c468f9b8b5a6/94d294dd-af54-43f7-9e9b-15472c788437"
-					(reference "R?")
+					(reference "R35")
 					(unit 1)
 				)
@@
 		(dnp no)
 		(fields_autoplaced yes)
-		(property "Reference" "#PWR0334"
+		(property "Reference" "#PWR0341"
 			(at 96.52 116.84 0)
 			(effects
@@
 			(project "raywatch"
 				(path "/7b654ee8-2a53-4d39-8b7d-32c7bb3cb0ed/6e6a70ea-4db2-4b59-a2d7-c468f9b8b5a6/94d294dd-af54-43f7-9e9b-15472c788437"
-					(reference "#PWR0334")
+					(reference "#PWR0341")
 					(unit 1)
 				)
@@
 		(dnp no)
 		(fields_autoplaced yes)
-		(property "Reference" "#PWR0337"
+		(property "Reference" "#PWR0343"
 			(at 166.37 116.84 0)
 			(effects
@@
 			(project "raywatch"
 				(path "/7b654ee8-2a53-4d39-8b7d-32c7bb3cb0ed/6e6a70ea-4db2-4b59-a2d7-c468f9b8b5a6/94d294dd-af54-43f7-9e9b-15472c788437"
-					(reference "#PWR0337")
+					(reference "#PWR0343")
 					(unit 1)
 				)
@@
 		(dnp no)
 		(fields_autoplaced yes)
-		(property "Reference" "B?"
+		(property "Reference" "B1"
 			(at 101.219 82.55 0)
 			(effects
@@
 			)
 		)
-		(property "Footprint" "CHIP2_KXOB25-05X3F-TR_AAR"
+		(property "Footprint" "Project:CHIP2_KXOB25-05X3F-TR_AAR"
 			(at 95.885 92.71 0)
 			(effects
@@
 			(project "raywatch"
 				(path "/7b654ee8-2a53-4d39-8b7d-32c7bb3cb0ed/6e6a70ea-4db2-4b59-a2d7-c468f9b8b5a6/94d294dd-af54-43f7-9e9b-15472c788437"
-					(reference "B?")
+					(reference "B1")
 					(unit 1)
 				)
@@
 		(dnp no)
 		(fields_autoplaced yes)
-		(property "Reference" "#PWR0336"
+		(property "Reference" "#PWR0342"
 			(at 127 106.68 0)
 			(effects
@@
 			(project "raywatch"
 				(path "/7b654ee8-2a53-4d39-8b7d-32c7bb3cb0ed/6e6a70ea-4db2-4b59-a2d7-c468f9b8b5a6/94d294dd-af54-43f7-9e9b-15472c788437"
-					(reference "#PWR0336")
-					(unit 1)
-				)
+					(reference "#PWR0342")
+					(unit 1)
+				)

Commit message: Cleanup & Fixes; Changed GPIO; Added Camera; Added Microphone
Parts:
- renumbered C68 to C66, C69 to C67, C70 to C68, R35 to R33, R36 to R34
Changed lines of the file:
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@@
 		(dnp no)
 		(fields_autoplaced yes)
-		(property "Reference" "C69"
+		(property "Reference" "C67"
 			(at 186.69 100.3299 0)
 			(effects
@@
 			(project "raywatch"
 				(path "/7b654ee8-2a53-4d39-8b7d-32c7bb3cb0ed/6e6a70ea-4db2-4b59-a2d7-c468f9b8b5a6/94d294dd-af54-43f7-9e9b-15472c788437"
-					(reference "C69")
+					(reference "C67")
 					(unit 1)
 				)
@@
 		(dnp no)
 		(fields_autoplaced yes)
-		(property "Reference" "#PWR0347"
+		(property "Reference" "#PWR0343"
 			(at 194.31 111.76 0)
 			(effects
@@
 			(project "raywatch"
 				(path "/7b654ee8-2a53-4d39-8b7d-32c7bb3cb0ed/6e6a70ea-4db2-4b59-a2d7-c468f9b8b5a6/94d294dd-af54-43f7-9e9b-15472c788437"
-					(reference "#PWR0347")
+					(reference "#PWR0343")
 					(unit 1)
 				)
@@
 		(dnp no)
 		(fields_autoplaced yes)
-		(property "Reference" "#PWR0346"
+		(property "Reference" "#PWR0342"
 			(at 194.31 101.6 0)
 			(effects
@@
 			(project "raywatch"
 				(path "/7b654ee8-2a53-4d39-8b7d-32c7bb3cb0ed/6e6a70ea-4db2-4b59-a2d7-c468f9b8b5a6/94d294dd-af54-43f7-9e9b-15472c788437"
-					(reference "#PWR0346")
+					(reference "#PWR0342")
 					(unit 1)
 				)
@@
 		(dnp no)
 		(fields_autoplaced yes)
-		(property "Reference" "#PWR0344"
+		(property "Reference" "#PWR0340"
 			(at 172.72 119.38 0)
 			(effects
@@
 			(project "raywatch"
 				(path "/7b654ee8-2a53-4d39-8b7d-32c7bb3cb0ed/6e6a70ea-4db2-4b59-a2d7-c468f9b8b5a6/94d294dd-af54-43f7-9e9b-15472c788437"
-					(reference "#PWR0344")
+					(reference "#PWR0340")
 					(unit 1)
 				)
@@
 		(dnp no)
 		(fields_autoplaced yes)
-		(property "Reference" "C68"
+		(property "Reference" "C66"
 			(at 123.19 95.2499 0)
 			(effects
@@
 			(project "raywatch"
 				(path "/7b654ee8-2a53-4d39-8b7d-32c7bb3cb0ed/6e6a70ea-4db2-4b59-a2d7-c468f9b8b5a6/94d294dd-af54-43f7-9e9b-15472c788437"
-					(reference "C68")
+					(reference "C66")
 					(unit 1)
 				)
@@
 		(dnp no)
 		(fields_autoplaced yes)
-		(property "Reference" "#PWR0340"
+		(property "Reference" "#PWR0336"
 			(at 95.885 99.06 0)
 			(effects
@@
 			(project "raywatch"
 				(path "/7b654ee8-2a53-4d39-8b7d-32c7bb3cb0ed/6e6a70ea-4db2-4b59-a2d7-c468f9b8b5a6/94d294dd-af54-43f7-9e9b-15472c788437"
-					(reference "#PWR0340")
+					(reference "#PWR0336")
 					(unit 1)
 				)
@@
 		(dnp no)
 		(fields_autoplaced yes)
-		(property "Reference" "R36"
+		(property "Reference" "R34"
 			(at 175.26 107.9499 0)
 			(effects
@@
 			(project "raywatch"
 				(path "/7b654ee8-2a53-4d39-8b7d-32c7bb3cb0ed/6e6a70ea-4db2-4b59-a2d7-c468f9b8b5a6/94d294dd-af54-43f7-9e9b-15472c788437"
-					(reference "R36")
+					(reference "R34")
 					(unit 1)
 				)
@@
 		(dnp no)
 		(fields_autoplaced yes)
-		(property "Reference" "#PWR0345"
+		(property "Reference" "#PWR0341"
 			(at 182.88 111.76 0)
 			(effects
@@
 			(project "raywatch"
 				(path "/7b654ee8-2a53-4d39-8b7d-32c7bb3cb0ed/6e6a70ea-4db2-4b59-a2d7-c468f9b8b5a6/94d294dd-af54-43f7-9e9b-15472c788437"
-					(reference "#PWR0345")
+					(reference "#PWR0341")
 					(unit 1)
 				)
@@
 		(dnp no)
 		(fields_autoplaced yes)
-		(property "Reference" "C70"
+		(property "Reference" "C68"
 			(at 198.12 100.3299 0)
 			(effects
@@
 			(project "raywatch"
 				(path "/7b654ee8-2a53-4d39-8b7d-32c7bb3cb0ed/6e6a70ea-4db2-4b59-a2d7-c468f9b8b5a6/94d294dd-af54-43f7-9e9b-15472c788437"
-					(reference "C70")
+					(reference "C68")
 					(unit 1)
 				)
@@
 		(dnp no)
 		(fields_autoplaced yes)
-		(property "Reference" "R35"
+		(property "Reference" "R33"
 			(at 175.26 100.3299 0)
 			(effects
@@
 			(project "raywatch"
 				(path "/7b654ee8-2a53-4d39-8b7d-32c7bb3cb0ed/6e6a70ea-4db2-4b59-a2d7-c468f9b8b5a6/94d294dd-af54-43f7-9e9b-15472c788437"
-					(reference "R35")
+					(reference "R33")
 					(unit 1)
 				)
@@
 		(dnp no)
 		(fields_autoplaced yes)
-		(property "Reference" "#PWR0341"
+		(property "Reference" "#PWR0337"
 			(at 96.52 116.84 0)
 			(effects
@@
 			(project "raywatch"
 				(path "/7b654ee8-2a53-4d39-8b7d-32c7bb3cb0ed/6e6a70ea-4db2-4b59-a2d7-c468f9b8b5a6/94d294dd-af54-43f7-9e9b-15472c788437"
-					(reference "#PWR0341")
+					(reference "#PWR0337")
 					(unit 1)
 				)
@@
 		(dnp no)
 		(fields_autoplaced yes)
-		(property "Reference" "#PWR0343"
+		(property "Reference" "#PWR0339"
 			(at 166.37 116.84 0)
 			(effects
@@
 			(project "raywatch"
 				(path "/7b654ee8-2a53-4d39-8b7d-32c7bb3cb0ed/6e6a70ea-4db2-4b59-a2d7-c468f9b8b5a6/94d294dd-af54-43f7-9e9b-15472c788437"
-					(reference "#PWR0343")
+					(reference "#PWR0339")
 					(unit 1)
 				)
@@
 		(dnp no)
 		(fields_autoplaced yes)
-		(property "Reference" "#PWR0342"
+		(property "Reference" "#PWR0338"
 			(at 127 106.68 0)
 			(effects
@@
 			(project "raywatch"
 				(path "/7b654ee8-2a53-4d39-8b7d-32c7bb3cb0ed/6e6a70ea-4db2-4b59-a2d7-c468f9b8b5a6/94d294dd-af54-43f7-9e9b-15472c788437"
-					(reference "#PWR0342")
-					(unit 1)
-				)
+					(reference "#PWR0338")
+					(unit 1)
+				)

Commit message: Add Light Sensor and Proximity & Gesture Sensor; Changed GPIO
Parts:
- renumbered R33 to R34, R34 to R35, U23 to U24
Changed lines of the file:
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@@
 		(dnp no)
 		(fields_autoplaced yes)
-		(property "Reference" "#PWR0343"
+		(property "Reference" "#PWR0347"
 			(at 194.31 111.76 0)
 			(effects
@@
 			(project "raywatch"
 				(path "/7b654ee8-2a53-4d39-8b7d-32c7bb3cb0ed/6e6a70ea-4db2-4b59-a2d7-c468f9b8b5a6/94d294dd-af54-43f7-9e9b-15472c788437"
-					(reference "#PWR0343")
+					(reference "#PWR0347")
 					(unit 1)
 				)
@@
 		(dnp no)
 		(fields_autoplaced yes)
-		(property "Reference" "#PWR0342"
+		(property "Reference" "#PWR0346"
 			(at 194.31 101.6 0)
 			(effects
@@
 			(project "raywatch"
 				(path "/7b654ee8-2a53-4d39-8b7d-32c7bb3cb0ed/6e6a70ea-4db2-4b59-a2d7-c468f9b8b5a6/94d294dd-af54-43f7-9e9b-15472c788437"
-					(reference "#PWR0342")
+					(reference "#PWR0346")
 					(unit 1)
 				)
@@
 		(dnp no)
 		(fields_autoplaced yes)
-		(property "Reference" "#PWR0340"
+		(property "Reference" "#PWR0344"
 			(at 172.72 119.38 0)
 			(effects
@@
 			(project "raywatch"
 				(path "/7b654ee8-2a53-4d39-8b7d-32c7bb3cb0ed/6e6a70ea-4db2-4b59-a2d7-c468f9b8b5a6/94d294dd-af54-43f7-9e9b-15472c788437"
-					(reference "#PWR0340")
+					(reference "#PWR0344")
 					(unit 1)
 				)
@@
 		(dnp no)
 		(fields_autoplaced yes)
-		(property "Reference" "#PWR0336"
+		(property "Reference" "#PWR0340"
 			(at 95.885 99.06 0)
 			(effects
@@
 			(project "raywatch"
 				(path "/7b654ee8-2a53-4d39-8b7d-32c7bb3cb0ed/6e6a70ea-4db2-4b59-a2d7-c468f9b8b5a6/94d294dd-af54-43f7-9e9b-15472c788437"
-					(reference "#PWR0336")
+					(reference "#PWR0340")
 					(unit 1)
 				)
@@
 		(dnp no)
 		(fields_autoplaced yes)
-		(property "Reference" "R34"
+		(property "Reference" "R35"
 			(at 175.26 107.9499 0)
 			(effects
@@
 			(project "raywatch"
 				(path "/7b654ee8-2a53-4d39-8b7d-32c7bb3cb0ed/6e6a70ea-4db2-4b59-a2d7-c468f9b8b5a6/94d294dd-af54-43f7-9e9b-15472c788437"
-					(reference "R34")
+					(reference "R35")
 					(unit 1)
 				)
@@
 		(dnp no)
 		(fields_autoplaced yes)
-		(property "Reference" "#PWR0341"
+		(property "Reference" "#PWR0345"
 			(at 182.88 111.76 0)
 			(effects
@@
 			(project "raywatch"
 				(path "/7b654ee8-2a53-4d39-8b7d-32c7bb3cb0ed/6e6a70ea-4db2-4b59-a2d7-c468f9b8b5a6/94d294dd-af54-43f7-9e9b-15472c788437"
-					(reference "#PWR0341")
+					(reference "#PWR0345")
 					(unit 1)
 				)
@@
 		(dnp no)
 		(fields_autoplaced yes)
-		(property "Reference" "U23"
+		(property "Reference" "U24"
 			(at 148.59 82.55 0)
 			(effects
@@
 			(project "raywatch"
 				(path "/7b654ee8-2a53-4d39-8b7d-32c7bb3cb0ed/6e6a70ea-4db2-4b59-a2d7-c468f9b8b5a6/94d294dd-af54-43f7-9e9b-15472c788437"
-					(reference "U23")
+					(reference "U24")
 					(unit 1)
 				)
@@
 		(dnp no)
 		(fields_autoplaced yes)
-		(property "Reference" "R33"
+		(property "Reference" "R34"
 			(at 175.26 100.3299 0)
 			(effects
@@
 			(project "raywatch"
 				(path "/7b654ee8-2a53-4d39-8b7d-32c7bb3cb0ed/6e6a70ea-4db2-4b59-a2d7-c468f9b8b5a6/94d294dd-af54-43f7-9e9b-15472c788437"
-					(reference "R33")
+					(reference "R34")
 					(unit 1)
 				)
@@
 		(dnp no)
 		(fields_autoplaced yes)
-		(property "Reference" "#PWR0337"
+		(property "Reference" "#PWR0341"
 			(at 96.52 116.84 0)
 			(effects
@@
 			(project "raywatch"
 				(path "/7b654ee8-2a53-4d39-8b7d-32c7bb3cb0ed/6e6a70ea-4db2-4b59-a2d7-c468f9b8b5a6/94d294dd-af54-43f7-9e9b-15472c788437"
-					(reference "#PWR0337")
+					(reference "#PWR0341")
 					(unit 1)
 				)
@@
 		(dnp no)
 		(fields_autoplaced yes)
-		(property "Reference" "#PWR0339"
+		(property "Reference" "#PWR0343"
 			(at 166.37 116.84 0)
 			(effects
@@
 			(project "raywatch"
 				(path "/7b654ee8-2a53-4d39-8b7d-32c7bb3cb0ed/6e6a70ea-4db2-4b59-a2d7-c468f9b8b5a6/94d294dd-af54-43f7-9e9b-15472c788437"
-					(reference "#PWR0339")
+					(reference "#PWR0343")
 					(unit 1)
 				)
@@
 		(dnp no)
 		(fields_autoplaced yes)
-		(property "Reference" "#PWR0338"
+		(property "Reference" "#PWR0342"
 			(at 127 106.68 0)
 			(effects
@@
 			(project "raywatch"
 				(path "/7b654ee8-2a53-4d39-8b7d-32c7bb3cb0ed/6e6a70ea-4db2-4b59-a2d7-c468f9b8b5a6/94d294dd-af54-43f7-9e9b-15472c788437"
-					(reference "#PWR0338")
-					(unit 1)
-				)
+					(reference "#PWR0342")
+					(unit 1)
+				)
