File: src/hardware/solar.kicad_sch (KiCad schematic)
At the start: 9 parts, among them U24 TPS61099YFFT

Commit message: Flattend hirachy
Parts:
- renumbered C66 to C82, C67 to C83, C68 to C84, R34 to R44, R35 to R45, U24 to U32
Changed lines of the file:
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@@
 		(dnp no)
 		(fields_autoplaced yes)
-		(property "Reference" "C67"
+		(property "Reference" "C83"
 			(at 186.69 100.3299 0)
 			(effects
@@
 		(instances
 			(project "raywatch"
-				(path "/7b654ee8-2a53-4d39-8b7d-32c7bb3cb0ed/6e6a70ea-4db2-4b59-a2d7-c468f9b8b5a6/94d294dd-af54-43f7-9e9b-15472c788437"
-					(reference "C67")
+				(path "/7b654ee8-2a53-4d39-8b7d-32c7bb3cb0ed/e90fef96-f7b6-4971-b8da-32a927b888f0"
+					(reference "C83")
 					(unit 1)
 				)
@@
 		(dnp no)
 		(fields_autoplaced yes)
-		(property "Reference" "#PWR0347"
+		(property "Reference" "#PWR0397"
 			(at 194.31 111.76 0)
 			(effects
@@
 		(instances
 			(project "raywatch"
-				(path "/7b654ee8-2a53-4d39-8b7d-32c7bb3cb0ed/6e6a70ea-4db2-4b59-a2d7-c468f9b8b5a6/94d294dd-af54-43f7-9e9b-15472c788437"
-					(reference "#PWR0347")
+				(path "/7b654ee8-2a53-4d39-8b7d-32c7bb3cb0ed/e90fef96-f7b6-4971-b8da-32a927b888f0"
+					(reference "#PWR0397")
 					(unit 1)
 				)
@@
 		(dnp no)
 		(fields_autoplaced yes)
-		(property "Reference" "#PWR0346"
+		(property "Reference" "#PWR0396"
 			(at 194.31 101.6 0)
 			(effects
@@
 		(instances
 			(project "raywatch"
-				(path "/7b654ee8-2a53-4d39-8b7d-32c7bb3cb0ed/6e6a70ea-4db2-4b59-a2d7-c468f9b8b5a6/94d294dd-af54-43f7-9e9b-15472c788437"
-					(reference "#PWR0346")
+				(path "/7b654ee8-2a53-4d39-8b7d-32c7bb3cb0ed/e90fef96-f7b6-4971-b8da-32a927b888f0"
+					(reference "#PWR0396")
 					(unit 1)
 				)
@@
 		(dnp no)
 		(fields_autoplaced yes)
-		(property "Reference" "#PWR0344"
+		(property "Reference" "#PWR0394"
 			(at 172.72 119.38 0)
 			(effects
@@
 		(instances
 			(project "raywatch"
-				(path "/7b654ee8-2a53-4d39-8b7d-32c7bb3cb0ed/6e6a70ea-4db2-4b59-a2d7-c468f9b8b5a6/94d294dd-af54-43f7-9e9b-15472c788437"
-					(reference "#PWR0344")
+				(path "/7b654ee8-2a53-4d39-8b7d-32c7bb3cb0ed/e90fef96-f7b6-4971-b8da-32a927b888f0"
+					(reference "#PWR0394")
 					(unit 1)
 				)
@@
 		(dnp no)
 		(fields_autoplaced yes)
-		(property "Reference" "C66"
+		(property "Reference" "C82"
 			(at 123.19 95.2499 0)
 			(effects
@@
 		(instances
 			(project "raywatch"
-				(path "/7b654ee8-2a53-4d39-8b7d-32c7bb3cb0ed/6e6a70ea-4db2-4b59-a2d7-c468f9b8b5a6/94d294dd-af54-43f7-9e9b-15472c788437"
-					(reference "C66")
+				(path "/7b654ee8-2a53-4d39-8b7d-32c7bb3cb0ed/e90fef96-f7b6-4971-b8da-32a927b888f0"
+					(reference "C82")
 					(unit 1)
 				)
@@
 		(dnp no)
 		(fields_autoplaced yes)
-		(property "Reference" "#PWR0340"
+		(property "Reference" "#PWR0390"
 			(at 95.885 99.06 0)
 			(effects
@@
 		(instances
 			(project "raywatch"
-				(path "/7b654ee8-2a53-4d39-8b7d-32c7bb3cb0ed/6e6a70ea-4db2-4b59-a2d7-c468f9b8b5a6/94d294dd-af54-43f7-9e9b-15472c788437"
-					(reference "#PWR0340")
+				(path "/7b654ee8-2a53-4d39-8b7d-32c7bb3cb0ed/e90fef96-f7b6-4971-b8da-32a927b888f0"
+					(reference "#PWR0390")
 					(unit 1)
 				)
@@
 		(dnp no)
 		(fields_autoplaced yes)
-		(property "Reference" "R35"
+		(property "Reference" "R45"
 			(at 175.26 107.9499 0)
 			(effects
@@
 		(instances
 			(project "raywatch"
-				(path "/7b654ee8-2a53-4d39-8b7d-32c7bb3cb0ed/6e6a70ea-4db2-4b59-a2d7-c468f9b8b5a6/94d294dd-af54-43f7-9e9b-15472c788437"
-					(reference "R35")
+				(path "/7b654ee8-2a53-4d39-8b7d-32c7bb3cb0ed/e90fef96-f7b6-4971-b8da-32a927b888f0"
+					(reference "R45")
 					(unit 1)
 				)
@@
 		(dnp no)
 		(fields_autoplaced yes)
-		(property "Reference" "#PWR0345"
+		(property "Reference" "#PWR0395"
 			(at 182.88 111.76 0)
 			(effects
@@
 		(instances
 			(project "raywatch"
-				(path "/7b654ee8-2a53-4d39-8b7d-32c7bb3cb0ed/6e6a70ea-4db2-4b59-a2d7-c468f9b8b5a6/94d294dd-af54-43f7-9e9b-15472c788437"
-					(reference "#PWR0345")
+				(path "/7b654ee8-2a53-4d39-8b7d-32c7bb3cb0ed/e90fef96-f7b6-4971-b8da-32a927b888f0"
+					(reference "#PWR0395")
 					(unit 1)
 				)
@@
 		(dnp no)
 		(fields_autoplaced yes)
-		(property "Reference" "U24"
+		(property "Reference" "U32"
 			(at 148.59 82.55 0)
 			(effects
@@
 		(instances
 			(project "raywatch"
-				(path "/7b654ee8-2a53-4d39-8b7d-32c7bb3cb0ed/6e6a70ea-4db2-4b59-a2d7-c468f9b8b5a6/94d294dd-af54-43f7-9e9b-15472c788437"
-					(reference "U24")
+				(path "/7b654ee8-2a53-4d39-8b7d-32c7bb3cb0ed/e90fef96-f7b6-4971-b8da-32a927b888f0"
+					(reference "U32")
 					(unit 1)
 				)
@@
 		(instances
 			(project "raywatch"
-				(path "/7b654ee8-2a53-4d39-8b7d-32c7bb3cb0ed/6e6a70ea-4db2-4b59-a2d7-c468f9b8b5a6/94d294dd-af54-43f7-9e9b-15472c788437"
+				(path "/7b654ee8-2a53-4d39-8b7d-32c7bb3cb0ed/e90fef96-f7b6-4971-b8da-32a927b888f0"
 					(reference "L9")
 					(unit 1)
@@
 		(dnp no)
 		(fields_autoplaced yes)
-		(property "Reference" "C68"
+		(property "Reference" "C84"
 			(at 198.12 100.3299 0)
 			(effects
@@
 		(instances
 			(project "raywatch"
-				(path "/7b654ee8-2a53-4d39-8b7d-32c7bb3cb0ed/6e6a70ea-4db2-4b59-a2d7-c468f9b8b5a6/94d294dd-af54-43f7-9e9b-15472c788437"
-					(reference "C68")
+				(path "/7b654ee8-2a53-4d39-8b7d-32c7bb3cb0ed/e90fef96-f7b6-4971-b8da-32a927b888f0"
+					(reference "C84")
 					(unit 1)
 				)
@@
 		(instances
 			(project "raywatch"
-				(path "/7b654ee8-2a53-4d39-8b7d-32c7bb3cb0ed/6e6a70ea-4db2-4b59-a2d7-c468f9b8b5a6/94d294dd-af54-43f7-9e9b-15472c788437"
+				(path "/7b654ee8-2a53-4d39-8b7d-32c7bb3cb0ed/e90fef96-f7b6-4971-b8da-32a927b888f0"
 					(reference "B2")
 					(unit 1)
@@
 		(dnp no)
 		(fields_autoplaced yes)
-		(property "Reference" "R34"
+		(property "Reference" "R44"
 			(at 175.26 100.3299 0)
 			(effects
@@
 		(instances
 			(project "raywatch"
-				(path "/7b654ee8-2a53-4d39-8b7d-32c7bb3cb0ed/6e6a70ea-4db2-4b59-a2d7-c468f9b8b5a6/94d294dd-af54-43f7-9e9b-15472c788437"
-					(reference "R34")
+				(path "/7b654ee8-2a53-4d39-8b7d-32c7bb3cb0ed/e90fef96-f7b6-4971-b8da-32a927b888f0"
+					(reference "R44")
 					(unit 1)
 				)
@@
 		(dnp no)
 		(fields_autoplaced yes)
-		(property "Reference" "#PWR0341"
+		(property "Reference" "#PWR0391"
 			(at 96.52 116.84 0)
 			(effects
@@
 		(instances
 			(project "raywatch"
-				(path "/7b654ee8-2a53-4d39-8b7d-32c7bb3cb0ed/6e6a70ea-4db2-4b59-a2d7-c468f9b8b5a6/94d294dd-af54-43f7-9e9b-15472c788437"
-					(reference "#PWR0341")
+				(path "/7b654ee8-2a53-4d39-8b7d-32c7bb3cb0ed/e90fef96-f7b6-4971-b8da-32a927b888f0"
+					(reference "#PWR0391")
 					(unit 1)
 				)
@@
 		(dnp no)
 		(fields_autoplaced yes)
-		(property "Reference" "#PWR0343"
+		(property "Reference" "#PWR0393"
 			(at 166.37 116.84 0)
 			(effects
@@
 		(instances
 			(project "raywatch"
-				(path "/7b654ee8-2a53-4d39-8b7d-32c7bb3cb0ed/6e6a70ea-4db2-4b59-a2d7-c468f9b8b5a6/94d294dd-af54-43f7-9e9b-15472c788437"
-					(reference "#PWR0343")
+				(path "/7b654ee8-2a53-4d39-8b7d-32c7bb3cb0ed/e90fef96-f7b6-4971-b8da-32a927b888f0"
+					(reference "#PWR0393")
 					(unit 1)
 				)
@@
 		(instances
 			(project "raywatch"
-				(path "/7b654ee8-2a53-4d39-8b7d-32c7bb3cb0ed/6e6a70ea-4db2-4b59-a2d7-c468f9b8b5a6/94d294dd-af54-43f7-9e9b-15472c788437"
+				(path "/7b654ee8-2a53-4d39-8b7d-32c7bb3cb0ed/e90fef96-f7b6-4971-b8da-32a927b888f0"
 					(reference "B1")
 					(unit 1)
@@
 		(dnp no)
 		(fields_autoplaced yes)
-		(property "Reference" "#PWR0342"
+		(property "Reference" "#PWR0392"
 			(at 127 106.68 0)
 			(effects
@@
 		(instances
 			(project "raywatch"
-				(path "/7b654ee8-2a53-4d39-8b7d-32c7bb3cb0ed/6e6a70ea-4db2-4b59-a2d7-c468f9b8b5a6/94d294dd-af54-43f7-9e9b-15472c788437"
-					(reference "#PWR0342")
-					(unit 1)
-				)
+				(path "/7b654ee8-2a53-4d39-8b7d-32c7bb3cb0ed/e90fef96-f7b6-4971-b8da-32a927b888f0"
+					(reference "#PWR0392")
+					(unit 1)
+				)

Commit message: Cleanup
Other:
- moved on the sheet: C83, C84
Changed lines of the file:
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@@
 	)
 	(junction
-		(at 182.88 97.79)
+		(at 185.42 97.79)
 		(diameter 0)
 		(color 0 0 0 0)
@@
 	)
 	(junction
-		(at 194.31 97.79)
+		(at 196.85 97.79)
 		(diameter 0)
 		(color 0 0 0 0)
@@
 	(wire
 		(pts
-			(xy 172.72 97.79) (xy 182.88 97.79)
+			(xy 172.72 97.79) (xy 185.42 97.79)
 		)
 		(stroke
@@
 	(wire
 		(pts
-			(xy 194.31 97.79) (xy 182.88 97.79)
+			(xy 185.42 97.79) (xy 196.85 97.79)
 		)
 		(stroke
@@
 	(symbol
 		(lib_id "Device:C")
-		(at 182.88 101.6 0)
+		(at 185.42 101.6 0)
 		(unit 1)
 		(exclude_from_sim no)
@@
 		(fields_autoplaced yes)
 		(property "Reference" "C83"
-			(at 186.69 100.3299 0)
+			(at 189.23 100.3299 0)
 			(effects
 				(font
@@
 		)
 		(property "Value" "10µF"
-			(at 186.69 102.8699 0)
+			(at 189.23 102.8699 0)
 			(effects
 				(font
@@
 		)
 		(property "Footprint" "Capacitor_SMD:C_0603_1608Metric"
-			(at 183.8452 105.41 0)
+			(at 186.3852 105.41 0)
 			(effects
 				(font
@@
 		)
 		(property "Datasheet" "~"
-			(at 182.88 101.6 0)
+			(at 185.42 101.6 0)
 			(effects
 				(font
@@
 		)
 		(property "Description" "Unpolarized capacitor"
-			(at 182.88 101.6 0)
+			(at 185.42 101.6 0)
 			(effects
 				(font
@@
 	(symbol
 		(lib_id "power:GND")
-		(at 194.31 105.41 0)
+		(at 196.85 105.41 0)
 		(unit 1)
 		(exclude_from_sim no)
@@
 		(fields_autoplaced yes)
 		(property "Reference" "#PWR0397"
-			(at 194.31 111.76 0)
+			(at 196.85 111.76 0)
 			(effects
 				(font
@@
 		)
 		(property "Value" "GND"
-			(at 194.31 110.49 0)
+			(at 196.85 110.49 0)
 			(effects
 				(font
@@
 		)
 		(property "Footprint" ""
-			(at 194.31 105.41 0)
+			(at 196.85 105.41 0)
 			(effects
 				(font
@@
 		)
 		(property "Datasheet" ""
-			(at 194.31 105.41 0)
+			(at 196.85 105.41 0)
 			(effects
 				(font
@@
 		)
 		(property "Description" "Power symbol creates a global label with name \"GND\" , ground"
-			(at 194.31 105.41 0)
+			(at 196.85 105.41 0)
 			(effects
 				(font
@@
 	(symbol
 		(lib_id "power:LINE")
-		(at 194.31 97.79 0)
+		(at 196.85 97.79 0)
 		(unit 1)
 		(exclude_from_sim no)
@@
 		(fields_autoplaced yes)
 		(property "Reference" "#PWR0396"
-			(at 194.31 101.6 0)
+			(at 196.85 101.6 0)
 			(effects
 				(font
@@
 		)
 		(property "Value" "VSOLAR"
-			(at 194.31 92.71 0)
+			(at 196.85 92.71 0)
 			(effects
 				(font
@@
 		)
 		(property "Footprint" ""
-			(at 194.31 97.79 0)
+			(at 196.85 97.79 0)
 			(effects
 				(font
@@
 		)
 		(property "Datasheet" ""
-			(at 194.31 97.79 0)
+			(at 196.85 97.79 0)
 			(effects
 				(font
@@
 		)
 		(property "Description" "Power symbol creates a global label with name \"LINE\""
-			(at 194.31 97.79 0)
+			(at 196.85 97.79 0)
 			(effects
 				(font
@@
 	(symbol
 		(lib_id "power:GND")
-		(at 182.88 105.41 0)
+		(at 185.42 105.41 0)
 		(unit 1)
 		(exclude_from_sim no)
@@
 		(fields_autoplaced yes)
 		(property "Reference" "#PWR0395"
-			(at 182.88 111.76 0)
+			(at 185.42 111.76 0)
 			(effects
 				(font
@@
 		)
 		(property "Value" "GND"
-			(at 182.88 110.49 0)
+			(at 185.42 110.49 0)
 			(effects
 				(font
@@
 		)
 		(property "Footprint" ""
-			(at 182.88 105.41 0)
+			(at 185.42 105.41 0)
 			(effects
 				(font
@@
 		)
 		(property "Datasheet" ""
-			(at 182.88 105.41 0)
+			(at 185.42 105.41 0)
 			(effects
 				(font
@@
 		)
 		(property "Description" "Power symbol creates a global label with name \"GND\" , ground"
-			(at 182.88 105.41 0)
+			(at 185.42 105.41 0)
 			(effects
 				(font
@@
 	(symbol
 		(lib_id "Device:C")
-		(at 194.31 101.6 0)
+		(at 196.85 101.6 0)
 		(unit 1)
 		(exclude_from_sim no)
@@
 		(fields_autoplaced yes)
 		(property "Reference" "C84"
-			(at 198.12 100.3299 0)
+			(at 200.66 100.3299 0)
 			(effects
 				(font
@@
 		)
 		(property "Value" "10µF"
-			(at 198.12 102.8699 0)
+			(at 200.66 102.8699 0)
 			(effects
 				(font
@@
 		)
 		(property "Footprint" "Capacitor_SMD:C_0603_1608Metric"
-			(at 195.2752 105.41 0)
+			(at 197.8152 105.41 0)
 			(effects
 				(font
@@
 		)
 		(property "Datasheet" "~"
-			(at 194.31 101.6 0)
+			(at 196.85 101.6 0)
 			(effects
 				(font
@@
 		)
 		(property "Description" "Unpolarized capacitor"
-			(at 194.31 101.6 0)
-			(effects
-				(font
+			(at 196.85 101.6 0)
+			(effects
+				(font

Commit message: Changed footprints from 0603 to 0402
Parts:
- C82, C83, C84: footprint Capacitor_SMD:C_0603_1608Metric -> Capacitor_SMD:C_0504_1310Metric
- R44, R45: footprint Resistor_SMD:R_0603_1608Metric -> Resistor_SMD:R_0402_1005Metric
Changed lines of the file:
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@@
 			)
 		)
-		(property "Footprint" "Capacitor_SMD:C_0603_1608Metric"
+		(property "Footprint" "Capacitor_SMD:C_0504_1310Metric"
 			(at 186.3852 105.41 0)
 			(effects
@@
 			)
 		)
-		(property "Footprint" "Capacitor_SMD:C_0603_1608Metric"
+		(property "Footprint" "Capacitor_SMD:C_0504_1310Metric"
 			(at 126.0348 100.33 0)
 			(effects
@@
 			)
 		)
-		(property "Footprint" "Resistor_SMD:R_0603_1608Metric"
+		(property "Footprint" "Resistor_SMD:R_0402_1005Metric"
 			(at 170.942 109.22 90)
 			(effects
@@
 			)
 		)
-		(property "Footprint" "Capacitor_SMD:C_0603_1608Metric"
+		(property "Footprint" "Capacitor_SMD:C_0504_1310Metric"
 			(at 197.8152 105.41 0)
 			(effects
@@
 			)
 		)
-		(property "Footprint" "Resistor_SMD:R_0603_1608Metric"
+		(property "Footprint" "Resistor_SMD:R_0402_1005Metric"
 			(at 170.942 101.6 90)
 			(effects

Commit message: Replaced global labels with pin headers
Parts:
- added J14: Conn_01x02_Pin, symbol Connector:Conn_01x02_Pin
Connections:
- net GND: now also J14.2 (Pin_2)
- net VSOLAR: now also J14.1 (Pin_1)
Changed lines of the file:
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@@
+	)
+	(symbol
+		(lib_id "power:LINE")
+		(at 185.42 74.93 270)
+		(unit 1)
+		(exclude_from_sim no)
+		(in_bom yes)
+		(on_board yes)
+		(dnp no)
+		(fields_autoplaced yes)
+		(property "Reference" "#PWR0436"
+			(at 181.61 74.93 0)
+			(effects
+				(font
+					(size 1.27 1.27)
+				)
+				(hide yes)
+			)
+		)
+		(property "Value" "VSOLAR"
+			(at 189.23 74.9299 90)
+			(effects
+				(font
+					(size 1.27 1.27)
+				)
+				(justify left)
+			)
+		)
+		(property "Footprint" ""
+			(at 185.42 74.93 0)
+			(effects
+				(font
+					(size 1.27 1.27)
+				)
+				(hide yes)
+			)
+		)
+		(property "Datasheet" ""
+			(at 185.42 74.93 0)
+			(effects
+				(font
+					(size 1.27 1.27)
+				)
+				(hide yes)
+			)
+		)
+		(property "Description" "Power symbol creates a global label with name \"LINE\""
+			(at 185.42 74.93 0)
+			(effects
+				(font
+					(size 1.27 1.27)
+				)
+				(hide yes)
+			)
+		)
+		(pin "1"
+		)
+		(instances
+			(project "raywatch"
+				(path "/7b654ee8-2a53-4d39-8b7d-32c7bb3cb0ed/e90fef96-f7b6-4971-b8da-32a927b888f0"
+					(reference "#PWR0436")
+					(unit 1)
+				)
+			)
+		)
 	)
 	(symbol
@@
 					(unit 1)
 				)
+			)
+		)
+	)
+	(symbol
+		(lib_id "power:GND")
+		(at 185.42 77.47 90)
+		(unit 1)
+		(exclude_from_sim no)
+		(in_bom yes)
+		(on_board yes)
+		(dnp no)
+		(fields_autoplaced yes)
+		(property "Reference" "#PWR0437"
+			(at 191.77 77.47 0)
+			(effects
+				(font
+					(size 1.27 1.27)
+				)
+				(hide yes)
+			)
+		)
+		(property "Value" "GND"
+			(at 189.23 77.4699 90)
+			(effects
+				(font
+					(size 1.27 1.27)
+				)
+				(justify right)
+			)
+		)
+		(property "Footprint" ""
+			(at 185.42 77.47 0)
+			(effects
+				(font
+					(size 1.27 1.27)
+				)
+				(hide yes)
+			)
+		)
+		(property "Datasheet" ""
+			(at 185.42 77.47 0)
+			(effects
+				(font
+					(size 1.27 1.27)
+				)
+				(hide yes)
+			)
+		)
+		(property "Description" "Power symbol creates a global label with name \"GND\" , ground"
+			(at 185.42 77.47 0)
+			(effects
+				(font
+					(size 1.27 1.27)
+				)
+				(hide yes)
+			)
+		)
+		(pin "1"
+		)
+		(instances
+			(project "raywatch"
+				(path "/7b654ee8-2a53-4d39-8b7d-32c7bb3cb0ed/e90fef96-f7b6-4971-b8da-32a927b888f0"
+					(reference "#PWR0437")
+					(unit 1)
+				)
+			)
+		)
+	)
+	(symbol
+		(lib_id "Connector:Conn_01x02_Pin")
+		(at 180.34 74.93 0)
+		(unit 1)
+		(exclude_from_sim no)
+		(in_bom yes)
+		(on_board yes)
+		(dnp no)
+		(fields_autoplaced yes)
+		(property "Reference" "J14"
+			(at 180.975 69.85 0)
+			(effects
+				(font
+					(size 1.27 1.27)
+				)
+			)
+		)
+		(property "Value" "Conn_01x02_Pin"
+			(at 180.975 72.39 0)
+			(effects
+				(font
+					(size 1.27 1.27)
+				)
+			)
+		)
+		(property "Footprint" ""
+			(at 180.34 74.93 0)
+			(effects
+				(font
+					(size 1.27 1.27)
+				)
+				(hide yes)
+			)
+		)
+		(property "Datasheet" "~"
+			(at 180.34 74.93 0)
+			(effects
+				(font
+					(size 1.27 1.27)
+				)
+				(hide yes)
+			)
+		)
+		(property "Description" "Generic connector, single row, 01x02, script generated"
+			(at 180.34 74.93 0)
+			(effects
+				(font
+					(size 1.27 1.27)
+				)
+				(hide yes)
+			)
+		)
+		(pin "1"
+		)
+		(pin "2"
+		)
+		(instances
+			(project "raywatch"
+				(path "/7b654ee8-2a53-4d39-8b7d-32c7bb3cb0ed/e90fef96-f7b6-4971-b8da-32a927b888f0"
+					(reference "J14")
+					(unit 1)
+				)

Commit message: Reannotated schematic
Parts:
- renumbered C82 to C77, C83 to C78, C84 to C79, J14 to J88, R44 to R38, R45 to R39, U32 to U33
Changed lines of the file:
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@@
 		(dnp no)
 		(fields_autoplaced yes)
-		(property "Reference" "C83"
+		(property "Reference" "C78"
 			(at 189.23 100.3299 0)
 			(effects
@@
 			(project "raywatch"
 				(path "/7b654ee8-2a53-4d39-8b7d-32c7bb3cb0ed/e90fef96-f7b6-4971-b8da-32a927b888f0"
-					(reference "C83")
+					(reference "C78")
 					(unit 1)
 				)
@@
 		(dnp no)
 		(fields_autoplaced yes)
-		(property "Reference" "#PWR0397"
+		(property "Reference" "#PWR0450"
 			(at 196.85 111.76 0)
 			(effects
@@
 			(project "raywatch"
 				(path "/7b654ee8-2a53-4d39-8b7d-32c7bb3cb0ed/e90fef96-f7b6-4971-b8da-32a927b888f0"
-					(reference "#PWR0397")
+					(reference "#PWR0450")
 					(unit 1)
 				)
@@
 		(dnp no)
 		(fields_autoplaced yes)
-		(property "Reference" "#PWR0396"
+		(property "Reference" "#PWR0449"
 			(at 196.85 101.6 0)
 			(effects
@@
 			(project "raywatch"
 				(path "/7b654ee8-2a53-4d39-8b7d-32c7bb3cb0ed/e90fef96-f7b6-4971-b8da-32a927b888f0"
-					(reference "#PWR0396")
+					(reference "#PWR0449")
 					(unit 1)
 				)
@@
 		(dnp no)
 		(fields_autoplaced yes)
-		(property "Reference" "#PWR0394"
+		(property "Reference" "#PWR0445"
 			(at 172.72 119.38 0)
 			(effects
@@
 			(project "raywatch"
 				(path "/7b654ee8-2a53-4d39-8b7d-32c7bb3cb0ed/e90fef96-f7b6-4971-b8da-32a927b888f0"
-					(reference "#PWR0394")
+					(reference "#PWR0445")
 					(unit 1)
 				)
@@
 		(dnp no)
 		(fields_autoplaced yes)
-		(property "Reference" "C82"
+		(property "Reference" "C77"
 			(at 123.19 95.2499 0)
 			(effects
@@
 			(project "raywatch"
 				(path "/7b654ee8-2a53-4d39-8b7d-32c7bb3cb0ed/e90fef96-f7b6-4971-b8da-32a927b888f0"
-					(reference "C82")
+					(reference "C77")
 					(unit 1)
 				)
@@
 		(dnp no)
 		(fields_autoplaced yes)
-		(property "Reference" "#PWR0436"
+		(property "Reference" "#PWR0446"
 			(at 181.61 74.93 0)
 			(effects
@@
 			(project "raywatch"
 				(path "/7b654ee8-2a53-4d39-8b7d-32c7bb3cb0ed/e90fef96-f7b6-4971-b8da-32a927b888f0"
-					(reference "#PWR0436")
+					(reference "#PWR0446")
 					(unit 1)
 				)
@@
 		(dnp no)
 		(fields_autoplaced yes)
-		(property "Reference" "#PWR0390"
+		(property "Reference" "#PWR0441"
 			(at 95.885 99.06 0)
 			(effects
@@
 			(project "raywatch"
 				(path "/7b654ee8-2a53-4d39-8b7d-32c7bb3cb0ed/e90fef96-f7b6-4971-b8da-32a927b888f0"
-					(reference "#PWR0390")
+					(reference "#PWR0441")
 					(unit 1)
 				)
@@
 		(dnp no)
 		(fields_autoplaced yes)
-		(property "Reference" "R45"
+		(property "Reference" "R39"
 			(at 175.26 107.9499 0)
 			(effects
@@
 			(project "raywatch"
 				(path "/7b654ee8-2a53-4d39-8b7d-32c7bb3cb0ed/e90fef96-f7b6-4971-b8da-32a927b888f0"
-					(reference "R45")
+					(reference "R39")
 					(unit 1)
 				)
@@
 		(dnp no)
 		(fields_autoplaced yes)
-		(property "Reference" "#PWR0395"
+		(property "Reference" "#PWR0448"
 			(at 185.42 111.76 0)
 			(effects
@@
 			(project "raywatch"
 				(path "/7b654ee8-2a53-4d39-8b7d-32c7bb3cb0ed/e90fef96-f7b6-4971-b8da-32a927b888f0"
-					(reference "#PWR0395")
+					(reference "#PWR0448")
 					(unit 1)
 				)
@@
 		(dnp no)
 		(fields_autoplaced yes)
-		(property "Reference" "U32"
+		(property "Reference" "U33"
 			(at 148.59 82.55 0)
 			(effects
@@
 			(project "raywatch"
 				(path "/7b654ee8-2a53-4d39-8b7d-32c7bb3cb0ed/e90fef96-f7b6-4971-b8da-32a927b888f0"
-					(reference "U32")
+					(reference "U33")
 					(unit 1)
 				)
@@
 		(dnp no)
 		(fields_autoplaced yes)
-		(property "Reference" "C84"
+		(property "Reference" "C79"
 			(at 200.66 100.3299 0)
 			(effects
@@
 			(project "raywatch"
 				(path "/7b654ee8-2a53-4d39-8b7d-32c7bb3cb0ed/e90fef96-f7b6-4971-b8da-32a927b888f0"
-					(reference "C84")
+					(reference "C79")
 					(unit 1)
 				)
@@
 		(dnp no)
 		(fields_autoplaced yes)
-		(property "Reference" "R44"
+		(property "Reference" "R38"
 			(at 175.26 100.3299 0)
 			(effects
@@
 			(project "raywatch"
 				(path "/7b654ee8-2a53-4d39-8b7d-32c7bb3cb0ed/e90fef96-f7b6-4971-b8da-32a927b888f0"
-					(reference "R44")
+					(reference "R38")
 					(unit 1)
 				)
@@
 		(dnp no)
 		(fields_autoplaced yes)
-		(property "Reference" "#PWR0437"
+		(property "Reference" "#PWR0447"
 			(at 191.77 77.47 0)
 			(effects
@@
 			(project "raywatch"
 				(path "/7b654ee8-2a53-4d39-8b7d-32c7bb3cb0ed/e90fef96-f7b6-4971-b8da-32a927b888f0"
-					(reference "#PWR0437")
+					(reference "#PWR0447")
 					(unit 1)
 				)
@@
 		(dnp no)
 		(fields_autoplaced yes)
-		(property "Reference" "J14"
+		(property "Reference" "J88"
 			(at 180.975 69.85 0)
 			(effects
@@
 			(project "raywatch"
 				(path "/7b654ee8-2a53-4d39-8b7d-32c7bb3cb0ed/e90fef96-f7b6-4971-b8da-32a927b888f0"
-					(reference "J14")
+					(reference "J88")
 					(unit 1)
 				)
@@
 		(dnp no)
 		(fields_autoplaced yes)
-		(property "Reference" "#PWR0391"
+		(property "Reference" "#PWR0442"
 			(at 96.52 116.84 0)
 			(effects
@@
 			(project "raywatch"
 				(path "/7b654ee8-2a53-4d39-8b7d-32c7bb3cb0ed/e90fef96-f7b6-4971-b8da-32a927b888f0"
-					(reference "#PWR0391")
+					(reference "#PWR0442")
 					(unit 1)
 				)
@@
 		(dnp no)
 		(fields_autoplaced yes)
-		(property "Reference" "#PWR0393"
+		(property "Reference" "#PWR0444"
 			(at 166.37 116.84 0)
 			(effects
@@
 			(project "raywatch"
 				(path "/7b654ee8-2a53-4d39-8b7d-32c7bb3cb0ed/e90fef96-f7b6-4971-b8da-32a927b888f0"
-					(reference "#PWR0393")
+					(reference "#PWR0444")
 					(unit 1)
 				)
@@
 		(dnp no)
 		(fields_autoplaced yes)
-		(property "Reference" "#PWR0392"
+		(property "Reference" "#PWR0443"
 			(at 127 106.68 0)
 			(effects
@@
 			(project "raywatch"
 				(path "/7b654ee8-2a53-4d39-8b7d-32c7bb3cb0ed/e90fef96-f7b6-4971-b8da-32a927b888f0"
-					(reference "#PWR0392")
-					(unit 1)
-				)
+					(reference "#PWR0443")
+					(unit 1)
+				)

Commit message: Assigned pin header footprints
Parts:
- J88: footprint (none) -> Connector_PinHeader_2.54mm:PinHeader_1x02_P2.54mm_Horizontal
Changed lines of the file:
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@@
 			)
 		)
-		(property "Footprint" ""
+		(property "Footprint" "Connector_PinHeader_2.54mm:PinHeader_1x02_P2.54mm_Horizontal"
 			(at 180.34 74.93 0)
 			(effects
