File: src/hardware/vibration_motor.kicad_sch (KiCad schematic)
At the start: 3 parts, among them U1 DRV2605LYZFR

Commit message: Replaced schematics, 3d models and footprints. Added vibration motor.
Parts:
- removed U1: DRV2605LYZFR, YZF0009ADAD, symbol DRV2605LYZFR:DRV2605LYZFR
- added LS?: HD-LA1307-SM, HD-LA1307-SM:XDCR_HD-LA1307-SM, symbol HD-LA1307-SM:HD-LA1307-SM
- added U?: DRV2605LYZFR, YZF0009ADAD, symbol DRV2605LYZFR:DRV2605LYZFR
Connections:
- net GND: now also U?.B1 (IN_TRIG), U?.B3 (GND)
- net SCL: now also U?.C1 (SCL)
- net SDA: now also U?.B2 (SDA)
- net VIBEN: now also U?.A1 (EN)
- net VBAT: now reaches C19.1
- net VBAT: now also U?.C2 (VDD)
- net at C18.1: now also U?.A2 (REG)
- new net: LS?.N1, LS?.N2, U?.C3 (OUT-)
- new net: LS?.P1, LS?.P2, U?.A3 (OUT+)
Other:
- note added: "90mA Max"

Commit message: Added LoRa
Changed lines of the file:
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@@
 		(fields_autoplaced yes)
 		(property "Reference" "C18"
-			(at 128.27 113.0299 0)
+			(at 120.65 113.0299 0)
 			(effects
 				(font
 					(size 1.27 1.27)
 				)
-				(justify left)
+				(justify right)
 			)
 		)
 		(property "Value" "1µF"
-			(at 128.27 115.5699 0)
+			(at 120.65 115.5699 0)
 			(effects
 				(font
 					(size 1.27 1.27)
 				)
-				(justify left)
+				(justify right)
 			)
 		)

Commit message: Selected GPIO
Changed lines of the file:
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@@
 		)
 		(property "Value" "GND"
-			(at 170.18 85.09 0)
+			(at 172.72 88.8999 0)
 			(effects
 				(font
 					(size 1.27 1.27)
 				)
+				(justify right)
 			)
 		)

Commit message: Changed power symboles
Connections:
- net VBAT renamed VSYS
Changed lines of the file:
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@@
 			)
 		)
-		(property "Value" "VBAT"
+		(property "Value" "VSYS"
 			(at 177.8 105.41 0)
 			(effects

Commit message: Added Accelerometer Clock; Cleanup & Fixes
Other:
- note added: "I²C: 1011010"
- moved on the sheet: C18, C19, LS?

Commit message: Cleanup & Fixes; Added footprints; Removed Light sensors
Parts:
- C57: renamed from C18; footprint (none) -> Capacitor_SMD:C_0603_1608Metric
- C58: renamed from C19; footprint (none) -> Capacitor_SMD:C_0603_1608Metric
- LS1: renamed from LS?; footprint HD-LA1307-SM:XDCR_HD-LA1307-SM -> Project:XDCR_HD-LA1307-SM
- U19: renamed from U?; footprint YZF0009ADAD -> Project:YZF0009ADAD
Changed lines of the file:
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@@
 		(dnp no)
 		(fields_autoplaced yes)
-		(property "Reference" "C19"
+		(property "Reference" "C58"
 			(at 171.45 113.0299 0)
 			(effects
@@
 			)
 		)
-		(property "Footprint" ""
+		(property "Footprint" "Capacitor_SMD:C_0603_1608Metric"
 			(at 168.6052 118.11 0)
 			(effects
@@
 			(project "raywatch"
 				(path "/7b654ee8-2a53-4d39-8b7d-32c7bb3cb0ed/34ecb33f-48ad-4657-abe2-b4caffc19e6d"
-					(reference "C19")
+					(reference "C58")
 					(unit 1)
 				)
@@
 		(dnp no)
 		(fields_autoplaced yes)
-		(property "Reference" "#PWR0312"
+		(property "Reference" "#PWR0319"
 			(at 129.54 124.46 0)
 			(effects
@@
 			(project "raywatch"
 				(path "/7b654ee8-2a53-4d39-8b7d-32c7bb3cb0ed/34ecb33f-48ad-4657-abe2-b4caffc19e6d"
-					(reference "#PWR0312")
+					(reference "#PWR0319")
 					(unit 1)
 				)
@@
 		(dnp no)
 		(fields_autoplaced yes)
-		(property "Reference" "#PWR0314"
+		(property "Reference" "#PWR0320"
 			(at 167.64 83.82 0)
 			(effects
@@
 			(project "raywatch"
 				(path "/7b654ee8-2a53-4d39-8b7d-32c7bb3cb0ed/34ecb33f-48ad-4657-abe2-b4caffc19e6d"
-					(reference "#PWR0314")
+					(reference "#PWR0320")
 					(unit 1)
 				)
@@
 		(dnp no)
 		(fields_autoplaced yes)
-		(property "Reference" "#PWR0313"
+		(property "Reference" "#PWR0321"
 			(at 167.64 114.3 0)
 			(effects
@@
 			(project "raywatch"
 				(path "/7b654ee8-2a53-4d39-8b7d-32c7bb3cb0ed/34ecb33f-48ad-4657-abe2-b4caffc19e6d"
-					(reference "#PWR0313")
+					(reference "#PWR0321")
 					(unit 1)
 				)
@@
 		(dnp no)
 		(fields_autoplaced yes)
-		(property "Reference" "#PWR0315"
+		(property "Reference" "#PWR0318"
 			(at 129.54 83.82 0)
 			(effects
@@
 		)
 		(property "Value" "GND"
-			(at 129.54 85.09 0)
-			(effects
-				(font
-					(size 1.27 1.27)
-				)
+			(at 127 88.8999 0)
+			(effects
+				(font
+					(size 1.27 1.27)
+				)
+				(justify left)
 			)
 		)
@@
 			(project "raywatch"
 				(path "/7b654ee8-2a53-4d39-8b7d-32c7bb3cb0ed/34ecb33f-48ad-4657-abe2-b4caffc19e6d"
-					(reference "#PWR0315")
+					(reference "#PWR0318")
 					(unit 1)
 				)
@@
 		(dnp no)
 		(fields_autoplaced yes)
-		(property "Reference" "LS?"
+		(property "Reference" "LS1"
 			(at 114.3 97.7899 0)
 			(effects
@@
 			)
 		)
-		(property "Footprint" "HD-LA1307-SM:XDCR_HD-LA1307-SM"
+		(property "Footprint" "Project:XDCR_HD-LA1307-SM"
 			(at 107.95 99.06 0)
 			(effects
@@
 			(project "raywatch"
 				(path "/7b654ee8-2a53-4d39-8b7d-32c7bb3cb0ed/34ecb33f-48ad-4657-abe2-b4caffc19e6d"
-					(reference "LS?")
+					(reference "LS1")
 					(unit 1)
 				)
@@
 		(dnp no)
 		(fields_autoplaced yes)
-		(property "Reference" "#PWR0311"
+		(property "Reference" "#PWR0322"
 			(at 167.64 124.46 0)
 			(effects
@@
 			(project "raywatch"
 				(path "/7b654ee8-2a53-4d39-8b7d-32c7bb3cb0ed/34ecb33f-48ad-4657-abe2-b4caffc19e6d"
-					(reference "#PWR0311")
+					(reference "#PWR0322")
 					(unit 1)
 				)
@@
 		(dnp no)
 		(fields_autoplaced yes)
-		(property "Reference" "U?"
+		(property "Reference" "U19"
 			(at 148.59 80.01 0)
 			(effects
@@
 			)
 		)
-		(property "Footprint" "YZF0009ADAD"
+		(property "Footprint" "Project:YZF0009ADAD"
 			(at 149.86 100.33 0)
 			(effects
@@
 			(project "raywatch"
 				(path "/7b654ee8-2a53-4d39-8b7d-32c7bb3cb0ed/34ecb33f-48ad-4657-abe2-b4caffc19e6d"
-					(reference "U?")
+					(reference "U19")
 					(unit 1)
 				)
@@
 		(dnp no)
 		(fields_autoplaced yes)
-		(property "Reference" "C18"
+		(property "Reference" "C57"
 			(at 125.73 113.0299 0)
 			(effects
@@
 			)
 		)
-		(property "Footprint" ""
+		(property "Footprint" "Capacitor_SMD:C_0603_1608Metric"
 			(at 130.5052 118.11 0)
 			(effects
@@
 			(project "raywatch"
 				(path "/7b654ee8-2a53-4d39-8b7d-32c7bb3cb0ed/34ecb33f-48ad-4657-abe2-b4caffc19e6d"
-					(reference "C18")
-					(unit 1)
-				)
+					(reference "C57")
+					(unit 1)
+				)

Commit message: Cleanup & Fixes; Changed GPIO; Added Camera; Added Microphone
Parts:
- renumbered C57 to C55, C58 to C56
Changed lines of the file:
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@@
 		(dnp no)
 		(fields_autoplaced yes)
-		(property "Reference" "C58"
+		(property "Reference" "C56"
 			(at 171.45 113.0299 0)
 			(effects
@@
 			(project "raywatch"
 				(path "/7b654ee8-2a53-4d39-8b7d-32c7bb3cb0ed/34ecb33f-48ad-4657-abe2-b4caffc19e6d"
-					(reference "C58")
+					(reference "C56")
 					(unit 1)
 				)
@@
 		(dnp no)
 		(fields_autoplaced yes)
-		(property "Reference" "#PWR0319"
+		(property "Reference" "#PWR0315"
 			(at 129.54 124.46 0)
 			(effects
@@
 			(project "raywatch"
 				(path "/7b654ee8-2a53-4d39-8b7d-32c7bb3cb0ed/34ecb33f-48ad-4657-abe2-b4caffc19e6d"
-					(reference "#PWR0319")
+					(reference "#PWR0315")
 					(unit 1)
 				)
@@
 		(dnp no)
 		(fields_autoplaced yes)
-		(property "Reference" "#PWR0320"
+		(property "Reference" "#PWR0316"
 			(at 167.64 83.82 0)
 			(effects
@@
 			(project "raywatch"
 				(path "/7b654ee8-2a53-4d39-8b7d-32c7bb3cb0ed/34ecb33f-48ad-4657-abe2-b4caffc19e6d"
-					(reference "#PWR0320")
+					(reference "#PWR0316")
 					(unit 1)
 				)
@@
 		(dnp no)
 		(fields_autoplaced yes)
-		(property "Reference" "#PWR0321"
+		(property "Reference" "#PWR0317"
 			(at 167.64 114.3 0)
 			(effects
@@
 			(project "raywatch"
 				(path "/7b654ee8-2a53-4d39-8b7d-32c7bb3cb0ed/34ecb33f-48ad-4657-abe2-b4caffc19e6d"
-					(reference "#PWR0321")
+					(reference "#PWR0317")
 					(unit 1)
 				)
@@
 		(dnp no)
 		(fields_autoplaced yes)
-		(property "Reference" "#PWR0318"
+		(property "Reference" "#PWR0314"
 			(at 129.54 83.82 0)
 			(effects
@@
 			(project "raywatch"
 				(path "/7b654ee8-2a53-4d39-8b7d-32c7bb3cb0ed/34ecb33f-48ad-4657-abe2-b4caffc19e6d"
-					(reference "#PWR0318")
+					(reference "#PWR0314")
 					(unit 1)
 				)
@@
 		(dnp no)
 		(fields_autoplaced yes)
-		(property "Reference" "#PWR0322"
+		(property "Reference" "#PWR0318"
 			(at 167.64 124.46 0)
 			(effects
@@
 			(project "raywatch"
 				(path "/7b654ee8-2a53-4d39-8b7d-32c7bb3cb0ed/34ecb33f-48ad-4657-abe2-b4caffc19e6d"
-					(reference "#PWR0322")
+					(reference "#PWR0318")
 					(unit 1)
 				)
@@
 		(dnp no)
 		(fields_autoplaced yes)
-		(property "Reference" "C57"
+		(property "Reference" "C55"
 			(at 125.73 113.0299 0)
 			(effects
@@
 			(project "raywatch"
 				(path "/7b654ee8-2a53-4d39-8b7d-32c7bb3cb0ed/34ecb33f-48ad-4657-abe2-b4caffc19e6d"
-					(reference "C57")
-					(unit 1)
-				)
+					(reference "C55")
+					(unit 1)
+				)

Commit message: Add Light Sensor and Proximity & Gesture Sensor; Changed GPIO
Parts:
- renumbered U19 to U20
Changed lines of the file:
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@@
 		(dnp no)
 		(fields_autoplaced yes)
-		(property "Reference" "#PWR0315"
+		(property "Reference" "#PWR0319"
 			(at 129.54 124.46 0)
 			(effects
@@
 			(project "raywatch"
 				(path "/7b654ee8-2a53-4d39-8b7d-32c7bb3cb0ed/34ecb33f-48ad-4657-abe2-b4caffc19e6d"
-					(reference "#PWR0315")
+					(reference "#PWR0319")
 					(unit 1)
 				)
@@
 		(dnp no)
 		(fields_autoplaced yes)
-		(property "Reference" "#PWR0316"
+		(property "Reference" "#PWR0320"
 			(at 167.64 83.82 0)
 			(effects
@@
 			(project "raywatch"
 				(path "/7b654ee8-2a53-4d39-8b7d-32c7bb3cb0ed/34ecb33f-48ad-4657-abe2-b4caffc19e6d"
-					(reference "#PWR0316")
+					(reference "#PWR0320")
 					(unit 1)
 				)
@@
 		(dnp no)
 		(fields_autoplaced yes)
-		(property "Reference" "#PWR0317"
+		(property "Reference" "#PWR0321"
 			(at 167.64 114.3 0)
 			(effects
@@
 			(project "raywatch"
 				(path "/7b654ee8-2a53-4d39-8b7d-32c7bb3cb0ed/34ecb33f-48ad-4657-abe2-b4caffc19e6d"
-					(reference "#PWR0317")
+					(reference "#PWR0321")
 					(unit 1)
 				)
@@
 		(dnp no)
 		(fields_autoplaced yes)
-		(property "Reference" "#PWR0314"
+		(property "Reference" "#PWR0318"
 			(at 129.54 83.82 0)
 			(effects
@@
 			(project "raywatch"
 				(path "/7b654ee8-2a53-4d39-8b7d-32c7bb3cb0ed/34ecb33f-48ad-4657-abe2-b4caffc19e6d"
-					(reference "#PWR0314")
+					(reference "#PWR0318")
 					(unit 1)
 				)
@@
 		(dnp no)
 		(fields_autoplaced yes)
-		(property "Reference" "#PWR0318"
+		(property "Reference" "#PWR0322"
 			(at 167.64 124.46 0)
 			(effects
@@
 			(project "raywatch"
 				(path "/7b654ee8-2a53-4d39-8b7d-32c7bb3cb0ed/34ecb33f-48ad-4657-abe2-b4caffc19e6d"
-					(reference "#PWR0318")
+					(reference "#PWR0322")
 					(unit 1)
 				)
@@
 		(dnp no)
 		(fields_autoplaced yes)
-		(property "Reference" "U19"
+		(property "Reference" "U20"
 			(at 148.59 80.01 0)
 			(effects
@@
 			(project "raywatch"
 				(path "/7b654ee8-2a53-4d39-8b7d-32c7bb3cb0ed/34ecb33f-48ad-4657-abe2-b4caffc19e6d"
-					(reference "U19")
-					(unit 1)
-				)
+					(reference "U20")
+					(unit 1)
+				)
