File: src/hardware/vibration_motor.kicad_sch (KiCad schematic)
At the start: 4 parts, among them U20 DRV2605LYZFR

Commit message: Changed footprints from 0603 to 0402
Parts:
- C55, C56: footprint Capacitor_SMD:C_0603_1608Metric -> Capacitor_SMD:C_0504_1310Metric
Changed lines of the file:
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@@
 			)
 		)
-		(property "Footprint" "Capacitor_SMD:C_0603_1608Metric"
+		(property "Footprint" "Capacitor_SMD:C_0504_1310Metric"
 			(at 168.6052 118.11 0)
 			(effects
@@
 			)
 		)
-		(property "Footprint" "Capacitor_SMD:C_0603_1608Metric"
+		(property "Footprint" "Capacitor_SMD:C_0504_1310Metric"
 			(at 130.5052 118.11 0)
 			(effects

Commit message: Replaced global labels with pin headers
Parts:
- added J29: Conn_01x01_Pin, symbol Connector:Conn_01x01_Pin
- added J37, J39: Conn_01x02_Pin, symbol Connector:Conn_01x02_Pin
- added TP2: TestPoint_2Pole, symbol Connector:TestPoint_2Pole
Connections:
- net GND: now also J37.2 (Pin_2)
- net SCL: now also J39.1 (Pin_1)
- net SDA: now also J39.2 (Pin_2)
- net VIBEN: now also J29.1 (Pin_1)
- net VSYS: now also J37.1 (Pin_1)
- net at LS1.N1, LS1.N2, U20.C3 (OUT-): now also TP2.1
- net at LS1.P1, LS1.P2, U20.A3 (OUT+): now also TP2.2

Commit message: Reannotated schematic
Parts:
- renumbered C55 to C49, C56 to C50, J37 to J61, J29 to J62, J39 to J63, TP2 to TP1
Changed lines of the file:
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@@
 		(dnp no)
 		(fields_autoplaced yes)
-		(property "Reference" "C56"
+		(property "Reference" "C50"
 			(at 171.45 113.0299 0)
 			(effects
@@
 			(project "raywatch"
 				(path "/7b654ee8-2a53-4d39-8b7d-32c7bb3cb0ed/34ecb33f-48ad-4657-abe2-b4caffc19e6d"
-					(reference "C56")
+					(reference "C50")
 					(unit 1)
 				)
@@
 		(dnp no)
 		(fields_autoplaced yes)
-		(property "Reference" "#PWR0319"
+		(property "Reference" "#PWR0336"
 			(at 129.54 124.46 0)
 			(effects
@@
 			(project "raywatch"
 				(path "/7b654ee8-2a53-4d39-8b7d-32c7bb3cb0ed/34ecb33f-48ad-4657-abe2-b4caffc19e6d"
-					(reference "#PWR0319")
+					(reference "#PWR0336")
 					(unit 1)
 				)
@@
 		(dnp no)
 		(fields_autoplaced yes)
-		(property "Reference" "#PWR0472"
+		(property "Reference" "#PWR0333"
 			(at 95.25 46.99 0)
 			(effects
@@
 			(project "raywatch"
 				(path "/7b654ee8-2a53-4d39-8b7d-32c7bb3cb0ed/34ecb33f-48ad-4657-abe2-b4caffc19e6d"
-					(reference "#PWR0472")
+					(reference "#PWR0333")
 					(unit 1)
 				)
@@
 		(dnp no)
 		(fields_autoplaced yes)
-		(property "Reference" "#PWR0320"
+		(property "Reference" "#PWR0337"
 			(at 167.64 83.82 0)
 			(effects
@@
 			(project "raywatch"
 				(path "/7b654ee8-2a53-4d39-8b7d-32c7bb3cb0ed/34ecb33f-48ad-4657-abe2-b4caffc19e6d"
-					(reference "#PWR0320")
+					(reference "#PWR0337")
 					(unit 1)
 				)
@@
 		(dnp no)
 		(fields_autoplaced yes)
-		(property "Reference" "#PWR0321"
+		(property "Reference" "#PWR0338"
 			(at 167.64 114.3 0)
 			(effects
@@
 			(project "raywatch"
 				(path "/7b654ee8-2a53-4d39-8b7d-32c7bb3cb0ed/34ecb33f-48ad-4657-abe2-b4caffc19e6d"
-					(reference "#PWR0321")
+					(reference "#PWR0338")
 					(unit 1)
 				)
@@
 		(dnp no)
 		(fields_autoplaced yes)
-		(property "Reference" "J39"
+		(property "Reference" "J63"
 			(at 92.71 68.5799 0)
 			(effects
@@
 			(project "raywatch"
 				(path "/7b654ee8-2a53-4d39-8b7d-32c7bb3cb0ed/34ecb33f-48ad-4657-abe2-b4caffc19e6d"
-					(reference "J39")
+					(reference "J63")
 					(unit 1)
 				)
@@
 		(dnp no)
 		(fields_autoplaced yes)
-		(property "Reference" "TP2"
+		(property "Reference" "TP1"
 			(at 90.17 97.7899 90)
 			(effects
@@
 			(project "raywatch"
 				(path "/7b654ee8-2a53-4d39-8b7d-32c7bb3cb0ed/34ecb33f-48ad-4657-abe2-b4caffc19e6d"
-					(reference "TP2")
+					(reference "TP1")
 					(unit 1)
 				)
@@
 		(dnp no)
 		(fields_autoplaced yes)
-		(property "Reference" "J29"
+		(property "Reference" "J62"
 			(at 92.71 57.1499 0)
 			(effects
@@
 			(project "raywatch"
 				(path "/7b654ee8-2a53-4d39-8b7d-32c7bb3cb0ed/34ecb33f-48ad-4657-abe2-b4caffc19e6d"
-					(reference "J29")
+					(reference "J62")
 					(unit 1)
 				)
@@
 		(dnp no)
 		(fields_autoplaced yes)
-		(property "Reference" "#PWR0318"
+		(property "Reference" "#PWR0335"
 			(at 129.54 83.82 0)
 			(effects
@@
 			(project "raywatch"
 				(path "/7b654ee8-2a53-4d39-8b7d-32c7bb3cb0ed/34ecb33f-48ad-4657-abe2-b4caffc19e6d"
-					(reference "#PWR0318")
+					(reference "#PWR0335")
 					(unit 1)
 				)
@@
 		(dnp no)
 		(fields_autoplaced yes)
-		(property "Reference" "J37"
+		(property "Reference" "J61"
 			(at 92.71 46.9899 0)
 			(effects
@@
 			(project "raywatch"
 				(path "/7b654ee8-2a53-4d39-8b7d-32c7bb3cb0ed/34ecb33f-48ad-4657-abe2-b4caffc19e6d"
-					(reference "J37")
+					(reference "J61")
 					(unit 1)
 				)
@@
 		(dnp no)
 		(fields_autoplaced yes)
-		(property "Reference" "#PWR0322"
+		(property "Reference" "#PWR0339"
 			(at 167.64 124.46 0)
 			(effects
@@
 			(project "raywatch"
 				(path "/7b654ee8-2a53-4d39-8b7d-32c7bb3cb0ed/34ecb33f-48ad-4657-abe2-b4caffc19e6d"
-					(reference "#PWR0322")
+					(reference "#PWR0339")
 					(unit 1)
 				)
@@
 		(dnp no)
 		(fields_autoplaced yes)
-		(property "Reference" "C55"
+		(property "Reference" "C49"
 			(at 125.73 113.0299 0)
 			(effects
@@
 			(project "raywatch"
 				(path "/7b654ee8-2a53-4d39-8b7d-32c7bb3cb0ed/34ecb33f-48ad-4657-abe2-b4caffc19e6d"
-					(reference "C55")
+					(reference "C49")
 					(unit 1)
 				)
@@
 		(dnp no)
 		(fields_autoplaced yes)
-		(property "Reference" "#PWR0473"
+		(property "Reference" "#PWR0334"
 			(at 105.41 49.53 0)
 			(effects
@@
 			(project "raywatch"
 				(path "/7b654ee8-2a53-4d39-8b7d-32c7bb3cb0ed/34ecb33f-48ad-4657-abe2-b4caffc19e6d"
-					(reference "#PWR0473")
-					(unit 1)
-				)
+					(reference "#PWR0334")
+					(unit 1)
+				)

Commit message: Assigned pin header footprints
Parts:
- J61, J63: footprint (none) -> Connector_PinHeader_2.54mm:PinHeader_1x02_P2.54mm_Horizontal
- J62: footprint (none) -> Connector_PinHeader_2.54mm:PinHeader_1x01_P2.54mm_Horizontal
- TP1: footprint (none) -> TestPoint:TestPoint_2Pads_Pitch2.54mm_Drill0.8mm
Changed lines of the file:
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@@
 			)
 		)
-		(property "Footprint" ""
+		(property "Footprint" "Connector_PinHeader_2.54mm:PinHeader_1x02_P2.54mm_Horizontal"
 			(at 93.98 68.58 0)
 			(effects
@@
 			)
 		)
-		(property "Footprint" ""
+		(property "Footprint" "TestPoint:TestPoint_2Pads_Pitch2.54mm_Drill0.8mm"
 			(at 92.71 99.06 0)
 			(effects
@@
 			)
 		)
-		(property "Footprint" ""
+		(property "Footprint" "Connector_PinHeader_2.54mm:PinHeader_1x01_P2.54mm_Horizontal"
 			(at 93.98 58.42 0)
 			(effects
@@
 			)
 		)
-		(property "Footprint" ""
+		(property "Footprint" "Connector_PinHeader_2.54mm:PinHeader_1x02_P2.54mm_Horizontal"
 			(at 93.98 46.99 0)
 			(effects

Commit message: Reannotate
Parts:
- renumbered U20 to U19
Changed lines of the file:
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@@
 		(dnp no)
 		(fields_autoplaced yes)
-		(property "Reference" "#PWR0336"
+		(property "Reference" "#PWR0337"
 			(at 129.54 124.46 0)
 			(effects
@@
 			(project "raywatch"
 				(path "/7b654ee8-2a53-4d39-8b7d-32c7bb3cb0ed/34ecb33f-48ad-4657-abe2-b4caffc19e6d"
-					(reference "#PWR0336")
+					(reference "#PWR0337")
 					(unit 1)
 				)
@@
 		(dnp no)
 		(fields_autoplaced yes)
-		(property "Reference" "#PWR0333"
+		(property "Reference" "#PWR0334"
 			(at 95.25 46.99 0)
 			(effects
@@
 			(project "raywatch"
 				(path "/7b654ee8-2a53-4d39-8b7d-32c7bb3cb0ed/34ecb33f-48ad-4657-abe2-b4caffc19e6d"
-					(reference "#PWR0333")
+					(reference "#PWR0334")
 					(unit 1)
 				)
@@
 		(dnp no)
 		(fields_autoplaced yes)
-		(property "Reference" "#PWR0337"
+		(property "Reference" "#PWR0338"
 			(at 167.64 83.82 0)
 			(effects
@@
 			(project "raywatch"
 				(path "/7b654ee8-2a53-4d39-8b7d-32c7bb3cb0ed/34ecb33f-48ad-4657-abe2-b4caffc19e6d"
-					(reference "#PWR0337")
+					(reference "#PWR0338")
 					(unit 1)
 				)
@@
 		(dnp no)
 		(fields_autoplaced yes)
-		(property "Reference" "#PWR0338"
+		(property "Reference" "#PWR0339"
 			(at 167.64 114.3 0)
 			(effects
@@
 			(project "raywatch"
 				(path "/7b654ee8-2a53-4d39-8b7d-32c7bb3cb0ed/34ecb33f-48ad-4657-abe2-b4caffc19e6d"
-					(reference "#PWR0338")
+					(reference "#PWR0339")
 					(unit 1)
 				)
@@
 		(dnp no)
 		(fields_autoplaced yes)
-		(property "Reference" "#PWR0335"
+		(property "Reference" "#PWR0336"
 			(at 129.54 83.82 0)
 			(effects
@@
 			(project "raywatch"
 				(path "/7b654ee8-2a53-4d39-8b7d-32c7bb3cb0ed/34ecb33f-48ad-4657-abe2-b4caffc19e6d"
-					(reference "#PWR0335")
+					(reference "#PWR0336")
 					(unit 1)
 				)
@@
 		(dnp no)
 		(fields_autoplaced yes)
-		(property "Reference" "#PWR0339"
+		(property "Reference" "#PWR0340"
 			(at 167.64 124.46 0)
 			(effects
@@
 			(project "raywatch"
 				(path "/7b654ee8-2a53-4d39-8b7d-32c7bb3cb0ed/34ecb33f-48ad-4657-abe2-b4caffc19e6d"
-					(reference "#PWR0339")
+					(reference "#PWR0340")
 					(unit 1)
 				)
@@
 		(dnp no)
 		(fields_autoplaced yes)
-		(property "Reference" "U20"
+		(property "Reference" "U19"
 			(at 148.59 80.01 0)
 			(effects
@@
 			(project "raywatch"
 				(path "/7b654ee8-2a53-4d39-8b7d-32c7bb3cb0ed/34ecb33f-48ad-4657-abe2-b4caffc19e6d"
-					(reference "U20")
+					(reference "U19")
 					(unit 1)
 				)
@@
 		(dnp no)
 		(fields_autoplaced yes)
-		(property "Reference" "#PWR0334"
+		(property "Reference" "#PWR0335"
 			(at 105.41 49.53 0)
 			(effects
@@
 			(project "raywatch"
 				(path "/7b654ee8-2a53-4d39-8b7d-32c7bb3cb0ed/34ecb33f-48ad-4657-abe2-b4caffc19e6d"
-					(reference "#PWR0334")
-					(unit 1)
-				)
+					(reference "#PWR0335")
+					(unit 1)
+				)

Commit message: Changed pin headers to vertical
Parts:
- J61, J63: footprint Connector_PinHeader_2.54mm:PinHeader_1x02_P2.54mm_Horizontal -> Connector_PinHeader_2.54mm:PinHeader_1x02_P2.54mm_Vertical
- J62: footprint Connector_PinHeader_2.54mm:PinHeader_1x01_P2.54mm_Horizontal -> Connector_PinHeader_2.54mm:PinHeader_1x04_P2.54mm_Vertical
Changed lines of the file:
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@@
 			)
 		)
-		(property "Footprint" "Connector_PinHeader_2.54mm:PinHeader_1x02_P2.54mm_Horizontal"
+		(property "Footprint" "Connector_PinHeader_2.54mm:PinHeader_1x02_P2.54mm_Vertical"
 			(at 93.98 68.58 0)
 			(effects
@@
 			)
 		)
-		(property "Footprint" "Connector_PinHeader_2.54mm:PinHeader_1x01_P2.54mm_Horizontal"
+		(property "Footprint" "Connector_PinHeader_2.54mm:PinHeader_1x04_P2.54mm_Vertical"
 			(at 93.98 58.42 0)
 			(effects
@@
 			)
 		)
-		(property "Footprint" "Connector_PinHeader_2.54mm:PinHeader_1x02_P2.54mm_Horizontal"
+		(property "Footprint" "Connector_PinHeader_2.54mm:PinHeader_1x02_P2.54mm_Vertical"
 			(at 93.98 46.99 0)
 			(effects

Commit message: Fixed connector footprints; Changed conectors from 2.54 to 1.27
Parts:
- J59: renamed from J61; footprint Connector_PinHeader_2.54mm:PinHeader_1x02_P2.54mm_Vertical -> Connector_PinHeader_1.27mm:PinHeader_1x02_P1.27mm_Vertical
- J60: renamed from J62; footprint Connector_PinHeader_2.54mm:PinHeader_1x04_P2.54mm_Vertical -> Connector_PinHeader_1.27mm:PinHeader_1x01_P1.27mm_Vertical
- J61: renamed from J63; footprint Connector_PinHeader_2.54mm:PinHeader_1x02_P2.54mm_Vertical -> Connector_PinHeader_1.27mm:PinHeader_1x02_P1.27mm_Vertical
Changed lines of the file:
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@@
 		(dnp no)
 		(fields_autoplaced yes)
-		(property "Reference" "#PWR0337"
+		(property "Reference" "#PWR0339"
 			(at 129.54 124.46 0)
 			(effects
@@
 			(project "raywatch"
 				(path "/7b654ee8-2a53-4d39-8b7d-32c7bb3cb0ed/34ecb33f-48ad-4657-abe2-b4caffc19e6d"
-					(reference "#PWR0337")
+					(reference "#PWR0339")
 					(unit 1)
 				)
@@
 		(dnp no)
 		(fields_autoplaced yes)
-		(property "Reference" "#PWR0334"
+		(property "Reference" "#PWR0336"
 			(at 95.25 46.99 0)
 			(effects
@@
 			(project "raywatch"
 				(path "/7b654ee8-2a53-4d39-8b7d-32c7bb3cb0ed/34ecb33f-48ad-4657-abe2-b4caffc19e6d"
-					(reference "#PWR0334")
+					(reference "#PWR0336")
 					(unit 1)
 				)
@@
 		(dnp no)
 		(fields_autoplaced yes)
-		(property "Reference" "#PWR0338"
+		(property "Reference" "#PWR0340"
 			(at 167.64 83.82 0)
 			(effects
@@
 			(project "raywatch"
 				(path "/7b654ee8-2a53-4d39-8b7d-32c7bb3cb0ed/34ecb33f-48ad-4657-abe2-b4caffc19e6d"
-					(reference "#PWR0338")
+					(reference "#PWR0340")
 					(unit 1)
 				)
@@
 		(dnp no)
 		(fields_autoplaced yes)
-		(property "Reference" "#PWR0339"
+		(property "Reference" "#PWR0341"
 			(at 167.64 114.3 0)
 			(effects
@@
 			(project "raywatch"
 				(path "/7b654ee8-2a53-4d39-8b7d-32c7bb3cb0ed/34ecb33f-48ad-4657-abe2-b4caffc19e6d"
-					(reference "#PWR0339")
+					(reference "#PWR0341")
 					(unit 1)
 				)
@@
 		(dnp no)
 		(fields_autoplaced yes)
-		(property "Reference" "J63"
+		(property "Reference" "J61"
 			(at 92.71 68.5799 0)
 			(effects
@@
 			)
 		)
-		(property "Footprint" "Connector_PinHeader_2.54mm:PinHeader_1x02_P2.54mm_Vertical"
+		(property "Footprint" "Connector_PinHeader_1.27mm:PinHeader_1x02_P1.27mm_Vertical"
 			(at 93.98 68.58 0)
 			(effects
@@
 			(project "raywatch"
 				(path "/7b654ee8-2a53-4d39-8b7d-32c7bb3cb0ed/34ecb33f-48ad-4657-abe2-b4caffc19e6d"
-					(reference "J63")
+					(reference "J61")
 					(unit 1)
 				)
@@
 		(dnp no)
 		(fields_autoplaced yes)
-		(property "Reference" "J62"
+		(property "Reference" "J60"
 			(at 92.71 57.1499 0)
 			(effects
@@
 			)
 		)
-		(property "Footprint" "Connector_PinHeader_2.54mm:PinHeader_1x04_P2.54mm_Vertical"
+		(property "Footprint" "Connector_PinHeader_1.27mm:PinHeader_1x01_P1.27mm_Vertical"
 			(at 93.98 58.42 0)
 			(effects
@@
 			(project "raywatch"
 				(path "/7b654ee8-2a53-4d39-8b7d-32c7bb3cb0ed/34ecb33f-48ad-4657-abe2-b4caffc19e6d"
-					(reference "J62")
+					(reference "J60")
 					(unit 1)
 				)
@@
 		(dnp no)
 		(fields_autoplaced yes)
-		(property "Reference" "#PWR0336"
+		(property "Reference" "#PWR0338"
 			(at 129.54 83.82 0)
 			(effects
@@
 			(project "raywatch"
 				(path "/7b654ee8-2a53-4d39-8b7d-32c7bb3cb0ed/34ecb33f-48ad-4657-abe2-b4caffc19e6d"
-					(reference "#PWR0336")
+					(reference "#PWR0338")
 					(unit 1)
 				)
@@
 		(dnp no)
 		(fields_autoplaced yes)
-		(property "Reference" "J61"
+		(property "Reference" "J59"
 			(at 92.71 46.9899 0)
 			(effects
@@
 			)
 		)
-		(property "Footprint" "Connector_PinHeader_2.54mm:PinHeader_1x02_P2.54mm_Vertical"
+		(property "Footprint" "Connector_PinHeader_1.27mm:PinHeader_1x02_P1.27mm_Vertical"
 			(at 93.98 46.99 0)
 			(effects
@@
 			(project "raywatch"
 				(path "/7b654ee8-2a53-4d39-8b7d-32c7bb3cb0ed/34ecb33f-48ad-4657-abe2-b4caffc19e6d"
-					(reference "J61")
+					(reference "J59")
 					(unit 1)
 				)
@@
 		(dnp no)
 		(fields_autoplaced yes)
-		(property "Reference" "#PWR0340"
+		(property "Reference" "#PWR0342"
 			(at 167.64 124.46 0)
 			(effects
@@
 			(project "raywatch"
 				(path "/7b654ee8-2a53-4d39-8b7d-32c7bb3cb0ed/34ecb33f-48ad-4657-abe2-b4caffc19e6d"
-					(reference "#PWR0340")
+					(reference "#PWR0342")
 					(unit 1)
 				)
@@
 		(dnp no)
 		(fields_autoplaced yes)
-		(property "Reference" "#PWR0335"
+		(property "Reference" "#PWR0337"
 			(at 105.41 49.53 0)
 			(effects
@@
 			(project "raywatch"
 				(path "/7b654ee8-2a53-4d39-8b7d-32c7bb3cb0ed/34ecb33f-48ad-4657-abe2-b4caffc19e6d"
-					(reference "#PWR0335")
-					(unit 1)
-				)
+					(reference "#PWR0337")
+					(unit 1)
+				)
