File: src/hardware/vibration_motor.kicad_sch (KiCad schematic)
At the start: 8 parts, among them J59 Conn_01x02_Pin, J60 Conn_01x01_Pin, J61 Conn_01x02_Pin, U19 DRV2605LYZFR

Commit message: Fixes; Added TPM PCB
Parts:
- C49, C50: footprint Capacitor_SMD:C_0504_1310Metric -> Capacitor_SMD:C_0402_1005Metric
Changed lines of the file:
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@@
 			)
 		)
-		(property "Footprint" "Capacitor_SMD:C_0504_1310Metric"
+		(property "Footprint" "Capacitor_SMD:C_0402_1005Metric"
 			(at 168.6052 118.11 0)
 			(effects
@@
 			)
 		)
-		(property "Footprint" "Capacitor_SMD:C_0504_1310Metric"
+		(property "Footprint" "Capacitor_SMD:C_0402_1005Metric"
 			(at 130.5052 118.11 0)
 			(effects
