File: src/hardware/charging_controller.kicad_sch (KiCad schematic)
At the start: 14 parts, among them U30 TPS22916BYFPR, U31 BQ25185DLHR

Commit message: Selected S1..10 & TR1
Parts:
- removed TH1: 10kΩ at 25°C, symbol Device:Thermistor_NTC
- added RT1: NTCG103JF103FT1, Project:THERM_NTCG103JF103FT1, symbol NTCG103JF103FT1:NTCG103JF103FT1
Connections:
- net GND: now also RT1.2
- net at U31.6 (TS/MR): now also RT1.1
Changed lines of the file:
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@@
 	(wire
 		(pts
-			(xy 195.58 106.68) (xy 191.77 106.68)
+			(xy 172.72 74.93) (xy 179.07 74.93)
 		)
 		(stroke
@@
 	(wire
 		(pts
-			(xy 172.72 74.93) (xy 179.07 74.93)
+			(xy 168.91 91.44) (xy 165.1 91.44)
 		)
 		(stroke
@@
 	(wire
 		(pts
-			(xy 168.91 91.44) (xy 165.1 91.44)
+			(xy 190.5 74.93) (xy 190.5 91.44)
 		)
 		(stroke
@@
 	(wire
 		(pts
-			(xy 190.5 74.93) (xy 190.5 91.44)
+			(xy 104.14 99.06) (xy 105.41 99.06)
 		)
 		(stroke
@@
 	(wire
 		(pts
-			(xy 104.14 99.06) (xy 105.41 99.06)
+			(xy 165.1 106.68) (xy 184.15 106.68)
 		)
 		(stroke
@@
 	(wire
 		(pts
-			(xy 165.1 106.68) (xy 184.15 106.68)
+			(xy 96.52 115.57) (xy 96.52 104.14)
 		)
 		(stroke
@@
 	(wire
 		(pts
-			(xy 96.52 115.57) (xy 96.52 104.14)
+			(xy 165.1 91.44) (xy 165.1 93.98)
 		)
 		(stroke
@@
 	(wire
 		(pts
-			(xy 165.1 91.44) (xy 165.1 93.98)
+			(xy 104.14 96.52) (xy 105.41 96.52)
 		)
 		(stroke
@@
 	(wire
 		(pts
-			(xy 104.14 96.52) (xy 105.41 96.52)
+			(xy 165.1 74.93) (xy 168.91 74.93)
 		)
 		(stroke
@@
 	(wire
 		(pts
-			(xy 165.1 74.93) (xy 168.91 74.93)
+			(xy 165.1 99.06) (xy 165.1 106.68)
 		)
 		(stroke
@@
 	(wire
 		(pts
-			(xy 165.1 99.06) (xy 165.1 106.68)
+			(xy 124.46 106.68) (xy 129.54 106.68)
 		)
 		(stroke
@@
 	(wire
 		(pts
-			(xy 124.46 106.68) (xy 129.54 106.68)
+			(xy 105.41 96.52) (xy 129.54 96.52)
 		)
 		(stroke
@@
 	(wire
 		(pts
-			(xy 105.41 96.52) (xy 129.54 96.52)
+			(xy 105.41 91.44) (xy 105.41 93.98)
 		)
 		(stroke
@@
 	(wire
 		(pts
-			(xy 105.41 91.44) (xy 105.41 93.98)
+			(xy 168.91 74.93) (xy 172.72 74.93)
 		)
 		(stroke
@@
 	(wire
 		(pts
-			(xy 168.91 74.93) (xy 172.72 74.93)
+			(xy 96.52 104.14) (xy 129.54 104.14)
 		)
 		(stroke
@@
 	(wire
 		(pts
-			(xy 96.52 104.14) (xy 129.54 104.14)
+			(xy 105.41 93.98) (xy 129.54 93.98)
 		)
 		(stroke
@@
 	(wire
 		(pts
-			(xy 105.41 93.98) (xy 129.54 93.98)
+			(xy 104.14 91.44) (xy 105.41 91.44)
 		)
 		(stroke
@@
 	(wire
 		(pts
-			(xy 104.14 91.44) (xy 105.41 91.44)
+			(xy 125.73 74.93) (xy 129.54 74.93)
 		)
 		(stroke
@@
 	(wire
 		(pts
-			(xy 125.73 74.93) (xy 129.54 74.93)
+			(xy 101.6 114.3) (xy 124.46 114.3)
 		)
 		(stroke
@@
 	(wire
 		(pts
-			(xy 101.6 114.3) (xy 124.46 114.3)
+			(xy 96.52 124.46) (xy 96.52 123.19)
 		)
 		(stroke
@@
 	(wire
 		(pts
-			(xy 96.52 124.46) (xy 96.52 123.19)
+			(xy 190.5 91.44) (xy 179.07 91.44)
 		)
 		(stroke
@@
 		)
 	)
-	(wire
-		(pts
-			(xy 190.5 91.44) (xy 179.07 91.44)
-		)
-		(stroke
-			(width 0)
-			(type default)
-		)
-	)
 	(global_label "CHARGESTAT2"
 		(shape output)
@@
 	)
 	(symbol
-		(lib_id "Device:Thermistor_NTC")
-		(at 187.96 106.68 90)
-		(unit 1)
-		(exclude_from_sim no)
-		(in_bom yes)
-		(on_board yes)
-		(dnp no)
-		(fields_autoplaced yes)
-		(property "Reference" "TH1"
-			(at 188.2775 100.33 90)
-			(effects
-				(font
-					(size 1.27 1.27)
-				)
-			)
-		)
-		(property "Value" "10kΩ at 25°C"
-			(at 188.2775 102.87 90)
-			(effects
-				(font
-					(size 1.27 1.27)
-				)
-			)
-		)
-		(property "Footprint" ""
-			(at 186.69 106.68 0)
-			(effects
-				(font
-					(size 1.27 1.27)
-				)
-				(hide yes)
-			)
-		)
-		(property "Datasheet" "~"
-			(at 186.69 106.68 0)
-			(effects
-				(font
-					(size 1.27 1.27)
-				)
-				(hide yes)
-			)
-		)
-		(property "Description" "Temperature dependent resistor, negative temperature coefficient"
-			(at 187.96 106.68 0)
-			(effects
-				(font
-					(size 1.27 1.27)
-				)
-				(hide yes)
-			)
-		)
-		(property "β(25/85)" "3435K"
-			(at 187.96 106.68 90)
-			(effects
-				(font
-					(size 1.27 1.27)
-				)
-				(hide yes)
-			)
-		)
-		(pin "1"
-		)
-		(pin "2"
-		)
-		(instances
-			(project "raywatch"
-				(path "/7b654ee8-2a53-4d39-8b7d-32c7bb3cb0ed/8b20ce3c-0acc-410e-a16d-32a077d218e5"
-					(reference "TH1")
-					(unit 1)
-				)
-			)
-		)
-	)
-	(symbol
 		(lib_id "power:GND")
 		(at 124.46 149.86 0)
@@
 	(symbol
 		(lib_id "power:GND")
-		(at 195.58 106.68 0)
+		(at 199.39 106.68 0)
 		(unit 1)
 		(exclude_from_sim no)
@@
 		(fields_autoplaced yes)
 		(property "Reference" "#PWR0389"
-			(at 195.58 113.03 0)
+			(at 199.39 113.03 0)
 			(effects
 				(font
@@
 		)
 		(property "Value" "GND"
-			(at 195.58 111.76 0)
+			(at 199.39 111.76 0)
 			(effects
 				(font
@@
 		)
 		(property "Footprint" ""
-			(at 195.58 106.68 0)
+			(at 199.39 106.68 0)
 			(effects
 				(font
@@
 		)
 		(property "Datasheet" ""
-			(at 195.58 106.68 0)
+			(at 199.39 106.68 0)
 			(effects
 				(font
@@
 		)
 		(property "Description" "Power symbol creates a global label with name \"GND\" , ground"
-			(at 195.58 106.68 0)
+			(at 199.39 106.68 0)
 			(effects
 				(font
@@
 					(unit 1)
 				)
+			)
+		)
+	)
+	(symbol
+		(lib_id "NTCG103JF103FT1:NTCG103JF103FT1")
+		(at 191.77 106.68 0)
+		(unit 1)
+		(exclude_from_sim no)
+		(in_bom yes)
+		(on_board yes)
+		(dnp no)
+		(fields_autoplaced yes)
+		(property "Reference" "RT1"
+			(at 191.643 99.06 0)
+			(effects
+				(font
+					(size 1.27 1.27)
+				)
+			)
+		)
+		(property "Value" "NTCG103JF103FT1"
+			(at 191.643 101.6 0)
+			(effects
+				(font
+					(size 1.27 1.27)
+				)
+			)
+		)
+		(property "Footprint" "Project:THERM_NTCG103JF103FT1"
+			(at 191.77 106.68 0)
+			(effects
+				(font
+					(size 1.27 1.27)
+				)
+				(justify bottom)
+				(hide yes)
+			)
+		)
+		(property "Datasheet" ""
+			(at 191.77 106.68 0)
+			(effects
+				(font
+					(size 1.27 1.27)
+				)
+				(hide yes)
+			)
+		)
+		(property "Description" ""
+			(at 191.77 106.68 0)
+			(effects
+				(font
+					(size 1.27 1.27)
+				)
+				(hide yes)
+			)
+		)
+		(property "MF" "TDK"
+			(at 191.77 106.68 0)
+			(effects
+				(font
+					(size 1.27 1.27)
+				)
+				(justify bottom)
+				(hide yes)
+			)
+		)
+		(property "MAXIMUM_PACKAGE_HEIGHT" "0.55 mm"
+			(at 191.77 106.68 0)
+			(effects
+				(font
+					(size 1.27 1.27)
+				)
+				(justify bottom)
+				(hide yes)
+			)
+		)
+		(property "Package" "1005 TDK"
+			(at 191.77 106.68 0)
+			(effects
+				(font
+					(size 1.27 1.27)
+				)
+				(justify bottom)
+				(hide yes)
+			)
+		)
+		(property "Price" "None"
+			(at 191.77 106.68 0)
+			(effects
+				(font
+					(size 1.27 1.27)
+				)
+				(justify bottom)
+				(hide yes)
+			)
+		)
+		(property "Check_prices" "https://www.snapeda.com/parts/NTCG103JF103FT1/TDK/view-part/?ref=eda"
+			(at 191.77 106.68 0)
+			(effects
+				(font
+					(size 1.27 1.27)
+				)
+				(justify bottom)
+				(hide yes)
+			)
+		)
+		(property "STANDARD" "Manufacturer Recommendations"
+			(at 191.77 106.68 0)
+			(effects
+				(font
+					(size 1.27 1.27)
+				)
+				(justify bottom)
+				(hide yes)
+			)
+		)
+		(property "PARTREV" "8/12/2022"
+			(at 191.77 106.68 0)
+			(effects
+				(font
+					(size 1.27 1.27)
+				)
+				(justify bottom)
+				(hide yes)
+			)
+		)
+		(property "SnapEDA_Link" "https://www.snapeda.com/parts/NTCG103JF103FT1/TDK/view-part/?ref=snap"
+			(at 191.77 106.68 0)
+			(effects
+				(font
+					(size 1.27 1.27)
+				)
+				(justify bottom)
+				(hide yes)
+			)
+		)
+		(property "MP" "NTCG103JF103FT1"
+			(at 191.77 106.68 0)
+			(effects
+				(font
+					(size 1.27 1.27)
+				)
+				(justify bottom)
+				(hide yes)
+			)
+		)
+		(property "Description_1" "NTC Thermistor 10k 0402 (1005 Metric)"
+			(at 191.77 106.68 0)
+			(effects
+				(font
+					(size 1.27 1.27)
+				)
+				(justify bottom)
+				(hide yes)
+			)
+		)
+		(property "Availability" "In Stock"
+			(at 191.77 106.68 0)
+			(effects
+				(font
+					(size 1.27 1.27)
+				)
+				(justify bottom)
+				(hide yes)
+			)
+		)
+		(property "MANUFACTURER" "TDK"
+			(at 191.77 106.68 0)
+			(effects
+				(font
+					(size 1.27 1.27)
+				)
+				(justify bottom)
+				(hide yes)
+			)
+		)
+		(pin "1"
+		)
+		(pin "2"
+		)
+		(instances
+			(project "raywatch"
+				(path "/7b654ee8-2a53-4d39-8b7d-32c7bb3cb0ed/8b20ce3c-0acc-410e-a16d-32a077d218e5"
+					(reference "RT1")
+					(unit 1)
+				)
