File: src/hardware/charging_controller.kicad_sch (KiCad schematic)
At the start: 14 parts, among them U30 TPS22916BYFPR, U31 BQ25185DLHR

Commit message: Mapped battery pinout; Removed thermistor from PCB, now using thermistor in battery pack
Parts:
- removed RT1: NTCG103JF103FT1, Project:THERM_NTCG103JF103FT1, symbol NTCG103JF103FT1:NTCG103JF103FT1
Connections:
- net BATTERM: now reaches U31.6 (TS/MR)

Commit message: Changed footprints from 0603 to 0402
Parts:
- C76, C77, C78, C79, C80, C81: footprint Capacitor_SMD:C_0603_1608Metric -> Capacitor_SMD:C_0504_1310Metric
- R39, R40, R41, R42, R43: footprint Resistor_SMD:R_0603_1608Metric -> Resistor_SMD:R_0402_1005Metric
Changed lines of the file:
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@@
 			)
 		)
-		(property "Footprint" "Capacitor_SMD:C_0603_1608Metric"
+		(property "Footprint" "Capacitor_SMD:C_0504_1310Metric"
 			(at 126.6952 74.93 0)
 			(effects
@@
 			)
 		)
-		(property "Footprint" "Capacitor_SMD:C_0603_1608Metric"
+		(property "Footprint" "Capacitor_SMD:C_0504_1310Metric"
 			(at 178.1048 91.44 0)
 			(effects
@@
 			)
 		)
-		(property "Footprint" "Resistor_SMD:R_0603_1608Metric"
+		(property "Footprint" "Resistor_SMD:R_0402_1005Metric"
 			(at 100.33 93.218 90)
 			(effects
@@
 			)
 		)
-		(property "Footprint" "Capacitor_SMD:C_0603_1608Metric"
+		(property "Footprint" "Capacitor_SMD:C_0504_1310Metric"
 			(at 167.9448 74.93 0)
 			(effects
@@
 			)
 		)
-		(property "Footprint" "Capacitor_SMD:C_0603_1608Metric"
+		(property "Footprint" "Capacitor_SMD:C_0504_1310Metric"
 			(at 178.1048 74.93 0)
 			(effects
@@
 			)
 		)
-		(property "Footprint" "Capacitor_SMD:C_0603_1608Metric"
+		(property "Footprint" "Capacitor_SMD:C_0504_1310Metric"
 			(at 116.5352 74.93 0)
 			(effects
@@
 			)
 		)
-		(property "Footprint" "Capacitor_SMD:C_0603_1608Metric"
+		(property "Footprint" "Capacitor_SMD:C_0504_1310Metric"
 			(at 167.9448 91.44 0)
 			(effects
@@
 			)
 		)
-		(property "Footprint" "Resistor_SMD:R_0603_1608Metric"
+		(property "Footprint" "Resistor_SMD:R_0402_1005Metric"
 			(at 100.33 100.838 90)
 			(effects
@@
 			)
 		)
-		(property "Footprint" "Resistor_SMD:R_0603_1608Metric"
+		(property "Footprint" "Resistor_SMD:R_0402_1005Metric"
 			(at 103.378 119.38 90)
 			(effects
@@
 			)
 		)
-		(property "Footprint" "Resistor_SMD:R_0603_1608Metric"
+		(property "Footprint" "Resistor_SMD:R_0402_1005Metric"
 			(at 98.298 119.38 90)
 			(effects
@@
 			)
 		)
-		(property "Footprint" "Resistor_SMD:R_0603_1608Metric"
+		(property "Footprint" "Resistor_SMD:R_0402_1005Metric"
 			(at 122.682 110.49 90)
 			(effects

Commit message: Replaced global labels with pin headers
Parts:
- added J15: Conn_01x04_Pin, symbol Connector:Conn_01x04_Pin
- added J16, J18: Conn_01x02_Pin, symbol Connector:Conn_01x02_Pin
- added J17, J20: Conn_02x08_Top_Bottom, symbol Connector_Generic:Conn_02x08_Top_Bottom
- added J19: Conn_01x01_Pin, symbol Connector:Conn_01x01_Pin
Connections:
- net +4V5: now also J17.1 (Pin_1), J17.2 (Pin_2), J17.3 (Pin_3), J17.4 (Pin_4), J17.5 (Pin_5), J17.6 (Pin_6), J17.7 (Pin_7), J17.8 (Pin_8), J20.1 (Pin_1), J20.2 (Pin_2), J20.3 (Pin_3), J20.4 (Pin_4), J20.5 (Pin_5), J20.6 (Pin_6), J20.7 (Pin_7), J20.8 (Pin_8)
- net BATTERM: now also J19.1 (Pin_1)
- net CHARGESTAT1: now also J15.3 (Pin_3)
- net CHARGESTAT2: now also J15.4 (Pin_4)
- net FASTCHARGE: now also J15.1 (Pin_1)
- net GND: now also J16.2 (Pin_2), J17.10 (Pin_10), J17.11 (Pin_11), J17.12 (Pin_12), J17.13 (Pin_13), J17.14 (Pin_14), J17.15 (Pin_15), J17.16 (Pin_16), J17.9 (Pin_9), J18.2 (Pin_2), J20.10 (Pin_10), J20.11 (Pin_11), J20.12 (Pin_12), J20.13 (Pin_13), J20.14 (Pin_14), J20.15 (Pin_15), J20.16 (Pin_16), J20.9 (Pin_9)
- net VBAT: now also J18.1 (Pin_1)
- net VIN: now also J16.1 (Pin_1)
- net \ENCHARGE: now also J15.2 (Pin_2)

Commit message: Reannotated schematic
Parts:
- renumbered C76 to C71, C77 to C72, C78 to C73, C79 to C74, C80 to C75, C81 to C76, J16 to J82, J15 to J83, J17 to J84, J20 to J85, J18 to J86, J19 to J87, R39 to R33, R40 to R34, R41 to R35, R42 to R36, R43 to R37, U30 to U31, U31 to U32

Commit message: Assigned pin header footprints
Parts:
- J82, J86: footprint (none) -> Connector_PinHeader_2.54mm:PinHeader_1x02_P2.54mm_Horizontal
- J83: footprint (none) -> Connector_PinHeader_2.54mm:PinHeader_1x04_P2.54mm_Horizontal
- J84, J85: footprint (none) -> Connector_PinHeader_2.54mm:PinHeader_1x16_P2.54mm_Vertical
- J87: footprint (none) -> Connector_PinHeader_2.54mm:PinHeader_1x01_P2.54mm_Horizontal
Changed lines of the file:
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@@
 			)
 		)
-		(property "Footprint" ""
+		(property "Footprint" "Connector_PinHeader_2.54mm:PinHeader_1x01_P2.54mm_Horizontal"
 			(at 200.66 48.26 0)
 			(effects
@@
 			)
 		)
-		(property "Footprint" ""
+		(property "Footprint" "Connector_PinHeader_2.54mm:PinHeader_1x16_P2.54mm_Vertical"
 			(at 127 44.45 0)
 			(effects
@@
 			)
 		)
-		(property "Footprint" ""
+		(property "Footprint" "Connector_PinHeader_2.54mm:PinHeader_1x02_P2.54mm_Horizontal"
 			(at 74.93 44.45 0)
 			(effects
@@
 			)
 		)
-		(property "Footprint" ""
+		(property "Footprint" "Connector_PinHeader_2.54mm:PinHeader_1x02_P2.54mm_Horizontal"
 			(at 200.66 39.37 0)
 			(effects
@@
 			)
 		)
-		(property "Footprint" ""
+		(property "Footprint" "Connector_PinHeader_2.54mm:PinHeader_1x16_P2.54mm_Vertical"
 			(at 152.4 44.45 0)
 			(effects
@@
 			)
 		)
-		(property "Footprint" ""
+		(property "Footprint" "Connector_PinHeader_2.54mm:PinHeader_1x04_P2.54mm_Horizontal"
 			(at 74.93 54.61 0)
 			(effects

Commit message: Fixed footprints
Parts:
- J84, J85: footprint Connector_PinHeader_2.54mm:PinHeader_1x16_P2.54mm_Vertical -> Connector_PinHeader_2.54mm:PinHeader_2x08_P2.54mm_Vertical
Changed lines of the file:
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@@
 			)
 		)
-		(property "Footprint" "Connector_PinHeader_2.54mm:PinHeader_1x16_P2.54mm_Vertical"
+		(property "Footprint" "Connector_PinHeader_2.54mm:PinHeader_2x08_P2.54mm_Vertical"
 			(at 127 44.45 0)
 			(effects
@@
 			)
 		)
-		(property "Footprint" "Connector_PinHeader_2.54mm:PinHeader_1x16_P2.54mm_Vertical"
+		(property "Footprint" "Connector_PinHeader_2.54mm:PinHeader_2x08_P2.54mm_Vertical"
 			(at 152.4 44.45 0)
 			(effects

Commit message: Fixed Footprint of BQ25185DLHR
Parts:
- U32: footprint Project:IC_BQ25185DLHR -> BQ25185DLHR:IC_BQ25185DLHR
Changed lines of the file:
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@@
 			)
 		)
-		(property "Footprint" "Project:IC_BQ25185DLHR"
+		(property "Footprint" "BQ25185DLHR:IC_BQ25185DLHR"
 			(at 147.32 101.6 0)
 			(effects
