File: src/hardware/1v8_converter.kicad_sch (KiCad schematic)
At the start: 0 parts

Commit message: Added 1.8V converter
Parts:
- added C? (x2): 1µF, symbol Device:C
- added U?: TPS7A2018PDQNR, TPS7A2018PDQNR:VREG_TPS7A2018PDQNR, symbol TPS7A2018PDQNR:TPS7A2018PDQNR
Connections:
- new net: C?.2, U?.2 (GND)
- new net +1V8: C?.1, U?.1 (OUT)
- new net GND: C?.2, U?.5 (EXP)
- new net VSYS: C?.1, U?.3 (EN), U?.4 (IN)

Commit message: Fixed 1.8V converter
Connections:
- net GND: now also C?.2, U?.2 (GND)
Changed lines of the file:
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@@
+	)
+	(junction
+		(at 165.1 106.68)
+		(diameter 0)
+		(color 0 0 0 0)
 	)
 	(junction
 		(at 139.7 96.52)
+		(diameter 0)
+		(color 0 0 0 0)
+	)
+	(junction
+		(at 165.1 104.14)
 		(diameter 0)
 		(color 0 0 0 0)
@@
 		)
 		(stroke
+			(width 0)
+			(type default)
+		)
+	)
+	(wire
+		(pts
+			(xy 165.1 104.14) (xy 165.1 106.68)
+		)
+		(stroke

Commit message: Cleanup & Fixes; Added footprints; Removed Light sensors
Parts:
- C91, C92: renamed from C?; footprint (none) -> Capacitor_SMD:C_0603_1608Metric
- U28: renamed from U?; footprint TPS7A2018PDQNR:VREG_TPS7A2018PDQNR -> Project:VREG_TPS7A2018PDQNR
Changed lines of the file:
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@@
 		(dnp no)
 		(fields_autoplaced yes)
-		(property "Reference" "#PWR0383"
+		(property "Reference" "#PWR0372"
 			(at 165.1 113.03 0)
 			(effects
@@
 			(project "raywatch"
 				(path "/7b654ee8-2a53-4d39-8b7d-32c7bb3cb0ed/6e6a70ea-4db2-4b59-a2d7-c468f9b8b5a6/07fbbbca-9aa4-472c-8a7d-14bd6423f6c5"
-					(reference "#PWR0383")
+					(reference "#PWR0372")
 					(unit 1)
 				)
@@
 		(dnp no)
 		(fields_autoplaced yes)
-		(property "Reference" "C?"
+		(property "Reference" "C92"
 			(at 168.91 99.0599 0)
 			(effects
@@
 			)
 		)
-		(property "Footprint" ""
+		(property "Footprint" "Capacitor_SMD:C_0603_1608Metric"
 			(at 166.0652 104.14 0)
 			(effects
@@
 			(project "raywatch"
 				(path "/7b654ee8-2a53-4d39-8b7d-32c7bb3cb0ed/6e6a70ea-4db2-4b59-a2d7-c468f9b8b5a6/07fbbbca-9aa4-472c-8a7d-14bd6423f6c5"
-					(reference "C?")
+					(reference "C92")
 					(unit 1)
 				)
@@
 		(dnp no)
 		(fields_autoplaced yes)
-		(property "Reference" "#PWR0386"
+		(property "Reference" "#PWR0369"
 			(at 137.16 100.33 0)
 			(effects
@@
 			(project "raywatch"
 				(path "/7b654ee8-2a53-4d39-8b7d-32c7bb3cb0ed/6e6a70ea-4db2-4b59-a2d7-c468f9b8b5a6/07fbbbca-9aa4-472c-8a7d-14bd6423f6c5"
-					(reference "#PWR0386")
+					(reference "#PWR0369")
 					(unit 1)
 				)
@@
 		(dnp no)
 		(fields_autoplaced yes)
-		(property "Reference" "U?"
+		(property "Reference" "U28"
 			(at 152.4 88.9 0)
 			(effects
@@
 			)
 		)
-		(property "Footprint" "TPS7A2018PDQNR:VREG_TPS7A2018PDQNR"
+		(property "Footprint" "Project:VREG_TPS7A2018PDQNR"
 			(at 152.4 101.6 0)
 			(effects
@@
 			(project "raywatch"
 				(path "/7b654ee8-2a53-4d39-8b7d-32c7bb3cb0ed/6e6a70ea-4db2-4b59-a2d7-c468f9b8b5a6/07fbbbca-9aa4-472c-8a7d-14bd6423f6c5"
-					(reference "U?")
+					(reference "U28")
 					(unit 1)
 				)
@@
 		(dnp no)
 		(fields_autoplaced yes)
-		(property "Reference" "#PWR0384"
+		(property "Reference" "#PWR0370"
 			(at 137.16 110.49 0)
 			(effects
@@
 			(project "raywatch"
 				(path "/7b654ee8-2a53-4d39-8b7d-32c7bb3cb0ed/6e6a70ea-4db2-4b59-a2d7-c468f9b8b5a6/07fbbbca-9aa4-472c-8a7d-14bd6423f6c5"
-					(reference "#PWR0384")
+					(reference "#PWR0370")
 					(unit 1)
 				)
@@
 		(dnp no)
 		(fields_autoplaced yes)
-		(property "Reference" "C?"
+		(property "Reference" "C91"
 			(at 133.35 99.0599 0)
 			(effects
@@
 			)
 		)
-		(property "Footprint" ""
+		(property "Footprint" "Capacitor_SMD:C_0603_1608Metric"
 			(at 136.1948 104.14 0)
 			(effects
@@
 			(project "raywatch"
 				(path "/7b654ee8-2a53-4d39-8b7d-32c7bb3cb0ed/6e6a70ea-4db2-4b59-a2d7-c468f9b8b5a6/07fbbbca-9aa4-472c-8a7d-14bd6423f6c5"
-					(reference "C?")
+					(reference "C91")
 					(unit 1)
 				)
@@
 		(dnp no)
 		(fields_autoplaced yes)
-		(property "Reference" "#PWR0385"
+		(property "Reference" "#PWR0371"
 			(at 165.1 100.33 0)
 			(effects
@@
 			(project "raywatch"
 				(path "/7b654ee8-2a53-4d39-8b7d-32c7bb3cb0ed/6e6a70ea-4db2-4b59-a2d7-c468f9b8b5a6/07fbbbca-9aa4-472c-8a7d-14bd6423f6c5"
-					(reference "#PWR0385")
+					(reference "#PWR0371")
 					(unit 1)
 				)

Commit message: Cleanup & Fixes; Changed GPIO; Added Camera; Added Microphone
Parts:
- renumbered C91 to C89, C92 to C90
Changed lines of the file:
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@@
 		(dnp no)
 		(fields_autoplaced yes)
-		(property "Reference" "#PWR0372"
+		(property "Reference" "#PWR0368"
 			(at 165.1 113.03 0)
 			(effects
@@
 			(project "raywatch"
 				(path "/7b654ee8-2a53-4d39-8b7d-32c7bb3cb0ed/6e6a70ea-4db2-4b59-a2d7-c468f9b8b5a6/07fbbbca-9aa4-472c-8a7d-14bd6423f6c5"
-					(reference "#PWR0372")
+					(reference "#PWR0368")
 					(unit 1)
 				)
@@
 		(dnp no)
 		(fields_autoplaced yes)
-		(property "Reference" "C92"
+		(property "Reference" "C90"
 			(at 168.91 99.0599 0)
 			(effects
@@
 			(project "raywatch"
 				(path "/7b654ee8-2a53-4d39-8b7d-32c7bb3cb0ed/6e6a70ea-4db2-4b59-a2d7-c468f9b8b5a6/07fbbbca-9aa4-472c-8a7d-14bd6423f6c5"
-					(reference "C92")
+					(reference "C90")
 					(unit 1)
 				)
@@
 		(dnp no)
 		(fields_autoplaced yes)
-		(property "Reference" "#PWR0369"
+		(property "Reference" "#PWR0365"
 			(at 137.16 100.33 0)
 			(effects
@@
 			(project "raywatch"
 				(path "/7b654ee8-2a53-4d39-8b7d-32c7bb3cb0ed/6e6a70ea-4db2-4b59-a2d7-c468f9b8b5a6/07fbbbca-9aa4-472c-8a7d-14bd6423f6c5"
-					(reference "#PWR0369")
+					(reference "#PWR0365")
 					(unit 1)
 				)
@@
 		(dnp no)
 		(fields_autoplaced yes)
-		(property "Reference" "#PWR0370"
+		(property "Reference" "#PWR0366"
 			(at 137.16 110.49 0)
 			(effects
@@
 			(project "raywatch"
 				(path "/7b654ee8-2a53-4d39-8b7d-32c7bb3cb0ed/6e6a70ea-4db2-4b59-a2d7-c468f9b8b5a6/07fbbbca-9aa4-472c-8a7d-14bd6423f6c5"
-					(reference "#PWR0370")
+					(reference "#PWR0366")
 					(unit 1)
 				)
@@
 		(dnp no)
 		(fields_autoplaced yes)
-		(property "Reference" "C91"
+		(property "Reference" "C89"
 			(at 133.35 99.0599 0)
 			(effects
@@
 			(project "raywatch"
 				(path "/7b654ee8-2a53-4d39-8b7d-32c7bb3cb0ed/6e6a70ea-4db2-4b59-a2d7-c468f9b8b5a6/07fbbbca-9aa4-472c-8a7d-14bd6423f6c5"
-					(reference "C91")
+					(reference "C89")
 					(unit 1)
 				)
@@
 		(dnp no)
 		(fields_autoplaced yes)
-		(property "Reference" "#PWR0371"
+		(property "Reference" "#PWR0367"
 			(at 165.1 100.33 0)
 			(effects
@@
 			(project "raywatch"
 				(path "/7b654ee8-2a53-4d39-8b7d-32c7bb3cb0ed/6e6a70ea-4db2-4b59-a2d7-c468f9b8b5a6/07fbbbca-9aa4-472c-8a7d-14bd6423f6c5"
-					(reference "#PWR0371")
+					(reference "#PWR0367")
 					(unit 1)
 				)

Commit message: Add Light Sensor and Proximity & Gesture Sensor; Changed GPIO
Parts:
- renumbered U28 to U29
Changed lines of the file:
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@@
 		(dnp no)
 		(fields_autoplaced yes)
-		(property "Reference" "#PWR0368"
+		(property "Reference" "#PWR0372"
 			(at 165.1 113.03 0)
 			(effects
@@
 			(project "raywatch"
 				(path "/7b654ee8-2a53-4d39-8b7d-32c7bb3cb0ed/6e6a70ea-4db2-4b59-a2d7-c468f9b8b5a6/07fbbbca-9aa4-472c-8a7d-14bd6423f6c5"
-					(reference "#PWR0368")
+					(reference "#PWR0372")
 					(unit 1)
 				)
@@
 		(dnp no)
 		(fields_autoplaced yes)
-		(property "Reference" "#PWR0365"
+		(property "Reference" "#PWR0369"
 			(at 137.16 100.33 0)
 			(effects
@@
 			(project "raywatch"
 				(path "/7b654ee8-2a53-4d39-8b7d-32c7bb3cb0ed/6e6a70ea-4db2-4b59-a2d7-c468f9b8b5a6/07fbbbca-9aa4-472c-8a7d-14bd6423f6c5"
-					(reference "#PWR0365")
+					(reference "#PWR0369")
 					(unit 1)
 				)
@@
 		(dnp no)
 		(fields_autoplaced yes)
-		(property "Reference" "U28"
+		(property "Reference" "U29"
 			(at 152.4 88.9 0)
 			(effects
@@
 			(project "raywatch"
 				(path "/7b654ee8-2a53-4d39-8b7d-32c7bb3cb0ed/6e6a70ea-4db2-4b59-a2d7-c468f9b8b5a6/07fbbbca-9aa4-472c-8a7d-14bd6423f6c5"
-					(reference "U28")
+					(reference "U29")
 					(unit 1)
 				)
@@
 		(dnp no)
 		(fields_autoplaced yes)
-		(property "Reference" "#PWR0366"
+		(property "Reference" "#PWR0370"
 			(at 137.16 110.49 0)
 			(effects
@@
 			(project "raywatch"
 				(path "/7b654ee8-2a53-4d39-8b7d-32c7bb3cb0ed/6e6a70ea-4db2-4b59-a2d7-c468f9b8b5a6/07fbbbca-9aa4-472c-8a7d-14bd6423f6c5"
-					(reference "#PWR0366")
+					(reference "#PWR0370")
 					(unit 1)
 				)
@@
 		(dnp no)
 		(fields_autoplaced yes)
-		(property "Reference" "#PWR0367"
+		(property "Reference" "#PWR0371"
 			(at 165.1 100.33 0)
 			(effects
@@
 			(project "raywatch"
 				(path "/7b654ee8-2a53-4d39-8b7d-32c7bb3cb0ed/6e6a70ea-4db2-4b59-a2d7-c468f9b8b5a6/07fbbbca-9aa4-472c-8a7d-14bd6423f6c5"
-					(reference "#PWR0367")
+					(reference "#PWR0371")
 					(unit 1)
 				)

Commit message: Flattend hirachy
Parts:
- renumbered C89 to C66, C90 to C67, U29 to U24
Changed lines of the file:
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@@
 		(dnp no)
 		(fields_autoplaced yes)
-		(property "Reference" "#PWR0372"
+		(property "Reference" "#PWR0343"
 			(at 165.1 113.03 0)
 			(effects
@@
 		(instances
 			(project "raywatch"
-				(path "/7b654ee8-2a53-4d39-8b7d-32c7bb3cb0ed/6e6a70ea-4db2-4b59-a2d7-c468f9b8b5a6/07fbbbca-9aa4-472c-8a7d-14bd6423f6c5"
-					(reference "#PWR0372")
+				(path "/7b654ee8-2a53-4d39-8b7d-32c7bb3cb0ed/b8c5e1e6-da5e-4fb2-8283-82eb932a0e50"
+					(reference "#PWR0343")
 					(unit 1)
 				)
@@
 		(dnp no)
 		(fields_autoplaced yes)
-		(property "Reference" "C90"
+		(property "Reference" "C67"
 			(at 168.91 99.0599 0)
 			(effects
@@
 		(instances
 			(project "raywatch"
-				(path "/7b654ee8-2a53-4d39-8b7d-32c7bb3cb0ed/6e6a70ea-4db2-4b59-a2d7-c468f9b8b5a6/07fbbbca-9aa4-472c-8a7d-14bd6423f6c5"
-					(reference "C90")
+				(path "/7b654ee8-2a53-4d39-8b7d-32c7bb3cb0ed/b8c5e1e6-da5e-4fb2-8283-82eb932a0e50"
+					(reference "C67")
 					(unit 1)
 				)
@@
 		(dnp no)
 		(fields_autoplaced yes)
-		(property "Reference" "#PWR0369"
+		(property "Reference" "#PWR0340"
 			(at 137.16 100.33 0)
 			(effects
@@
 		(instances
 			(project "raywatch"
-				(path "/7b654ee8-2a53-4d39-8b7d-32c7bb3cb0ed/6e6a70ea-4db2-4b59-a2d7-c468f9b8b5a6/07fbbbca-9aa4-472c-8a7d-14bd6423f6c5"
-					(reference "#PWR0369")
+				(path "/7b654ee8-2a53-4d39-8b7d-32c7bb3cb0ed/b8c5e1e6-da5e-4fb2-8283-82eb932a0e50"
+					(reference "#PWR0340")
 					(unit 1)
 				)
@@
 		(dnp no)
 		(fields_autoplaced yes)
-		(property "Reference" "U29"
+		(property "Reference" "U24"
 			(at 152.4 88.9 0)
 			(effects
@@
 		(instances
 			(project "raywatch"
-				(path "/7b654ee8-2a53-4d39-8b7d-32c7bb3cb0ed/6e6a70ea-4db2-4b59-a2d7-c468f9b8b5a6/07fbbbca-9aa4-472c-8a7d-14bd6423f6c5"
-					(reference "U29")
+				(path "/7b654ee8-2a53-4d39-8b7d-32c7bb3cb0ed/b8c5e1e6-da5e-4fb2-8283-82eb932a0e50"
+					(reference "U24")
 					(unit 1)
 				)
@@
 		(dnp no)
 		(fields_autoplaced yes)
-		(property "Reference" "#PWR0370"
+		(property "Reference" "#PWR0341"
 			(at 137.16 110.49 0)
 			(effects
@@
 		(instances
 			(project "raywatch"
-				(path "/7b654ee8-2a53-4d39-8b7d-32c7bb3cb0ed/6e6a70ea-4db2-4b59-a2d7-c468f9b8b5a6/07fbbbca-9aa4-472c-8a7d-14bd6423f6c5"
-					(reference "#PWR0370")
+				(path "/7b654ee8-2a53-4d39-8b7d-32c7bb3cb0ed/b8c5e1e6-da5e-4fb2-8283-82eb932a0e50"
+					(reference "#PWR0341")
 					(unit 1)
 				)
@@
 		(dnp no)
 		(fields_autoplaced yes)
-		(property "Reference" "C89"
+		(property "Reference" "C66"
 			(at 133.35 99.0599 0)
 			(effects
@@
 		(instances
 			(project "raywatch"
-				(path "/7b654ee8-2a53-4d39-8b7d-32c7bb3cb0ed/6e6a70ea-4db2-4b59-a2d7-c468f9b8b5a6/07fbbbca-9aa4-472c-8a7d-14bd6423f6c5"
-					(reference "C89")
+				(path "/7b654ee8-2a53-4d39-8b7d-32c7bb3cb0ed/b8c5e1e6-da5e-4fb2-8283-82eb932a0e50"
+					(reference "C66")
 					(unit 1)
 				)
@@
 		(dnp no)
 		(fields_autoplaced yes)
-		(property "Reference" "#PWR0371"
+		(property "Reference" "#PWR0342"
 			(at 165.1 100.33 0)
 			(effects
@@
 		(instances
 			(project "raywatch"
-				(path "/7b654ee8-2a53-4d39-8b7d-32c7bb3cb0ed/6e6a70ea-4db2-4b59-a2d7-c468f9b8b5a6/07fbbbca-9aa4-472c-8a7d-14bd6423f6c5"
-					(reference "#PWR0371")
+				(path "/7b654ee8-2a53-4d39-8b7d-32c7bb3cb0ed/b8c5e1e6-da5e-4fb2-8283-82eb932a0e50"
+					(reference "#PWR0342")
 					(unit 1)
 				)
