File: src/hardware/battery_protection.kicad_sch (KiCad schematic)
At the start: 0 parts

Commit message: Added Battery Protection
Parts:
- added C?: 100µF, symbol Device:C
- added Q? (x2): Q_NMOS, symbol Device:Q_NMOS
- added R?: 330, symbol Device:R
- added R?: 2.2k, symbol Device:R
- added U?: BQ29700DSER, BQ29700DSER:SON50P150X150X80-6N, symbol BQ29700DSER:BQ29700DSER
Connections:
- new net: C?.1, R?.2, U?.5 (BAT)
- new net: Q?.D, Q?.D
- new net: Q?.G, U?.2 (COUT)
- new net: Q?.G, U?.3 (DOUT)
- new net: R?.2, U?.6 (V-)
- new net +BATT: R?.1
- new net -BATT: C?.2, Q?.S, U?.4 (VSS)
- new net GND: Q?.S, R?.1
- no-connect marks 0 -> 1

Commit message: Added Accelerometer Clock; Cleanup & Fixes
Parts:
- R?: value 2.2k -> 2.2kΩ
Changed lines of the file:
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@@
 			)
 		)
-		(property "Value" "2.2k"
+		(property "Value" "2.2kΩ"
 			(at 134.62 101.5999 0)
 			(effects

Commit message: Cleanup & Fixes; Added footprints; Removed Light sensors
Parts:
- removed Q? (x2): Q_NMOS, symbol Device:Q_NMOS
- added U33: CSD83325L, Project:YJE0006A, symbol CSD83325L:CSD83325L
- C99: renamed from C?; footprint (none) -> Capacitor_SMD:C_0603_1608Metric
- R47, R48: renamed from R?; footprint (none) -> Resistor_SMD:R_0603_1608Metric
- U32: renamed from U?; footprint BQ29700DSER:SON50P150X150X80-6N -> Project:SON50P150X150X80-6N
Connections:
- net -BATT: now also U33.A1 (S1), U33.C1 (S1)
- net GND: now also U33.A2 (S2), U33.C2 (S2)
- net at U32.2 (COUT): now also U33.B2 (G2)
- net at U32.3 (DOUT): now also U33.B1 (G1)

Commit message: Cleanup & Fixes; Changed GPIO; Added Camera; Added Microphone
Parts:
- renumbered C99 to C97, R47 to R45, R48 to R46
Changed lines of the file:
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@@
 		(dnp no)
 		(fields_autoplaced yes)
-		(property "Reference" "R47"
+		(property "Reference" "R45"
 			(at 123.19 86.3599 0)
 			(effects
@@
 			(project "raywatch"
 				(path "/7b654ee8-2a53-4d39-8b7d-32c7bb3cb0ed/6e6a70ea-4db2-4b59-a2d7-c468f9b8b5a6/7d73f677-e1d3-42ef-8813-aac813c5814d"
-					(reference "R47")
+					(reference "R45")
 					(unit 1)
 				)
@@
 		(dnp no)
 		(fields_autoplaced yes)
-		(property "Reference" "#PWR0396"
+		(property "Reference" "#PWR0392"
 			(at 137.16 110.49 0)
 			(effects
@@
 			(project "raywatch"
 				(path "/7b654ee8-2a53-4d39-8b7d-32c7bb3cb0ed/6e6a70ea-4db2-4b59-a2d7-c468f9b8b5a6/7d73f677-e1d3-42ef-8813-aac813c5814d"
-					(reference "#PWR0396")
+					(reference "#PWR0392")
 					(unit 1)
 				)
@@
 		(dnp no)
 		(fields_autoplaced yes)
-		(property "Reference" "#PWR0399"
+		(property "Reference" "#PWR0395"
 			(at 179.07 114.3 0)
 			(effects
@@
 			(project "raywatch"
 				(path "/7b654ee8-2a53-4d39-8b7d-32c7bb3cb0ed/6e6a70ea-4db2-4b59-a2d7-c468f9b8b5a6/7d73f677-e1d3-42ef-8813-aac813c5814d"
-					(reference "#PWR0399")
+					(reference "#PWR0395")
 					(unit 1)
 				)
@@
 		(dnp no)
 		(fields_autoplaced yes)
-		(property "Reference" "#PWR0395"
+		(property "Reference" "#PWR0391"
 			(at 120.65 95.25 0)
 			(effects
@@
 			(project "raywatch"
 				(path "/7b654ee8-2a53-4d39-8b7d-32c7bb3cb0ed/6e6a70ea-4db2-4b59-a2d7-c468f9b8b5a6/7d73f677-e1d3-42ef-8813-aac813c5814d"
-					(reference "#PWR0395")
+					(reference "#PWR0391")
 					(unit 1)
 				)
@@
 		(dnp no)
 		(fields_autoplaced yes)
-		(property "Reference" "#PWR0397"
+		(property "Reference" "#PWR0393"
 			(at 167.64 107.95 0)
 			(effects
@@
 			(project "raywatch"
 				(path "/7b654ee8-2a53-4d39-8b7d-32c7bb3cb0ed/6e6a70ea-4db2-4b59-a2d7-c468f9b8b5a6/7d73f677-e1d3-42ef-8813-aac813c5814d"
-					(reference "#PWR0397")
+					(reference "#PWR0393")
 					(unit 1)
 				)
@@
 		(dnp no)
 		(fields_autoplaced yes)
-		(property "Reference" "#PWR0394"
+		(property "Reference" "#PWR0390"
 			(at 120.65 87.63 0)
 			(effects
@@
 			(project "raywatch"
 				(path "/7b654ee8-2a53-4d39-8b7d-32c7bb3cb0ed/6e6a70ea-4db2-4b59-a2d7-c468f9b8b5a6/7d73f677-e1d3-42ef-8813-aac813c5814d"
-					(reference "#PWR0394")
+					(reference "#PWR0390")
 					(unit 1)
 				)
@@
 		(dnp no)
 		(fields_autoplaced yes)
-		(property "Reference" "R48"
+		(property "Reference" "R46"
 			(at 134.62 99.0599 0)
 			(effects
@@
 			(project "raywatch"
 				(path "/7b654ee8-2a53-4d39-8b7d-32c7bb3cb0ed/6e6a70ea-4db2-4b59-a2d7-c468f9b8b5a6/7d73f677-e1d3-42ef-8813-aac813c5814d"
-					(reference "R48")
+					(reference "R46")
 					(unit 1)
 				)
@@
 		(dnp no)
 		(fields_autoplaced yes)
-		(property "Reference" "C99"
+		(property "Reference" "C97"
 			(at 124.46 93.9799 0)
 			(effects
@@
 			(project "raywatch"
 				(path "/7b654ee8-2a53-4d39-8b7d-32c7bb3cb0ed/6e6a70ea-4db2-4b59-a2d7-c468f9b8b5a6/7d73f677-e1d3-42ef-8813-aac813c5814d"
-					(reference "C99")
+					(reference "C97")
 					(unit 1)
 				)
@@
 		(dnp no)
 		(fields_autoplaced yes)
-		(property "Reference" "#PWR0398"
+		(property "Reference" "#PWR0394"
 			(at 179.07 71.12 0)
 			(effects
@@
 			(project "raywatch"
 				(path "/7b654ee8-2a53-4d39-8b7d-32c7bb3cb0ed/6e6a70ea-4db2-4b59-a2d7-c468f9b8b5a6/7d73f677-e1d3-42ef-8813-aac813c5814d"
-					(reference "#PWR0398")
-					(unit 1)
-				)
+					(reference "#PWR0394")
+					(unit 1)
+				)

Commit message: Add Light Sensor and Proximity & Gesture Sensor; Changed GPIO
Parts:
- renumbered R45 to R46, R46 to R47
Changed lines of the file:
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@@
 		(dnp no)
 		(fields_autoplaced yes)
-		(property "Reference" "R45"
+		(property "Reference" "R46"
 			(at 123.19 86.3599 0)
 			(effects
@@
 			(project "raywatch"
 				(path "/7b654ee8-2a53-4d39-8b7d-32c7bb3cb0ed/6e6a70ea-4db2-4b59-a2d7-c468f9b8b5a6/7d73f677-e1d3-42ef-8813-aac813c5814d"
-					(reference "R45")
+					(reference "R46")
 					(unit 1)
 				)
@@
 		(dnp no)
 		(fields_autoplaced yes)
-		(property "Reference" "#PWR0392"
+		(property "Reference" "#PWR0394"
 			(at 137.16 110.49 0)
 			(effects
@@
 			(project "raywatch"
 				(path "/7b654ee8-2a53-4d39-8b7d-32c7bb3cb0ed/6e6a70ea-4db2-4b59-a2d7-c468f9b8b5a6/7d73f677-e1d3-42ef-8813-aac813c5814d"
-					(reference "#PWR0392")
+					(reference "#PWR0394")
 					(unit 1)
 				)
@@
 		(dnp no)
 		(fields_autoplaced yes)
-		(property "Reference" "#PWR0395"
+		(property "Reference" "#PWR0397"
 			(at 179.07 114.3 0)
 			(effects
@@
 			(project "raywatch"
 				(path "/7b654ee8-2a53-4d39-8b7d-32c7bb3cb0ed/6e6a70ea-4db2-4b59-a2d7-c468f9b8b5a6/7d73f677-e1d3-42ef-8813-aac813c5814d"
-					(reference "#PWR0395")
+					(reference "#PWR0397")
 					(unit 1)
 				)
@@
 		(dnp no)
 		(fields_autoplaced yes)
-		(property "Reference" "#PWR0391"
+		(property "Reference" "#PWR0393"
 			(at 120.65 95.25 0)
 			(effects
@@
 			(project "raywatch"
 				(path "/7b654ee8-2a53-4d39-8b7d-32c7bb3cb0ed/6e6a70ea-4db2-4b59-a2d7-c468f9b8b5a6/7d73f677-e1d3-42ef-8813-aac813c5814d"
-					(reference "#PWR0391")
+					(reference "#PWR0393")
 					(unit 1)
 				)
@@
 		(dnp no)
 		(fields_autoplaced yes)
-		(property "Reference" "#PWR0393"
+		(property "Reference" "#PWR0395"
 			(at 167.64 107.95 0)
 			(effects
@@
 			(project "raywatch"
 				(path "/7b654ee8-2a53-4d39-8b7d-32c7bb3cb0ed/6e6a70ea-4db2-4b59-a2d7-c468f9b8b5a6/7d73f677-e1d3-42ef-8813-aac813c5814d"
-					(reference "#PWR0393")
+					(reference "#PWR0395")
 					(unit 1)
 				)
@@
 		(dnp no)
 		(fields_autoplaced yes)
-		(property "Reference" "#PWR0390"
+		(property "Reference" "#PWR0392"
 			(at 120.65 87.63 0)
 			(effects
@@
 			(project "raywatch"
 				(path "/7b654ee8-2a53-4d39-8b7d-32c7bb3cb0ed/6e6a70ea-4db2-4b59-a2d7-c468f9b8b5a6/7d73f677-e1d3-42ef-8813-aac813c5814d"
-					(reference "#PWR0390")
+					(reference "#PWR0392")
 					(unit 1)
 				)
@@
 		(dnp no)
 		(fields_autoplaced yes)
-		(property "Reference" "R46"
+		(property "Reference" "R47"
 			(at 134.62 99.0599 0)
 			(effects
@@
 			(project "raywatch"
 				(path "/7b654ee8-2a53-4d39-8b7d-32c7bb3cb0ed/6e6a70ea-4db2-4b59-a2d7-c468f9b8b5a6/7d73f677-e1d3-42ef-8813-aac813c5814d"
-					(reference "R46")
+					(reference "R47")
 					(unit 1)
 				)
@@
 		(dnp no)
 		(fields_autoplaced yes)
-		(property "Reference" "#PWR0394"
+		(property "Reference" "#PWR0396"
 			(at 179.07 71.12 0)
 			(effects
@@
 			(project "raywatch"
 				(path "/7b654ee8-2a53-4d39-8b7d-32c7bb3cb0ed/6e6a70ea-4db2-4b59-a2d7-c468f9b8b5a6/7d73f677-e1d3-42ef-8813-aac813c5814d"
-					(reference "#PWR0394")
-					(unit 1)
-				)
+					(reference "#PWR0396")
+					(unit 1)
+				)

Commit message: Flattend hirachy
Parts:
- renumbered C97 to C75, R46 to R37, R47 to R38, U32 to U28, U33 to U29
Changed lines of the file:
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@@
 		(dnp no)
 		(fields_autoplaced yes)
-		(property "Reference" "R46"
+		(property "Reference" "R37"
 			(at 123.19 86.3599 0)
 			(effects
@@
 		(instances
 			(project "raywatch"
-				(path "/7b654ee8-2a53-4d39-8b7d-32c7bb3cb0ed/6e6a70ea-4db2-4b59-a2d7-c468f9b8b5a6/7d73f677-e1d3-42ef-8813-aac813c5814d"
-					(reference "R46")
+				(path "/7b654ee8-2a53-4d39-8b7d-32c7bb3cb0ed/78c9fb69-bd8b-4be2-a858-27c158c5dba8"
+					(reference "R37")
 					(unit 1)
 				)
@@
 		(dnp no)
 		(fields_autoplaced yes)
-		(property "Reference" "#PWR0394"
+		(property "Reference" "#PWR0367"
 			(at 137.16 110.49 0)
 			(effects
@@
 		(instances
 			(project "raywatch"
-				(path "/7b654ee8-2a53-4d39-8b7d-32c7bb3cb0ed/6e6a70ea-4db2-4b59-a2d7-c468f9b8b5a6/7d73f677-e1d3-42ef-8813-aac813c5814d"
-					(reference "#PWR0394")
+				(path "/7b654ee8-2a53-4d39-8b7d-32c7bb3cb0ed/78c9fb69-bd8b-4be2-a858-27c158c5dba8"
+					(reference "#PWR0367")
 					(unit 1)
 				)
@@
 		(dnp no)
 		(fields_autoplaced yes)
-		(property "Reference" "#PWR0397"
+		(property "Reference" "#PWR0370"
 			(at 179.07 114.3 0)
 			(effects
@@
 		(instances
 			(project "raywatch"
-				(path "/7b654ee8-2a53-4d39-8b7d-32c7bb3cb0ed/6e6a70ea-4db2-4b59-a2d7-c468f9b8b5a6/7d73f677-e1d3-42ef-8813-aac813c5814d"
-					(reference "#PWR0397")
+				(path "/7b654ee8-2a53-4d39-8b7d-32c7bb3cb0ed/78c9fb69-bd8b-4be2-a858-27c158c5dba8"
+					(reference "#PWR0370")
 					(unit 1)
 				)
@@
 		(dnp no)
 		(fields_autoplaced yes)
-		(property "Reference" "U32"
+		(property "Reference" "U28"
 			(at 152.4 83.82 0)
 			(effects
@@
 		(instances
 			(project "raywatch"
-				(path "/7b654ee8-2a53-4d39-8b7d-32c7bb3cb0ed/6e6a70ea-4db2-4b59-a2d7-c468f9b8b5a6/7d73f677-e1d3-42ef-8813-aac813c5814d"
-					(reference "U32")
+				(path "/7b654ee8-2a53-4d39-8b7d-32c7bb3cb0ed/78c9fb69-bd8b-4be2-a858-27c158c5dba8"
+					(reference "U28")
 					(unit 1)
 				)
@@
 		(dnp no)
 		(fields_autoplaced yes)
-		(property "Reference" "#PWR0393"
+		(property "Reference" "#PWR0366"
 			(at 120.65 95.25 0)
 			(effects
@@
 		(instances
 			(project "raywatch"
-				(path "/7b654ee8-2a53-4d39-8b7d-32c7bb3cb0ed/6e6a70ea-4db2-4b59-a2d7-c468f9b8b5a6/7d73f677-e1d3-42ef-8813-aac813c5814d"
-					(reference "#PWR0393")
+				(path "/7b654ee8-2a53-4d39-8b7d-32c7bb3cb0ed/78c9fb69-bd8b-4be2-a858-27c158c5dba8"
+					(reference "#PWR0366")
 					(unit 1)
 				)
@@
 		(dnp no)
 		(fields_autoplaced yes)
-		(property "Reference" "#PWR0395"
+		(property "Reference" "#PWR0368"
 			(at 167.64 107.95 0)
 			(effects
@@
 		(instances
 			(project "raywatch"
-				(path "/7b654ee8-2a53-4d39-8b7d-32c7bb3cb0ed/6e6a70ea-4db2-4b59-a2d7-c468f9b8b5a6/7d73f677-e1d3-42ef-8813-aac813c5814d"
-					(reference "#PWR0395")
+				(path "/7b654ee8-2a53-4d39-8b7d-32c7bb3cb0ed/78c9fb69-bd8b-4be2-a858-27c158c5dba8"
+					(reference "#PWR0368")
 					(unit 1)
 				)
@@
 		(dnp no)
 		(fields_autoplaced yes)
-		(property "Reference" "U33"
+		(property "Reference" "U29"
 			(at 182.88 96.5199 90)
 			(effects
@@
 		(instances
 			(project "raywatch"
-				(path "/7b654ee8-2a53-4d39-8b7d-32c7bb3cb0ed/6e6a70ea-4db2-4b59-a2d7-c468f9b8b5a6/7d73f677-e1d3-42ef-8813-aac813c5814d"
-					(reference "U33")
+				(path "/7b654ee8-2a53-4d39-8b7d-32c7bb3cb0ed/78c9fb69-bd8b-4be2-a858-27c158c5dba8"
+					(reference "U29")
 					(unit 1)
 				)
@@
 		(dnp no)
 		(fields_autoplaced yes)
-		(property "Reference" "#PWR0392"
+		(property "Reference" "#PWR0365"
 			(at 120.65 87.63 0)
 			(effects
@@
 		(instances
 			(project "raywatch"
-				(path "/7b654ee8-2a53-4d39-8b7d-32c7bb3cb0ed/6e6a70ea-4db2-4b59-a2d7-c468f9b8b5a6/7d73f677-e1d3-42ef-8813-aac813c5814d"
-					(reference "#PWR0392")
+				(path "/7b654ee8-2a53-4d39-8b7d-32c7bb3cb0ed/78c9fb69-bd8b-4be2-a858-27c158c5dba8"
+					(reference "#PWR0365")
 					(unit 1)
 				)
@@
 		(dnp no)
 		(fields_autoplaced yes)
-		(property "Reference" "R47"
+		(property "Reference" "R38"
 			(at 134.62 99.0599 0)
 			(effects
@@
 		(instances
 			(project "raywatch"
-				(path "/7b654ee8-2a53-4d39-8b7d-32c7bb3cb0ed/6e6a70ea-4db2-4b59-a2d7-c468f9b8b5a6/7d73f677-e1d3-42ef-8813-aac813c5814d"
-					(reference "R47")
+				(path "/7b654ee8-2a53-4d39-8b7d-32c7bb3cb0ed/78c9fb69-bd8b-4be2-a858-27c158c5dba8"
+					(reference "R38")
 					(unit 1)
 				)
@@
 		(dnp no)
 		(fields_autoplaced yes)
-		(property "Reference" "C97"
+		(property "Reference" "C75"
 			(at 124.46 93.9799 0)
 			(effects
@@
 		(instances
 			(project "raywatch"
-				(path "/7b654ee8-2a53-4d39-8b7d-32c7bb3cb0ed/6e6a70ea-4db2-4b59-a2d7-c468f9b8b5a6/7d73f677-e1d3-42ef-8813-aac813c5814d"
-					(reference "C97")
+				(path "/7b654ee8-2a53-4d39-8b7d-32c7bb3cb0ed/78c9fb69-bd8b-4be2-a858-27c158c5dba8"
+					(reference "C75")
 					(unit 1)
 				)
@@
 		(dnp no)
 		(fields_autoplaced yes)
-		(property "Reference" "#PWR0396"
+		(property "Reference" "#PWR0369"
 			(at 179.07 71.12 0)
 			(effects
@@
 		(instances
 			(project "raywatch"
-				(path "/7b654ee8-2a53-4d39-8b7d-32c7bb3cb0ed/6e6a70ea-4db2-4b59-a2d7-c468f9b8b5a6/7d73f677-e1d3-42ef-8813-aac813c5814d"
-					(reference "#PWR0396")
-					(unit 1)
-				)
+				(path "/7b654ee8-2a53-4d39-8b7d-32c7bb3cb0ed/78c9fb69-bd8b-4be2-a858-27c158c5dba8"
+					(reference "#PWR0369")
+					(unit 1)
+				)

Commit message: Cleanup
Parts:
- R37: value 330 -> 330Ω
Changed lines of the file:
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@@
 			)
 		)
-		(property "Value" "330"
+		(property "Value" "330Ω"
 			(at 123.19 88.8999 0)
 			(effects
