File: src/hardware/buttons.kicad_sch (KiCad schematic)
At the start: 0 parts

Commit message: Created Buttons
Parts:
- added C14, C15, C16, C17, C? (x6): 10nF, symbol Device:C
- added R2, R3, R4, R5, R? (x6): 200k, symbol Device:R
- added SW1, SW2, SW3, SW4, SW5, SW? (x5): SW_Push_Grounded, symbol Switch:SW_Push_Shielded
Connections:
- new net: R?.1, SW1.2
- new net: R4.1, SW4.2
- new net: R?.1, SW?.2 (x5)
- new net: R3.1, SW3.2
- new net: R2.1, SW2.2
- new net: R5.1, SW5.2
- new net +3V3: C14.2, C15.2, C16.2, C17.2, C?.2, C?.2, C?.2, C?.2, C?.2, C?.2
- new net BTN1: C?.1, R?.2
- new net BTN10: C?.1, R?.2
- new net BTN2: C14.1, R2.2
- new net BTN3: C15.1, R3.2
- new net BTN4: C16.1, R4.2
- new net BTN5: C17.1, R5.2
- new net BTN6: C?.1, R?.2
- new net BTN7: C?.1, R?.2
- new net BTN8: C?.1, R?.2
- new net BTN9: C?.1, R?.2
- new net GND: SW1.1, SW1.SH (B), SW2.1, SW2.SH (B), SW3.1, SW3.SH (B), SW4.1, SW4.SH (B), SW5.1, SW5.SH (B), SW?.1, SW?.1, SW?.1, SW?.1, SW?.1, SW?.SH (B), SW?.SH (B), SW?.SH (B), SW?.SH (B), SW?.SH (B)

Commit message: Added LoRa
Changed lines of the file:
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@@
 		)
 		(property "Value" "GND"
-			(at 107.95 85.09 0)
+			(at 105.41 81.2799 0)
 			(effects
 				(font
 					(size 1.27 1.27)
 				)
+				(justify right)
 			)
 		)
@@
 		)
 		(property "Value" "GND"
-			(at 189.23 85.09 0)
+			(at 191.77 81.2799 0)
 			(effects
 				(font
 					(size 1.27 1.27)
 				)
+				(justify right)
 			)
 		)
@@
 		)
 		(property "Value" "GND"
-			(at 189.23 64.77 0)
+			(at 191.77 60.9599 0)
 			(effects
 				(font
 					(size 1.27 1.27)
 				)
+				(justify right)
 			)
 		)
@@
 		)
 		(property "Value" "GND"
-			(at 107.95 123.19 0)
+			(at 105.41 119.3799 0)
 			(effects
 				(font
 					(size 1.27 1.27)
 				)
+				(justify right)
 			)
 		)
@@
 		)
 		(property "Value" "GND"
-			(at 107.95 104.14 0)
+			(at 105.41 100.3299 0)
 			(effects
 				(font
 					(size 1.27 1.27)
 				)
+				(justify right)
 			)
 		)
@@
 		)
 		(property "Value" "GND"
-			(at 107.95 64.77 0)
+			(at 105.41 60.9599 0)
 			(effects
 				(font
 					(size 1.27 1.27)
 				)
+				(justify right)
 			)
 		)
@@
 		)
 		(property "Value" "GND"
-			(at 189.23 142.24 0)
+			(at 191.77 138.4299 0)
 			(effects
 				(font
 					(size 1.27 1.27)
 				)
+				(justify right)
 			)
 		)
@@
 		)
 		(property "Value" "GND"
-			(at 189.23 104.14 0)
+			(at 191.77 100.3299 0)
 			(effects
 				(font
 					(size 1.27 1.27)
 				)
+				(justify right)
 			)
 		)
@@
 		)
 		(property "Value" "GND"
-			(at 189.23 123.19 0)
+			(at 191.77 119.3799 0)
 			(effects
 				(font
 					(size 1.27 1.27)
 				)
+				(justify right)
 			)
 		)
@@
 		)
 		(property "Value" "GND"
-			(at 107.95 142.24 0)
+			(at 105.41 138.4299 0)
 			(effects
 				(font
 					(size 1.27 1.27)
 				)
+				(justify right)
 			)
 		)

Commit message: Added Accelerometer Clock; Cleanup & Fixes
Parts:
- R2, R3, R4, R5, R? (x6): value 200k -> 200kΩ
Changed lines of the file:
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@@
 			)
 		)
-		(property "Value" "200k"
+		(property "Value" "200kΩ"
 			(at 125.73 114.3 90)
 			(effects
@@
 			)
 		)
-		(property "Value" "200k"
+		(property "Value" "200kΩ"
 			(at 171.45 95.25 90)
 			(effects
@@
 			)
 		)
-		(property "Value" "200k"
+		(property "Value" "200kΩ"
 			(at 125.73 95.25 90)
 			(effects
@@
 			)
 		)
-		(property "Value" "200k"
+		(property "Value" "200kΩ"
 			(at 171.45 76.2 90)
 			(effects
@@
 			)
 		)
-		(property "Value" "200k"
+		(property "Value" "200kΩ"
 			(at 171.45 55.88 90)
 			(effects
@@
 			)
 		)
-		(property "Value" "200k"
+		(property "Value" "200kΩ"
 			(at 125.73 133.35 90)
 			(effects
@@
 			)
 		)
-		(property "Value" "200k"
+		(property "Value" "200kΩ"
 			(at 171.45 133.35 90)
 			(effects
@@
 			)
 		)
-		(property "Value" "200k"
+		(property "Value" "200kΩ"
 			(at 171.45 114.3 90)
 			(effects
@@
 			)
 		)
-		(property "Value" "200k"
+		(property "Value" "200kΩ"
 			(at 125.73 55.88 90)
 			(effects
@@
 			)
 		)
-		(property "Value" "200k"
+		(property "Value" "200kΩ"
 			(at 125.73 76.2 90)
 			(effects

Commit message: Cleanup & Fixes; Added footprints; Removed Light sensors
Parts:
- C20, C25, C26, C27, C28, C29: renamed from C?; footprint (none) -> Capacitor_SMD:C_0603_1608Metric
- C21: renamed from C14; footprint (none) -> Capacitor_SMD:C_0603_1608Metric
- C22: renamed from C15; footprint (none) -> Capacitor_SMD:C_0603_1608Metric
- C23: renamed from C16; footprint (none) -> Capacitor_SMD:C_0603_1608Metric
- C24: renamed from C17; footprint (none) -> Capacitor_SMD:C_0603_1608Metric
- R14, R19, R20, R21, R22, R23: renamed from R?; footprint (none) -> Resistor_SMD:R_0603_1608Metric
- R15: renamed from R2; footprint (none) -> Resistor_SMD:R_0603_1608Metric
- R16: renamed from R3; footprint (none) -> Resistor_SMD:R_0603_1608Metric
- R17: renamed from R4; footprint (none) -> Resistor_SMD:R_0603_1608Metric
- R18: renamed from R5; footprint (none) -> Resistor_SMD:R_0603_1608Metric
- gave numbers to parts that had none: 5

Commit message: Cleanup & Fixes; Changed GPIO; Added Camera; Added Microphone
Parts:
- renumbered C20 to C18, C21 to C19, C22 to C20, C23 to C21, C24 to C22, C25 to C23, C26 to C24, C27 to C25, C28 to C26, C29 to C27, R14 to R12, R15 to R13, R16 to R14, R17 to R15, R18 to R16, R19 to R17, R20 to R18, R21 to R19, R22 to R20, R23 to R21

Commit message: Add Light Sensor and Proximity & Gesture Sensor; Changed GPIO
Parts:
- renumbered R12 to R13, R13 to R14, R14 to R15, R15 to R16, R16 to R17, R17 to R18, R18 to R19, R19 to R20, R20 to R21, R21 to R22

Commit message: Selected S1..10 & TR1
Parts:
- removed SW1, SW10, SW2, SW3, SW4, SW5, SW6, SW7, SW8, SW9: SW_Push_Grounded, symbol Switch:SW_Push_Shielded
- added S1, S10, S2, S3, S4, S5, S6, S7, S8, S9: EVQ-P7A01P, Project:SW_EVQ-P7A01P, symbol EVQ-P7A01P:EVQ-P7A01P
Connections:
- net GND: now also S1.1_1, S1.1_2, S10.1_1, S10.1_2, S2.1_1, S2.1_2, S3.1_1, S3.1_2, S4.1_1, S4.1_2, S5.1_1, S5.1_2, S6.1_1, S6.1_2, S7.1_1, S7.1_2, S8.1_1, S8.1_2, S9.1_1, S9.1_2
- net at R13.1: now also S1.2_1, S1.2_2
- net at R16.1: now also S4.2_1, S4.2_2
- net at R20.1: now also S8.2_1, S8.2_2
- net at R15.1: now also S3.2_1, S3.2_2
- net at R18.1: now also S6.2_1, S6.2_2
- net at R19.1: now also S7.2_1, S7.2_2
- net at R14.1: now also S2.2_1, S2.2_2
- net at R22.1: now also S10.2_1, S10.2_2
- net at R17.1: now also S5.2_1, S5.2_2
- net at R21.1: now also S9.2_1, S9.2_2
