File: src/hardware/microsd.kicad_sch (KiCad schematic)
At the start: 15 parts, among them J46 Conn_01x02_Pin, J47 Conn_01x02_Pin, J48 Conn_01x04_Pin, J49 MSD-1-A, U15 TPS22916BYFPR

Commit message: Fixes; Added TPM PCB
Parts:
- C39, C40: footprint Capacitor_SMD:C_0504_1310Metric -> Capacitor_SMD:C_0402_1005Metric
Changed lines of the file:
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@@
 			)
 		)
-		(property "Footprint" "Capacitor_SMD:C_0504_1310Metric"
+		(property "Footprint" "Capacitor_SMD:C_0402_1005Metric"
 			(at 148.2852 77.47 0)
 			(effects
@@
 			)
 		)
-		(property "Footprint" "Capacitor_SMD:C_0504_1310Metric"
+		(property "Footprint" "Capacitor_SMD:C_0402_1005Metric"
 			(at 159.7152 77.47 0)
 			(effects
