File: src/hardware/3v3_converter.kicad_sch (KiCad schematic)
At the start: 0 parts

Commit message: Added 3.3V Converter
Parts:
- added C? (x2): 1µF, symbol Device:C
- added U?: TPS7A2033DQNR, DQN0004A-MFG, symbol TPS7A2033DQNR:TPS7A2033DQNR
Connections:
- new net +3V3: C?.1, U?.1 (OUT)
- new net GND: C?.2, C?.2, U?.2 (GND), U?.5 (Thermal_Pad)
- new net VSYS: C?.1, U?.3 (EN), U?.4 (IN)

Commit message: Created Power Diagram
Other:
- moved on the sheet: C?, U?
Changed lines of the file:
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@@
 	)
 	(junction
-		(at 172.72 81.28)
+		(at 170.18 109.22)
 		(diameter 0)
 		(color 0 0 0 0)
 	)
 	(junction
-		(at 176.53 73.66)
+		(at 173.99 101.6)
 		(diameter 0)
 		(color 0 0 0 0)
 	)
 	(junction
-		(at 132.08 73.66)
+		(at 129.54 101.6)
 		(diameter 0)
 		(color 0 0 0 0)
 	)
 	(junction
-		(at 129.54 73.66)
+		(at 127 101.6)
 		(diameter 0)
 		(color 0 0 0 0)
@@
 	(wire
 		(pts
-			(xy 172.72 73.66) (xy 176.53 73.66)
+			(xy 170.18 101.6) (xy 173.99 101.6)
 		)
 		(stroke
@@
 	(wire
 		(pts
-			(xy 172.72 78.74) (xy 172.72 81.28)
+			(xy 170.18 106.68) (xy 170.18 109.22)
 		)
 		(stroke
@@
 	(wire
 		(pts
-			(xy 129.54 73.66) (xy 132.08 73.66)
+			(xy 127 101.6) (xy 129.54 101.6)
 		)
 		(stroke
@@
 	(wire
 		(pts
-			(xy 132.08 73.66) (xy 132.08 81.28)
+			(xy 129.54 101.6) (xy 129.54 109.22)
 		)
 		(stroke
@@
 	(symbol
 		(lib_id "TPS7A2033DQNR:TPS7A2033DQNR")
-		(at 132.08 73.66 0)
+		(at 129.54 101.6 0)
 		(unit 1)
 		(exclude_from_sim no)
@@
 		(fields_autoplaced yes)
 		(property "Reference" "U?"
-			(at 152.4 63.5 0)
+			(at 149.86 91.44 0)
 			(effects
 				(font
@@
 		)
 		(property "Value" "TPS7A2033DQNR"
-			(at 152.4 66.04 0)
+			(at 149.86 93.98 0)
 			(effects
 				(font
@@
 		)
 		(property "Footprint" "DQN0004A-MFG"
-			(at 132.08 73.66 0)
+			(at 129.54 101.6 0)
 			(effects
 				(font
@@
 		)
 		(property "Datasheet" "https://www.ti.com/lit/gpn/tps7a20"
-			(at 132.08 73.66 0)
+			(at 129.54 101.6 0)
 			(effects
 				(font
@@
 		)
 		(property "Description" ""
-			(at 132.08 73.66 0)
+			(at 129.54 101.6 0)
 			(effects
 				(font
@@
 	(symbol
 		(lib_id "power:GND")
-		(at 176.53 81.28 0)
+		(at 173.99 109.22 0)
 		(unit 1)
 		(exclude_from_sim no)
@@
 		(fields_autoplaced yes)
 		(property "Reference" "#PWR0395"
-			(at 176.53 87.63 0)
+			(at 173.99 115.57 0)
 			(effects
 				(font
@@
 		)
 		(property "Value" "GND"
-			(at 176.53 86.36 0)
-			(effects
-				(font
-					(size 1.27 1.27)
-				)
-			)
-		)
-		(property "Footprint" ""
-			(at 176.53 81.28 0)
+			(at 173.99 114.3 0)
+			(effects
+				(font
+					(size 1.27 1.27)
+				)
+			)
+		)
+		(property "Footprint" ""
+			(at 173.99 109.22 0)
 			(effects
 				(font
@@
 		)
 		(property "Datasheet" ""
-			(at 176.53 81.28 0)
+			(at 173.99 109.22 0)
 			(effects
 				(font
@@
 		)
 		(property "Description" "Power symbol creates a global label with name \"GND\" , ground"
-			(at 176.53 81.28 0)
+			(at 173.99 109.22 0)
 			(effects
 				(font
@@
 	(symbol
 		(lib_id "Device:C")
-		(at 129.54 77.47 0)
+		(at 127 105.41 0)
 		(mirror y)
 		(unit 1)
@@
 		(fields_autoplaced yes)
 		(property "Reference" "C?"
-			(at 125.73 76.1999 0)
+			(at 123.19 104.1399 0)
 			(effects
 				(font
@@
 		)
 		(property "Value" "1µF"
-			(at 125.73 78.7399 0)
+			(at 123.19 106.6799 0)
 			(effects
 				(font
@@
 		)
 		(property "Footprint" ""
-			(at 128.5748 81.28 0)
+			(at 126.0348 109.22 0)
 			(effects
 				(font
@@
 		)
 		(property "Datasheet" "~"
-			(at 129.54 77.47 0)
+			(at 127 105.41 0)
 			(effects
 				(font
@@
 		)
 		(property "Description" "Unpolarized capacitor"
-			(at 129.54 77.47 0)
+			(at 127 105.41 0)
 			(effects
 				(font
@@
 	(symbol
 		(lib_id "power:LINE")
-		(at 129.54 73.66 0)
+		(at 127 101.6 0)
 		(unit 1)
 		(exclude_from_sim no)
@@
 		(fields_autoplaced yes)
 		(property "Reference" "#PWR0391"
-			(at 129.54 77.47 0)
+			(at 127 105.41 0)
 			(effects
 				(font
@@
 		)
 		(property "Value" "VSYS"
-			(at 129.54 68.58 0)
-			(effects
-				(font
-					(size 1.27 1.27)
-				)
-			)
-		)
-		(property "Footprint" ""
-			(at 129.54 73.66 0)
+			(at 127 96.52 0)
+			(effects
+				(font
+					(size 1.27 1.27)
+				)
+			)
+		)
+		(property "Footprint" ""
+			(at 127 101.6 0)
 			(effects
 				(font
@@
 		)
 		(property "Datasheet" ""
-			(at 129.54 73.66 0)
+			(at 127 101.6 0)
 			(effects
 				(font
@@
 		)
 		(property "Description" "Power symbol creates a global label with name \"LINE\""
-			(at 129.54 73.66 0)
+			(at 127 101.6 0)
 			(effects
 				(font
@@
 	(symbol
 		(lib_id "power:GND")
-		(at 172.72 81.28 0)
+		(at 170.18 109.22 0)
 		(unit 1)
 		(exclude_from_sim no)
@@
 		(fields_autoplaced yes)
 		(property "Reference" "#PWR0394"
-			(at 172.72 87.63 0)
+			(at 170.18 115.57 0)
 			(effects
 				(font
@@
 		)
 		(property "Value" "GND"
-			(at 172.72 86.36 0)
-			(effects
-				(font
-					(size 1.27 1.27)
-				)
-			)
-		)
-		(property "Footprint" ""
-			(at 172.72 81.28 0)
+			(at 170.18 114.3 0)
+			(effects
+				(font
+					(size 1.27 1.27)
+				)
+			)
+		)
+		(property "Footprint" ""
+			(at 170.18 109.22 0)
 			(effects
 				(font
@@
 		)
 		(property "Datasheet" ""
-			(at 172.72 81.28 0)
+			(at 170.18 109.22 0)
 			(effects
 				(font
@@
 		)
 		(property "Description" "Power symbol creates a global label with name \"GND\" , ground"
-			(at 172.72 81.28 0)
+			(at 170.18 109.22 0)
 			(effects
 				(font
@@
 	(symbol
 		(lib_id "power:+3V3")
-		(at 176.53 73.66 0)
+		(at 173.99 101.6 0)
 		(unit 1)
 		(exclude_from_sim no)
@@
 		(fields_autoplaced yes)
 		(property "Reference" "#PWR0393"
-			(at 176.53 77.47 0)
+			(at 173.99 105.41 0)
 			(effects
 				(font
@@
 		)
 		(property "Value" "+3V3"
-			(at 176.53 68.58 0)
-			(effects
-				(font
-					(size 1.27 1.27)
-				)
-			)
-		)
-		(property "Footprint" ""
-			(at 176.53 73.66 0)
+			(at 173.99 96.52 0)
+			(effects
+				(font
+					(size 1.27 1.27)
+				)
+			)
+		)
+		(property "Footprint" ""
+			(at 173.99 101.6 0)
 			(effects
 				(font
@@
 		)
 		(property "Datasheet" ""
-			(at 176.53 73.66 0)
+			(at 173.99 101.6 0)
 			(effects
 				(font
@@
 		)
 		(property "Description" "Power symbol creates a global label with name \"+3V3\""
-			(at 176.53 73.66 0)
+			(at 173.99 101.6 0)
 			(effects
 				(font
@@
 	(symbol
 		(lib_id "power:GND")
-		(at 129.54 81.28 0)
+		(at 127 109.22 0)
 		(unit 1)
 		(exclude_from_sim no)
@@
 		(fields_autoplaced yes)
 		(property "Reference" "#PWR0392"
-			(at 129.54 87.63 0)
+			(at 127 115.57 0)
 			(effects
 				(font
@@
 		)
 		(property "Value" "GND"
-			(at 129.54 86.36 0)
-			(effects
-				(font
-					(size 1.27 1.27)
-				)
-			)
-		)
-		(property "Footprint" ""
-			(at 129.54 81.28 0)
+			(at 127 114.3 0)
+			(effects
+				(font
+					(size 1.27 1.27)
+				)
+			)
+		)
+		(property "Footprint" ""
+			(at 127 109.22 0)
 			(effects
 				(font
@@
 		)
 		(property "Datasheet" ""
-			(at 129.54 81.28 0)
+			(at 127 109.22 0)
 			(effects
 				(font
@@
 		)
 		(property "Description" "Power symbol creates a global label with name \"GND\" , ground"
-			(at 129.54 81.28 0)
+			(at 127 109.22 0)
 			(effects
 				(font
@@
 	(symbol
 		(lib_id "Device:C")
-		(at 176.53 77.47 0)
+		(at 173.99 105.41 0)
 		(unit 1)
 		(exclude_from_sim no)
@@
 		(fields_autoplaced yes)
 		(property "Reference" "C?"
-			(at 180.34 76.1999 0)
+			(at 177.8 104.1399 0)
 			(effects
 				(font
@@
 		)
 		(property "Value" "1µF"
-			(at 180.34 78.7399 0)
+			(at 177.8 106.6799 0)
 			(effects
 				(font
@@
 		)
 		(property "Footprint" ""
-			(at 177.4952 81.28 0)
+			(at 174.9552 109.22 0)
 			(effects
 				(font
@@
 		)
 		(property "Datasheet" "~"
-			(at 176.53 77.47 0)
+			(at 173.99 105.41 0)
 			(effects
 				(font
@@
 		)
 		(property "Description" "Unpolarized capacitor"
-			(at 176.53 77.47 0)
-			(effects
-				(font
+			(at 173.99 105.41 0)
+			(effects
+				(font

Commit message: Cleanup & Fixes; Added footprints; Removed Light sensors
Parts:
- C87, C88: renamed from C?; footprint (none) -> Capacitor_SMD:C_0603_1608Metric
- U26: renamed from U?; footprint DQN0004A-MFG -> Project:DQN0004A-MFG
Changed lines of the file:
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@@
 		(dnp no)
 		(fields_autoplaced yes)
-		(property "Reference" "U?"
+		(property "Reference" "U26"
 			(at 149.86 91.44 0)
 			(effects
@@
 			)
 		)
-		(property "Footprint" "DQN0004A-MFG"
+		(property "Footprint" "Project:DQN0004A-MFG"
 			(at 129.54 101.6 0)
 			(effects
@@
 			(project "raywatch"
 				(path "/7b654ee8-2a53-4d39-8b7d-32c7bb3cb0ed/6e6a70ea-4db2-4b59-a2d7-c468f9b8b5a6/b445ea2b-ce97-4fc9-a9bc-efa2f143df72"
-					(reference "U?")
+					(reference "U26")
 					(unit 1)
 				)
@@
 		(dnp no)
 		(fields_autoplaced yes)
-		(property "Reference" "#PWR0395"
+		(property "Reference" "#PWR0364"
 			(at 173.99 115.57 0)
 			(effects
@@
 			(project "raywatch"
 				(path "/7b654ee8-2a53-4d39-8b7d-32c7bb3cb0ed/6e6a70ea-4db2-4b59-a2d7-c468f9b8b5a6/b445ea2b-ce97-4fc9-a9bc-efa2f143df72"
-					(reference "#PWR0395")
+					(reference "#PWR0364")
 					(unit 1)
 				)
@@
 		(dnp no)
 		(fields_autoplaced yes)
-		(property "Reference" "C?"
+		(property "Reference" "C87"
 			(at 123.19 104.1399 0)
 			(effects
@@
 			)
 		)
-		(property "Footprint" ""
+		(property "Footprint" "Capacitor_SMD:C_0603_1608Metric"
 			(at 126.0348 109.22 0)
 			(effects
@@
 			(project "raywatch"
 				(path "/7b654ee8-2a53-4d39-8b7d-32c7bb3cb0ed/6e6a70ea-4db2-4b59-a2d7-c468f9b8b5a6/b445ea2b-ce97-4fc9-a9bc-efa2f143df72"
-					(reference "C?")
+					(reference "C87")
 					(unit 1)
 				)
@@
 		(dnp no)
 		(fields_autoplaced yes)
-		(property "Reference" "#PWR0391"
+		(property "Reference" "#PWR0360"
 			(at 127 105.41 0)
 			(effects
@@
 			(project "raywatch"
 				(path "/7b654ee8-2a53-4d39-8b7d-32c7bb3cb0ed/6e6a70ea-4db2-4b59-a2d7-c468f9b8b5a6/b445ea2b-ce97-4fc9-a9bc-efa2f143df72"
-					(reference "#PWR0391")
+					(reference "#PWR0360")
 					(unit 1)
 				)
@@
 		(dnp no)
 		(fields_autoplaced yes)
-		(property "Reference" "#PWR0394"
+		(property "Reference" "#PWR0362"
 			(at 170.18 115.57 0)
 			(effects
@@
 			(project "raywatch"
 				(path "/7b654ee8-2a53-4d39-8b7d-32c7bb3cb0ed/6e6a70ea-4db2-4b59-a2d7-c468f9b8b5a6/b445ea2b-ce97-4fc9-a9bc-efa2f143df72"
-					(reference "#PWR0394")
+					(reference "#PWR0362")
 					(unit 1)
 				)
@@
 		(dnp no)
 		(fields_autoplaced yes)
-		(property "Reference" "#PWR0393"
+		(property "Reference" "#PWR0363"
 			(at 173.99 105.41 0)
 			(effects
@@
 			(project "raywatch"
 				(path "/7b654ee8-2a53-4d39-8b7d-32c7bb3cb0ed/6e6a70ea-4db2-4b59-a2d7-c468f9b8b5a6/b445ea2b-ce97-4fc9-a9bc-efa2f143df72"
-					(reference "#PWR0393")
+					(reference "#PWR0363")
 					(unit 1)
 				)
@@
 		(dnp no)
 		(fields_autoplaced yes)
-		(property "Reference" "#PWR0392"
+		(property "Reference" "#PWR0361"
 			(at 127 115.57 0)
 			(effects
@@
 			(project "raywatch"
 				(path "/7b654ee8-2a53-4d39-8b7d-32c7bb3cb0ed/6e6a70ea-4db2-4b59-a2d7-c468f9b8b5a6/b445ea2b-ce97-4fc9-a9bc-efa2f143df72"
-					(reference "#PWR0392")
+					(reference "#PWR0361")
 					(unit 1)
 				)
@@
 		(dnp no)
 		(fields_autoplaced yes)
-		(property "Reference" "C?"
+		(property "Reference" "C88"
 			(at 177.8 104.1399 0)
 			(effects
@@
 			)
 		)
-		(property "Footprint" ""
+		(property "Footprint" "Capacitor_SMD:C_0603_1608Metric"
 			(at 174.9552 109.22 0)
 			(effects
@@
 			(project "raywatch"
 				(path "/7b654ee8-2a53-4d39-8b7d-32c7bb3cb0ed/6e6a70ea-4db2-4b59-a2d7-c468f9b8b5a6/b445ea2b-ce97-4fc9-a9bc-efa2f143df72"
-					(reference "C?")
-					(unit 1)
-				)
+					(reference "C88")
+					(unit 1)
+				)

Commit message: Cleanup & Fixes; Changed GPIO; Added Camera; Added Microphone
Parts:
- renumbered C87 to C85, C88 to C86
Changed lines of the file:
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@@
 		(dnp no)
 		(fields_autoplaced yes)
-		(property "Reference" "#PWR0364"
+		(property "Reference" "#PWR0360"
 			(at 173.99 115.57 0)
 			(effects
@@
 			(project "raywatch"
 				(path "/7b654ee8-2a53-4d39-8b7d-32c7bb3cb0ed/6e6a70ea-4db2-4b59-a2d7-c468f9b8b5a6/b445ea2b-ce97-4fc9-a9bc-efa2f143df72"
-					(reference "#PWR0364")
+					(reference "#PWR0360")
 					(unit 1)
 				)
@@
 		(dnp no)
 		(fields_autoplaced yes)
-		(property "Reference" "C87"
+		(property "Reference" "C85"
 			(at 123.19 104.1399 0)
 			(effects
@@
 			(project "raywatch"
 				(path "/7b654ee8-2a53-4d39-8b7d-32c7bb3cb0ed/6e6a70ea-4db2-4b59-a2d7-c468f9b8b5a6/b445ea2b-ce97-4fc9-a9bc-efa2f143df72"
-					(reference "C87")
+					(reference "C85")
 					(unit 1)
 				)
@@
 		(dnp no)
 		(fields_autoplaced yes)
-		(property "Reference" "#PWR0360"
+		(property "Reference" "#PWR0356"
 			(at 127 105.41 0)
 			(effects
@@
 			(project "raywatch"
 				(path "/7b654ee8-2a53-4d39-8b7d-32c7bb3cb0ed/6e6a70ea-4db2-4b59-a2d7-c468f9b8b5a6/b445ea2b-ce97-4fc9-a9bc-efa2f143df72"
-					(reference "#PWR0360")
+					(reference "#PWR0356")
 					(unit 1)
 				)
@@
 		(dnp no)
 		(fields_autoplaced yes)
-		(property "Reference" "#PWR0362"
+		(property "Reference" "#PWR0358"
 			(at 170.18 115.57 0)
 			(effects
@@
 			(project "raywatch"
 				(path "/7b654ee8-2a53-4d39-8b7d-32c7bb3cb0ed/6e6a70ea-4db2-4b59-a2d7-c468f9b8b5a6/b445ea2b-ce97-4fc9-a9bc-efa2f143df72"
-					(reference "#PWR0362")
+					(reference "#PWR0358")
 					(unit 1)
 				)
@@
 		(dnp no)
 		(fields_autoplaced yes)
-		(property "Reference" "#PWR0363"
+		(property "Reference" "#PWR0359"
 			(at 173.99 105.41 0)
 			(effects
@@
 			(project "raywatch"
 				(path "/7b654ee8-2a53-4d39-8b7d-32c7bb3cb0ed/6e6a70ea-4db2-4b59-a2d7-c468f9b8b5a6/b445ea2b-ce97-4fc9-a9bc-efa2f143df72"
-					(reference "#PWR0363")
+					(reference "#PWR0359")
 					(unit 1)
 				)
@@
 		(dnp no)
 		(fields_autoplaced yes)
-		(property "Reference" "#PWR0361"
+		(property "Reference" "#PWR0357"
 			(at 127 115.57 0)
 			(effects
@@
 			(project "raywatch"
 				(path "/7b654ee8-2a53-4d39-8b7d-32c7bb3cb0ed/6e6a70ea-4db2-4b59-a2d7-c468f9b8b5a6/b445ea2b-ce97-4fc9-a9bc-efa2f143df72"
-					(reference "#PWR0361")
+					(reference "#PWR0357")
 					(unit 1)
 				)
@@
 		(dnp no)
 		(fields_autoplaced yes)
-		(property "Reference" "C88"
+		(property "Reference" "C86"
 			(at 177.8 104.1399 0)
 			(effects
@@
 			(project "raywatch"
 				(path "/7b654ee8-2a53-4d39-8b7d-32c7bb3cb0ed/6e6a70ea-4db2-4b59-a2d7-c468f9b8b5a6/b445ea2b-ce97-4fc9-a9bc-efa2f143df72"
-					(reference "C88")
-					(unit 1)
-				)
+					(reference "C86")
+					(unit 1)
+				)

Commit message: Add Light Sensor and Proximity & Gesture Sensor; Changed GPIO
Parts:
- renumbered U26 to U27
Changed lines of the file:
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@@
 		(dnp no)
 		(fields_autoplaced yes)
-		(property "Reference" "U26"
+		(property "Reference" "U27"
 			(at 149.86 91.44 0)
 			(effects
@@
 			(project "raywatch"
 				(path "/7b654ee8-2a53-4d39-8b7d-32c7bb3cb0ed/6e6a70ea-4db2-4b59-a2d7-c468f9b8b5a6/b445ea2b-ce97-4fc9-a9bc-efa2f143df72"
-					(reference "U26")
+					(reference "U27")
 					(unit 1)
 				)
@@
 		(dnp no)
 		(fields_autoplaced yes)
-		(property "Reference" "#PWR0360"
+		(property "Reference" "#PWR0364"
 			(at 173.99 115.57 0)
 			(effects
@@
 			(project "raywatch"
 				(path "/7b654ee8-2a53-4d39-8b7d-32c7bb3cb0ed/6e6a70ea-4db2-4b59-a2d7-c468f9b8b5a6/b445ea2b-ce97-4fc9-a9bc-efa2f143df72"
-					(reference "#PWR0360")
+					(reference "#PWR0364")
 					(unit 1)
 				)
@@
 		(dnp no)
 		(fields_autoplaced yes)
-		(property "Reference" "#PWR0356"
+		(property "Reference" "#PWR0360"
 			(at 127 105.41 0)
 			(effects
@@
 			(project "raywatch"
 				(path "/7b654ee8-2a53-4d39-8b7d-32c7bb3cb0ed/6e6a70ea-4db2-4b59-a2d7-c468f9b8b5a6/b445ea2b-ce97-4fc9-a9bc-efa2f143df72"
-					(reference "#PWR0356")
+					(reference "#PWR0360")
 					(unit 1)
 				)
@@
 		(dnp no)
 		(fields_autoplaced yes)
-		(property "Reference" "#PWR0358"
+		(property "Reference" "#PWR0362"
 			(at 170.18 115.57 0)
 			(effects
@@
 			(project "raywatch"
 				(path "/7b654ee8-2a53-4d39-8b7d-32c7bb3cb0ed/6e6a70ea-4db2-4b59-a2d7-c468f9b8b5a6/b445ea2b-ce97-4fc9-a9bc-efa2f143df72"
-					(reference "#PWR0358")
+					(reference "#PWR0362")
 					(unit 1)
 				)
@@
 		(dnp no)
 		(fields_autoplaced yes)
-		(property "Reference" "#PWR0359"
+		(property "Reference" "#PWR0363"
 			(at 173.99 105.41 0)
 			(effects
@@
 			(project "raywatch"
 				(path "/7b654ee8-2a53-4d39-8b7d-32c7bb3cb0ed/6e6a70ea-4db2-4b59-a2d7-c468f9b8b5a6/b445ea2b-ce97-4fc9-a9bc-efa2f143df72"
-					(reference "#PWR0359")
+					(reference "#PWR0363")
 					(unit 1)
 				)
@@
 		(dnp no)
 		(fields_autoplaced yes)
-		(property "Reference" "#PWR0357"
+		(property "Reference" "#PWR0361"
 			(at 127 115.57 0)
 			(effects
@@
 			(project "raywatch"
 				(path "/7b654ee8-2a53-4d39-8b7d-32c7bb3cb0ed/6e6a70ea-4db2-4b59-a2d7-c468f9b8b5a6/b445ea2b-ce97-4fc9-a9bc-efa2f143df72"
-					(reference "#PWR0357")
-					(unit 1)
-				)
+					(reference "#PWR0361")
+					(unit 1)
+				)

Commit message: Flattend hirachy
Parts:
- renumbered C85 to C70, C86 to C71, U27 to U26
Changed lines of the file:
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@@
 		(dnp no)
 		(fields_autoplaced yes)
-		(property "Reference" "U27"
+		(property "Reference" "U26"
 			(at 149.86 91.44 0)
 			(effects
@@
 		(instances
 			(project "raywatch"
-				(path "/7b654ee8-2a53-4d39-8b7d-32c7bb3cb0ed/6e6a70ea-4db2-4b59-a2d7-c468f9b8b5a6/b445ea2b-ce97-4fc9-a9bc-efa2f143df72"
-					(reference "U27")
+				(path "/7b654ee8-2a53-4d39-8b7d-32c7bb3cb0ed/1d8b2961-678d-411b-851f-e266eaec5e93"
+					(reference "U26")
 					(unit 1)
 				)
@@
 		(dnp no)
 		(fields_autoplaced yes)
-		(property "Reference" "#PWR0364"
+		(property "Reference" "#PWR0352"
 			(at 173.99 115.57 0)
 			(effects
@@
 		(instances
 			(project "raywatch"
-				(path "/7b654ee8-2a53-4d39-8b7d-32c7bb3cb0ed/6e6a70ea-4db2-4b59-a2d7-c468f9b8b5a6/b445ea2b-ce97-4fc9-a9bc-efa2f143df72"
-					(reference "#PWR0364")
+				(path "/7b654ee8-2a53-4d39-8b7d-32c7bb3cb0ed/1d8b2961-678d-411b-851f-e266eaec5e93"
+					(reference "#PWR0352")
 					(unit 1)
 				)
@@
 		(dnp no)
 		(fields_autoplaced yes)
-		(property "Reference" "C85"
+		(property "Reference" "C70"
 			(at 123.19 104.1399 0)
 			(effects
@@
 		(instances
 			(project "raywatch"
-				(path "/7b654ee8-2a53-4d39-8b7d-32c7bb3cb0ed/6e6a70ea-4db2-4b59-a2d7-c468f9b8b5a6/b445ea2b-ce97-4fc9-a9bc-efa2f143df72"
-					(reference "C85")
+				(path "/7b654ee8-2a53-4d39-8b7d-32c7bb3cb0ed/1d8b2961-678d-411b-851f-e266eaec5e93"
+					(reference "C70")
 					(unit 1)
 				)
@@
 		(dnp no)
 		(fields_autoplaced yes)
-		(property "Reference" "#PWR0360"
+		(property "Reference" "#PWR0348"
 			(at 127 105.41 0)
 			(effects
@@
 		(instances
 			(project "raywatch"
-				(path "/7b654ee8-2a53-4d39-8b7d-32c7bb3cb0ed/6e6a70ea-4db2-4b59-a2d7-c468f9b8b5a6/b445ea2b-ce97-4fc9-a9bc-efa2f143df72"
-					(reference "#PWR0360")
+				(path "/7b654ee8-2a53-4d39-8b7d-32c7bb3cb0ed/1d8b2961-678d-411b-851f-e266eaec5e93"
+					(reference "#PWR0348")
 					(unit 1)
 				)
@@
 		(dnp no)
 		(fields_autoplaced yes)
-		(property "Reference" "#PWR0362"
+		(property "Reference" "#PWR0350"
 			(at 170.18 115.57 0)
 			(effects
@@
 		(instances
 			(project "raywatch"
-				(path "/7b654ee8-2a53-4d39-8b7d-32c7bb3cb0ed/6e6a70ea-4db2-4b59-a2d7-c468f9b8b5a6/b445ea2b-ce97-4fc9-a9bc-efa2f143df72"
-					(reference "#PWR0362")
+				(path "/7b654ee8-2a53-4d39-8b7d-32c7bb3cb0ed/1d8b2961-678d-411b-851f-e266eaec5e93"
+					(reference "#PWR0350")
 					(unit 1)
 				)
@@
 		(dnp no)
 		(fields_autoplaced yes)
-		(property "Reference" "#PWR0363"
+		(property "Reference" "#PWR0351"
 			(at 173.99 105.41 0)
 			(effects
@@
 		(instances
 			(project "raywatch"
-				(path "/7b654ee8-2a53-4d39-8b7d-32c7bb3cb0ed/6e6a70ea-4db2-4b59-a2d7-c468f9b8b5a6/b445ea2b-ce97-4fc9-a9bc-efa2f143df72"
-					(reference "#PWR0363")
+				(path "/7b654ee8-2a53-4d39-8b7d-32c7bb3cb0ed/1d8b2961-678d-411b-851f-e266eaec5e93"
+					(reference "#PWR0351")
 					(unit 1)
 				)
@@
 		(dnp no)
 		(fields_autoplaced yes)
-		(property "Reference" "#PWR0361"
+		(property "Reference" "#PWR0349"
 			(at 127 115.57 0)
 			(effects
@@
 		(instances
 			(project "raywatch"
-				(path "/7b654ee8-2a53-4d39-8b7d-32c7bb3cb0ed/6e6a70ea-4db2-4b59-a2d7-c468f9b8b5a6/b445ea2b-ce97-4fc9-a9bc-efa2f143df72"
-					(reference "#PWR0361")
+				(path "/7b654ee8-2a53-4d39-8b7d-32c7bb3cb0ed/1d8b2961-678d-411b-851f-e266eaec5e93"
+					(reference "#PWR0349")
 					(unit 1)
 				)
@@
 		(dnp no)
 		(fields_autoplaced yes)
-		(property "Reference" "C86"
+		(property "Reference" "C71"
 			(at 177.8 104.1399 0)
 			(effects
@@
 		(instances
 			(project "raywatch"
-				(path "/7b654ee8-2a53-4d39-8b7d-32c7bb3cb0ed/6e6a70ea-4db2-4b59-a2d7-c468f9b8b5a6/b445ea2b-ce97-4fc9-a9bc-efa2f143df72"
-					(reference "C86")
-					(unit 1)
-				)
+				(path "/7b654ee8-2a53-4d39-8b7d-32c7bb3cb0ed/1d8b2961-678d-411b-851f-e266eaec5e93"
+					(reference "C71")
+					(unit 1)
+				)

Commit message: Changed footprints from 0603 to 0402
Parts:
- C70, C71: footprint Capacitor_SMD:C_0603_1608Metric -> Capacitor_SMD:C_0504_1310Metric
Changed lines of the file:
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@@
 			)
 		)
-		(property "Footprint" "Capacitor_SMD:C_0603_1608Metric"
+		(property "Footprint" "Capacitor_SMD:C_0504_1310Metric"
 			(at 126.0348 109.22 0)
 			(effects
@@
 			)
 		)
-		(property "Footprint" "Capacitor_SMD:C_0603_1608Metric"
+		(property "Footprint" "Capacitor_SMD:C_0504_1310Metric"
 			(at 174.9552 109.22 0)
 			(effects
