File: src/hardware/battery_gauge.kicad_sch (KiCad schematic)
At the start: 7 parts, among them U34 BQ27426YZFR

Commit message: Flattend hirachy
Parts:
- renumbered C98 to C72, C99 to C73, C100 to C74, R48 to R34, R49 to R35, R50 to R36, U34 to U27
Changed lines of the file:
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@@
 		(dnp no)
 		(fields_autoplaced yes)
-		(property "Reference" "#PWR0406"
+		(property "Reference" "#PWR0361"
 			(at 170.18 97.79 0)
 			(effects
@@
 		(instances
 			(project "raywatch"
-				(path "/7b654ee8-2a53-4d39-8b7d-32c7bb3cb0ed/6e6a70ea-4db2-4b59-a2d7-c468f9b8b5a6/27d482b0-7b63-432c-88d1-098048a1418a"
-					(reference "#PWR0406")
+				(path "/7b654ee8-2a53-4d39-8b7d-32c7bb3cb0ed/354d9a88-ab50-41ba-b40e-476fe78e4ce7"
+					(reference "#PWR0361")
 					(unit 1)
 				)
@@
 		(dnp no)
 		(fields_autoplaced yes)
-		(property "Reference" "R48"
+		(property "Reference" "R34"
 			(at 113.03 116.84 90)
 			(effects
@@
 		(instances
 			(project "raywatch"
-				(path "/7b654ee8-2a53-4d39-8b7d-32c7bb3cb0ed/6e6a70ea-4db2-4b59-a2d7-c468f9b8b5a6/27d482b0-7b63-432c-88d1-098048a1418a"
-					(reference "R48")
+				(path "/7b654ee8-2a53-4d39-8b7d-32c7bb3cb0ed/354d9a88-ab50-41ba-b40e-476fe78e4ce7"
+					(reference "R34")
 					(unit 1)
 				)
@@
 		(dnp no)
 		(fields_autoplaced yes)
-		(property "Reference" "#PWR0404"
+		(property "Reference" "#PWR0359"
 			(at 154.94 118.11 0)
 			(effects
@@
 		(instances
 			(project "raywatch"
-				(path "/7b654ee8-2a53-4d39-8b7d-32c7bb3cb0ed/6e6a70ea-4db2-4b59-a2d7-c468f9b8b5a6/27d482b0-7b63-432c-88d1-098048a1418a"
-					(reference "#PWR0404")
+				(path "/7b654ee8-2a53-4d39-8b7d-32c7bb3cb0ed/354d9a88-ab50-41ba-b40e-476fe78e4ce7"
+					(reference "#PWR0359")
 					(unit 1)
 				)
@@
 		(dnp no)
 		(fields_autoplaced yes)
-		(property "Reference" "U34"
+		(property "Reference" "U27"
 			(at 139.7 83.82 0)
 			(effects
@@
 		(instances
 			(project "raywatch"
-				(path "/7b654ee8-2a53-4d39-8b7d-32c7bb3cb0ed/6e6a70ea-4db2-4b59-a2d7-c468f9b8b5a6/27d482b0-7b63-432c-88d1-098048a1418a"
-					(reference "U34")
+				(path "/7b654ee8-2a53-4d39-8b7d-32c7bb3cb0ed/354d9a88-ab50-41ba-b40e-476fe78e4ce7"
+					(reference "U27")
 					(unit 1)
 				)
@@
 		(dnp no)
 		(fields_autoplaced yes)
-		(property "Reference" "#PWR0399"
+		(property "Reference" "#PWR0356"
 			(at 109.22 107.95 0)
 			(effects
@@
 		(instances
 			(project "raywatch"
-				(path "/7b654ee8-2a53-4d39-8b7d-32c7bb3cb0ed/6e6a70ea-4db2-4b59-a2d7-c468f9b8b5a6/27d482b0-7b63-432c-88d1-098048a1418a"
-					(reference "#PWR0399")
+				(path "/7b654ee8-2a53-4d39-8b7d-32c7bb3cb0ed/354d9a88-ab50-41ba-b40e-476fe78e4ce7"
+					(reference "#PWR0356")
 					(unit 1)
 				)
@@
 		(dnp no)
 		(fields_autoplaced yes)
-		(property "Reference" "C99"
+		(property "Reference" "C73"
 			(at 167.64 80.0099 0)
 			(effects
@@
 		(instances
 			(project "raywatch"
-				(path "/7b654ee8-2a53-4d39-8b7d-32c7bb3cb0ed/6e6a70ea-4db2-4b59-a2d7-c468f9b8b5a6/27d482b0-7b63-432c-88d1-098048a1418a"
-					(reference "C99")
+				(path "/7b654ee8-2a53-4d39-8b7d-32c7bb3cb0ed/354d9a88-ab50-41ba-b40e-476fe78e4ce7"
+					(reference "C73")
 					(unit 1)
 				)
@@
 		(dnp no)
 		(fields_autoplaced yes)
-		(property "Reference" "C98"
+		(property "Reference" "C72"
 			(at 105.41 96.5199 0)
 			(effects
@@
 		(instances
 			(project "raywatch"
-				(path "/7b654ee8-2a53-4d39-8b7d-32c7bb3cb0ed/6e6a70ea-4db2-4b59-a2d7-c468f9b8b5a6/27d482b0-7b63-432c-88d1-098048a1418a"
-					(reference "C98")
+				(path "/7b654ee8-2a53-4d39-8b7d-32c7bb3cb0ed/354d9a88-ab50-41ba-b40e-476fe78e4ce7"
+					(reference "C72")
 					(unit 1)
 				)
@@
 		(dnp no)
 		(fields_autoplaced yes)
-		(property "Reference" "#PWR0401"
+		(property "Reference" "#PWR0358"
 			(at 121.92 125.73 0)
 			(effects
@@
 		(instances
 			(project "raywatch"
-				(path "/7b654ee8-2a53-4d39-8b7d-32c7bb3cb0ed/6e6a70ea-4db2-4b59-a2d7-c468f9b8b5a6/27d482b0-7b63-432c-88d1-098048a1418a"
-					(reference "#PWR0401")
+				(path "/7b654ee8-2a53-4d39-8b7d-32c7bb3cb0ed/354d9a88-ab50-41ba-b40e-476fe78e4ce7"
+					(reference "#PWR0358")
 					(unit 1)
 				)
@@
 		(dnp no)
 		(fields_autoplaced yes)
-		(property "Reference" "#PWR0400"
+		(property "Reference" "#PWR0357"
 			(at 109.22 116.84 0)
 			(effects
@@
 		(instances
 			(project "raywatch"
-				(path "/7b654ee8-2a53-4d39-8b7d-32c7bb3cb0ed/6e6a70ea-4db2-4b59-a2d7-c468f9b8b5a6/27d482b0-7b63-432c-88d1-098048a1418a"
-					(reference "#PWR0400")
+				(path "/7b654ee8-2a53-4d39-8b7d-32c7bb3cb0ed/354d9a88-ab50-41ba-b40e-476fe78e4ce7"
+					(reference "#PWR0357")
 					(unit 1)
 				)
@@
 		(dnp no)
 		(fields_autoplaced yes)
-		(property "Reference" "#PWR0408"
+		(property "Reference" "#PWR0363"
 			(at 176.53 81.28 0)
 			(effects
@@
 		(instances
 			(project "raywatch"
-				(path "/7b654ee8-2a53-4d39-8b7d-32c7bb3cb0ed/6e6a70ea-4db2-4b59-a2d7-c468f9b8b5a6/27d482b0-7b63-432c-88d1-098048a1418a"
-					(reference "#PWR0408")
+				(path "/7b654ee8-2a53-4d39-8b7d-32c7bb3cb0ed/354d9a88-ab50-41ba-b40e-476fe78e4ce7"
+					(reference "#PWR0363")
 					(unit 1)
 				)
@@
 		(dnp no)
 		(fields_autoplaced yes)
-		(property "Reference" "#PWR0407"
+		(property "Reference" "#PWR0362"
 			(at 170.18 97.79 0)
 			(effects
@@
 		(instances
 			(project "raywatch"
-				(path "/7b654ee8-2a53-4d39-8b7d-32c7bb3cb0ed/6e6a70ea-4db2-4b59-a2d7-c468f9b8b5a6/27d482b0-7b63-432c-88d1-098048a1418a"
-					(reference "#PWR0407")
+				(path "/7b654ee8-2a53-4d39-8b7d-32c7bb3cb0ed/354d9a88-ab50-41ba-b40e-476fe78e4ce7"
+					(reference "#PWR0362")
 					(unit 1)
 				)
@@
 		(dnp no)
 		(fields_autoplaced yes)
-		(property "Reference" "#PWR0409"
+		(property "Reference" "#PWR0364"
 			(at 176.53 91.44 0)
 			(effects
@@
 		(instances
 			(project "raywatch"
-				(path "/7b654ee8-2a53-4d39-8b7d-32c7bb3cb0ed/6e6a70ea-4db2-4b59-a2d7-c468f9b8b5a6/27d482b0-7b63-432c-88d1-098048a1418a"
-					(reference "#PWR0409")
+				(path "/7b654ee8-2a53-4d39-8b7d-32c7bb3cb0ed/354d9a88-ab50-41ba-b40e-476fe78e4ce7"
+					(reference "#PWR0364")
 					(unit 1)
 				)
@@
 		(dnp no)
 		(fields_autoplaced yes)
-		(property "Reference" "#PWR0405"
+		(property "Reference" "#PWR0360"
 			(at 163.83 91.44 0)
 			(effects
@@
 		(instances
 			(project "raywatch"
-				(path "/7b654ee8-2a53-4d39-8b7d-32c7bb3cb0ed/6e6a70ea-4db2-4b59-a2d7-c468f9b8b5a6/27d482b0-7b63-432c-88d1-098048a1418a"
-					(reference "#PWR0405")
+				(path "/7b654ee8-2a53-4d39-8b7d-32c7bb3cb0ed/354d9a88-ab50-41ba-b40e-476fe78e4ce7"
+					(reference "#PWR0360")
 					(unit 1)
 				)
@@
 		(dnp no)
 		(fields_autoplaced yes)
-		(property "Reference" "R50"
+		(property "Reference" "R36"
 			(at 172.72 96.5199 0)
 			(effects
@@
 		(instances
 			(project "raywatch"
-				(path "/7b654ee8-2a53-4d39-8b7d-32c7bb3cb0ed/6e6a70ea-4db2-4b59-a2d7-c468f9b8b5a6/27d482b0-7b63-432c-88d1-098048a1418a"
-					(reference "R50")
+				(path "/7b654ee8-2a53-4d39-8b7d-32c7bb3cb0ed/354d9a88-ab50-41ba-b40e-476fe78e4ce7"
+					(reference "R36")
 					(unit 1)
 				)
@@
 		(dnp no)
 		(fields_autoplaced yes)
-		(property "Reference" "R49"
+		(property "Reference" "R35"
 			(at 124.46 114.2999 0)
 			(effects
@@
 		(instances
 			(project "raywatch"
-				(path "/7b654ee8-2a53-4d39-8b7d-32c7bb3cb0ed/6e6a70ea-4db2-4b59-a2d7-c468f9b8b5a6/27d482b0-7b63-432c-88d1-098048a1418a"
-					(reference "R49")
+				(path "/7b654ee8-2a53-4d39-8b7d-32c7bb3cb0ed/354d9a88-ab50-41ba-b40e-476fe78e4ce7"
+					(reference "R35")
 					(unit 1)
 				)
@@
 		(dnp no)
 		(fields_autoplaced yes)
-		(property "Reference" "C100"
+		(property "Reference" "C74"
 			(at 180.34 80.0099 0)
 			(effects
@@
 		(instances
 			(project "raywatch"
-				(path "/7b654ee8-2a53-4d39-8b7d-32c7bb3cb0ed/6e6a70ea-4db2-4b59-a2d7-c468f9b8b5a6/27d482b0-7b63-432c-88d1-098048a1418a"
-					(reference "C100")
+				(path "/7b654ee8-2a53-4d39-8b7d-32c7bb3cb0ed/354d9a88-ab50-41ba-b40e-476fe78e4ce7"
+					(reference "C74")
 					(unit 1)
 				)
@@
 		(dnp no)
 		(fields_autoplaced yes)
-		(property "Reference" "#PWR0398"
+		(property "Reference" "#PWR0355"
 			(at 109.22 97.79 0)
 			(effects
@@
 		(instances
 			(project "raywatch"
-				(path "/7b654ee8-2a53-4d39-8b7d-32c7bb3cb0ed/6e6a70ea-4db2-4b59-a2d7-c468f9b8b5a6/27d482b0-7b63-432c-88d1-098048a1418a"
-					(reference "#PWR0398")
-					(unit 1)
-				)
+				(path "/7b654ee8-2a53-4d39-8b7d-32c7bb3cb0ed/354d9a88-ab50-41ba-b40e-476fe78e4ce7"
+					(reference "#PWR0355")
+					(unit 1)
+				)

Commit message: Changed footprints from 0603 to 0402
Parts:
- C72, C73, C74: footprint Capacitor_SMD:C_0603_1608Metric -> Capacitor_SMD:C_0504_1310Metric
- R34, R35, R36: footprint Resistor_SMD:R_0603_1608Metric -> Resistor_SMD:R_0402_1005Metric
Changed lines of the file:
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@@
 			)
 		)
-		(property "Footprint" "Resistor_SMD:R_0603_1608Metric"
+		(property "Footprint" "Resistor_SMD:R_0402_1005Metric"
 			(at 113.03 111.252 90)
 			(effects
@@
 			)
 		)
-		(property "Footprint" "Capacitor_SMD:C_0603_1608Metric"
+		(property "Footprint" "Capacitor_SMD:C_0504_1310Metric"
 			(at 164.7952 77.47 0)
 			(effects
@@
 			)
 		)
-		(property "Footprint" "Capacitor_SMD:C_0603_1608Metric"
+		(property "Footprint" "Capacitor_SMD:C_0504_1310Metric"
 			(at 108.2548 93.98 0)
 			(effects
@@
 			)
 		)
-		(property "Footprint" "Resistor_SMD:R_0603_1608Metric"
+		(property "Footprint" "Resistor_SMD:R_0402_1005Metric"
 			(at 168.402 97.79 90)
 			(effects
@@
 			)
 		)
-		(property "Footprint" "Resistor_SMD:R_0603_1608Metric"
+		(property "Footprint" "Resistor_SMD:R_0402_1005Metric"
 			(at 123.698 115.57 90)
 			(effects
@@
 			)
 		)
-		(property "Footprint" "Capacitor_SMD:C_0603_1608Metric"
+		(property "Footprint" "Capacitor_SMD:C_0504_1310Metric"
 			(at 177.4952 77.47 0)
 			(effects
