File: src/hardware/3v0_converter.kicad_sch (KiCad schematic)
At the start: 0 parts

Commit message: Added 3.0V Converter
Parts:
- added C? (x2): 1µF, symbol Device:C
- added U?: TPS7A2030PDQNR, TPS7A2030PDQNR:VREG_TPS7A2030PDQNR, symbol TPS7A2030PDQNR:TPS7A2030PDQNR
Connections:
- new net +3V0: C?.1, U?.1 (OUT)
- new net 3VEN: U?.3 (EN)
- new net GND: C?.2, C?.2, U?.2 (GND), U?.5 (EXP)
- new net VSYS: C?.1, U?.4 (IN)

Commit message: Cleanup & Fixes; Added footprints; Removed Light sensors
Parts:
- C89, C90: renamed from C?; footprint (none) -> Capacitor_SMD:C_0603_1608Metric
- U27: renamed from U?; footprint TPS7A2030PDQNR:VREG_TPS7A2030PDQNR -> Project:VREG_TPS7A2030PDQNR
Changed lines of the file:
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@@
 		(dnp no)
 		(fields_autoplaced yes)
-		(property "Reference" "U?"
+		(property "Reference" "U27"
 			(at 152.4 88.9 0)
 			(effects
@@
 			)
 		)
-		(property "Footprint" "TPS7A2030PDQNR:VREG_TPS7A2030PDQNR"
+		(property "Footprint" "Project:VREG_TPS7A2030PDQNR"
 			(at 152.4 101.6 0)
 			(effects
@@
 			(project "raywatch"
 				(path "/7b654ee8-2a53-4d39-8b7d-32c7bb3cb0ed/6e6a70ea-4db2-4b59-a2d7-c468f9b8b5a6/965e2c2b-77bd-439d-8b14-adaa270f722d"
-					(reference "U?")
+					(reference "U27")
 					(unit 1)
 				)
@@
 		(dnp no)
 		(fields_autoplaced yes)
-		(property "Reference" "#PWR0388"
+		(property "Reference" "#PWR0366"
 			(at 129.54 110.49 0)
 			(effects
@@
 			(project "raywatch"
 				(path "/7b654ee8-2a53-4d39-8b7d-32c7bb3cb0ed/6e6a70ea-4db2-4b59-a2d7-c468f9b8b5a6/965e2c2b-77bd-439d-8b14-adaa270f722d"
-					(reference "#PWR0388")
+					(reference "#PWR0366")
 					(unit 1)
 				)
@@
 		(dnp no)
 		(fields_autoplaced yes)
-		(property "Reference" "#PWR0390"
+		(property "Reference" "#PWR0368"
 			(at 165.1 113.03 0)
 			(effects
@@
 			(project "raywatch"
 				(path "/7b654ee8-2a53-4d39-8b7d-32c7bb3cb0ed/6e6a70ea-4db2-4b59-a2d7-c468f9b8b5a6/965e2c2b-77bd-439d-8b14-adaa270f722d"
-					(reference "#PWR0390")
+					(reference "#PWR0368")
 					(unit 1)
 				)
@@
 		(dnp no)
 		(fields_autoplaced yes)
-		(property "Reference" "C?"
+		(property "Reference" "C90"
 			(at 168.91 99.0599 0)
 			(effects
@@
 			)
 		)
-		(property "Footprint" ""
+		(property "Footprint" "Capacitor_SMD:C_0603_1608Metric"
 			(at 166.0652 104.14 0)
 			(effects
@@
 			(project "raywatch"
 				(path "/7b654ee8-2a53-4d39-8b7d-32c7bb3cb0ed/6e6a70ea-4db2-4b59-a2d7-c468f9b8b5a6/965e2c2b-77bd-439d-8b14-adaa270f722d"
-					(reference "C?")
+					(reference "C90")
 					(unit 1)
 				)
@@
 		(dnp no)
 		(fields_autoplaced yes)
-		(property "Reference" "#PWR0389"
+		(property "Reference" "#PWR0367"
 			(at 165.1 100.33 0)
 			(effects
@@
 			(project "raywatch"
 				(path "/7b654ee8-2a53-4d39-8b7d-32c7bb3cb0ed/6e6a70ea-4db2-4b59-a2d7-c468f9b8b5a6/965e2c2b-77bd-439d-8b14-adaa270f722d"
-					(reference "#PWR0389")
+					(reference "#PWR0367")
 					(unit 1)
 				)
@@
 		(dnp no)
 		(fields_autoplaced yes)
-		(property "Reference" "#PWR0387"
+		(property "Reference" "#PWR0365"
 			(at 129.54 100.33 0)
 			(effects
@@
 			(project "raywatch"
 				(path "/7b654ee8-2a53-4d39-8b7d-32c7bb3cb0ed/6e6a70ea-4db2-4b59-a2d7-c468f9b8b5a6/965e2c2b-77bd-439d-8b14-adaa270f722d"
-					(reference "#PWR0387")
+					(reference "#PWR0365")
 					(unit 1)
 				)
@@
 		(dnp no)
 		(fields_autoplaced yes)
-		(property "Reference" "C?"
+		(property "Reference" "C89"
 			(at 125.73 99.0599 0)
 			(effects
@@
 			)
 		)
-		(property "Footprint" ""
+		(property "Footprint" "Capacitor_SMD:C_0603_1608Metric"
 			(at 128.5748 104.14 0)
 			(effects
@@
 			(project "raywatch"
 				(path "/7b654ee8-2a53-4d39-8b7d-32c7bb3cb0ed/6e6a70ea-4db2-4b59-a2d7-c468f9b8b5a6/965e2c2b-77bd-439d-8b14-adaa270f722d"
-					(reference "C?")
+					(reference "C89")
 					(unit 1)
 				)

Commit message: Cleanup & Fixes; Changed GPIO; Added Camera; Added Microphone
Parts:
- renumbered C89 to C87, C90 to C88
Changed lines of the file:
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@@
 		(dnp no)
 		(fields_autoplaced yes)
-		(property "Reference" "#PWR0366"
+		(property "Reference" "#PWR0362"
 			(at 129.54 110.49 0)
 			(effects
@@
 			(project "raywatch"
 				(path "/7b654ee8-2a53-4d39-8b7d-32c7bb3cb0ed/6e6a70ea-4db2-4b59-a2d7-c468f9b8b5a6/965e2c2b-77bd-439d-8b14-adaa270f722d"
-					(reference "#PWR0366")
+					(reference "#PWR0362")
 					(unit 1)
 				)
@@
 		(dnp no)
 		(fields_autoplaced yes)
-		(property "Reference" "#PWR0368"
+		(property "Reference" "#PWR0364"
 			(at 165.1 113.03 0)
 			(effects
@@
 			(project "raywatch"
 				(path "/7b654ee8-2a53-4d39-8b7d-32c7bb3cb0ed/6e6a70ea-4db2-4b59-a2d7-c468f9b8b5a6/965e2c2b-77bd-439d-8b14-adaa270f722d"
-					(reference "#PWR0368")
+					(reference "#PWR0364")
 					(unit 1)
 				)
@@
 		(dnp no)
 		(fields_autoplaced yes)
-		(property "Reference" "C90"
+		(property "Reference" "C88"
 			(at 168.91 99.0599 0)
 			(effects
@@
 			(project "raywatch"
 				(path "/7b654ee8-2a53-4d39-8b7d-32c7bb3cb0ed/6e6a70ea-4db2-4b59-a2d7-c468f9b8b5a6/965e2c2b-77bd-439d-8b14-adaa270f722d"
-					(reference "C90")
+					(reference "C88")
 					(unit 1)
 				)
@@
 		(dnp no)
 		(fields_autoplaced yes)
-		(property "Reference" "#PWR0367"
+		(property "Reference" "#PWR0363"
 			(at 165.1 100.33 0)
 			(effects
@@
 			(project "raywatch"
 				(path "/7b654ee8-2a53-4d39-8b7d-32c7bb3cb0ed/6e6a70ea-4db2-4b59-a2d7-c468f9b8b5a6/965e2c2b-77bd-439d-8b14-adaa270f722d"
-					(reference "#PWR0367")
+					(reference "#PWR0363")
 					(unit 1)
 				)
@@
 		(dnp no)
 		(fields_autoplaced yes)
-		(property "Reference" "#PWR0365"
+		(property "Reference" "#PWR0361"
 			(at 129.54 100.33 0)
 			(effects
@@
 			(project "raywatch"
 				(path "/7b654ee8-2a53-4d39-8b7d-32c7bb3cb0ed/6e6a70ea-4db2-4b59-a2d7-c468f9b8b5a6/965e2c2b-77bd-439d-8b14-adaa270f722d"
-					(reference "#PWR0365")
+					(reference "#PWR0361")
 					(unit 1)
 				)
@@
 		(dnp no)
 		(fields_autoplaced yes)
-		(property "Reference" "C89"
+		(property "Reference" "C87"
 			(at 125.73 99.0599 0)
 			(effects
@@
 			(project "raywatch"
 				(path "/7b654ee8-2a53-4d39-8b7d-32c7bb3cb0ed/6e6a70ea-4db2-4b59-a2d7-c468f9b8b5a6/965e2c2b-77bd-439d-8b14-adaa270f722d"
-					(reference "C89")
-					(unit 1)
-				)
+					(reference "C87")
+					(unit 1)
+				)

Commit message: Add Light Sensor and Proximity & Gesture Sensor; Changed GPIO
Parts:
- renumbered U27 to U28
Changed lines of the file:
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@@
 		(dnp no)
 		(fields_autoplaced yes)
-		(property "Reference" "U27"
+		(property "Reference" "U28"
 			(at 152.4 88.9 0)
 			(effects
@@
 			(project "raywatch"
 				(path "/7b654ee8-2a53-4d39-8b7d-32c7bb3cb0ed/6e6a70ea-4db2-4b59-a2d7-c468f9b8b5a6/965e2c2b-77bd-439d-8b14-adaa270f722d"
-					(reference "U27")
+					(reference "U28")
 					(unit 1)
 				)
@@
 		(dnp no)
 		(fields_autoplaced yes)
-		(property "Reference" "#PWR0362"
+		(property "Reference" "#PWR0366"
 			(at 129.54 110.49 0)
 			(effects
@@
 			(project "raywatch"
 				(path "/7b654ee8-2a53-4d39-8b7d-32c7bb3cb0ed/6e6a70ea-4db2-4b59-a2d7-c468f9b8b5a6/965e2c2b-77bd-439d-8b14-adaa270f722d"
-					(reference "#PWR0362")
+					(reference "#PWR0366")
 					(unit 1)
 				)
@@
 		(dnp no)
 		(fields_autoplaced yes)
-		(property "Reference" "#PWR0364"
+		(property "Reference" "#PWR0368"
 			(at 165.1 113.03 0)
 			(effects
@@
 			(project "raywatch"
 				(path "/7b654ee8-2a53-4d39-8b7d-32c7bb3cb0ed/6e6a70ea-4db2-4b59-a2d7-c468f9b8b5a6/965e2c2b-77bd-439d-8b14-adaa270f722d"
-					(reference "#PWR0364")
+					(reference "#PWR0368")
 					(unit 1)
 				)
@@
 		(dnp no)
 		(fields_autoplaced yes)
-		(property "Reference" "#PWR0363"
+		(property "Reference" "#PWR0367"
 			(at 165.1 100.33 0)
 			(effects
@@
 			(project "raywatch"
 				(path "/7b654ee8-2a53-4d39-8b7d-32c7bb3cb0ed/6e6a70ea-4db2-4b59-a2d7-c468f9b8b5a6/965e2c2b-77bd-439d-8b14-adaa270f722d"
-					(reference "#PWR0363")
+					(reference "#PWR0367")
 					(unit 1)
 				)
@@
 		(dnp no)
 		(fields_autoplaced yes)
-		(property "Reference" "#PWR0361"
+		(property "Reference" "#PWR0365"
 			(at 129.54 100.33 0)
 			(effects
@@
 			(project "raywatch"
 				(path "/7b654ee8-2a53-4d39-8b7d-32c7bb3cb0ed/6e6a70ea-4db2-4b59-a2d7-c468f9b8b5a6/965e2c2b-77bd-439d-8b14-adaa270f722d"
-					(reference "#PWR0361")
+					(reference "#PWR0365")
 					(unit 1)
 				)

Commit message: Flattend hirachy
Parts:
- renumbered C87 to C68, C88 to C69, U28 to U25
Changed lines of the file:
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@@
 		(dnp no)
 		(fields_autoplaced yes)
-		(property "Reference" "U28"
+		(property "Reference" "U25"
 			(at 152.4 88.9 0)
 			(effects
@@
 		(instances
 			(project "raywatch"
-				(path "/7b654ee8-2a53-4d39-8b7d-32c7bb3cb0ed/6e6a70ea-4db2-4b59-a2d7-c468f9b8b5a6/965e2c2b-77bd-439d-8b14-adaa270f722d"
-					(reference "U28")
+				(path "/7b654ee8-2a53-4d39-8b7d-32c7bb3cb0ed/2714add3-2889-4ca2-9511-f797ac8197f4"
+					(reference "U25")
 					(unit 1)
 				)
@@
 		(dnp no)
 		(fields_autoplaced yes)
-		(property "Reference" "#PWR0366"
+		(property "Reference" "#PWR0345"
 			(at 129.54 110.49 0)
 			(effects
@@
 		(instances
 			(project "raywatch"
-				(path "/7b654ee8-2a53-4d39-8b7d-32c7bb3cb0ed/6e6a70ea-4db2-4b59-a2d7-c468f9b8b5a6/965e2c2b-77bd-439d-8b14-adaa270f722d"
-					(reference "#PWR0366")
+				(path "/7b654ee8-2a53-4d39-8b7d-32c7bb3cb0ed/2714add3-2889-4ca2-9511-f797ac8197f4"
+					(reference "#PWR0345")
 					(unit 1)
 				)
@@
 		(dnp no)
 		(fields_autoplaced yes)
-		(property "Reference" "#PWR0368"
+		(property "Reference" "#PWR0347"
 			(at 165.1 113.03 0)
 			(effects
@@
 		(instances
 			(project "raywatch"
-				(path "/7b654ee8-2a53-4d39-8b7d-32c7bb3cb0ed/6e6a70ea-4db2-4b59-a2d7-c468f9b8b5a6/965e2c2b-77bd-439d-8b14-adaa270f722d"
-					(reference "#PWR0368")
+				(path "/7b654ee8-2a53-4d39-8b7d-32c7bb3cb0ed/2714add3-2889-4ca2-9511-f797ac8197f4"
+					(reference "#PWR0347")
 					(unit 1)
 				)
@@
 		(dnp no)
 		(fields_autoplaced yes)
-		(property "Reference" "C88"
+		(property "Reference" "C69"
 			(at 168.91 99.0599 0)
 			(effects
@@
 		(instances
 			(project "raywatch"
-				(path "/7b654ee8-2a53-4d39-8b7d-32c7bb3cb0ed/6e6a70ea-4db2-4b59-a2d7-c468f9b8b5a6/965e2c2b-77bd-439d-8b14-adaa270f722d"
-					(reference "C88")
+				(path "/7b654ee8-2a53-4d39-8b7d-32c7bb3cb0ed/2714add3-2889-4ca2-9511-f797ac8197f4"
+					(reference "C69")
 					(unit 1)
 				)
@@
 		(dnp no)
 		(fields_autoplaced yes)
-		(property "Reference" "#PWR0367"
+		(property "Reference" "#PWR0346"
 			(at 165.1 100.33 0)
 			(effects
@@
 		(instances
 			(project "raywatch"
-				(path "/7b654ee8-2a53-4d39-8b7d-32c7bb3cb0ed/6e6a70ea-4db2-4b59-a2d7-c468f9b8b5a6/965e2c2b-77bd-439d-8b14-adaa270f722d"
-					(reference "#PWR0367")
+				(path "/7b654ee8-2a53-4d39-8b7d-32c7bb3cb0ed/2714add3-2889-4ca2-9511-f797ac8197f4"
+					(reference "#PWR0346")
 					(unit 1)
 				)
@@
 		(dnp no)
 		(fields_autoplaced yes)
-		(property "Reference" "#PWR0365"
+		(property "Reference" "#PWR0344"
 			(at 129.54 100.33 0)
 			(effects
@@
 		(instances
 			(project "raywatch"
-				(path "/7b654ee8-2a53-4d39-8b7d-32c7bb3cb0ed/6e6a70ea-4db2-4b59-a2d7-c468f9b8b5a6/965e2c2b-77bd-439d-8b14-adaa270f722d"
-					(reference "#PWR0365")
+				(path "/7b654ee8-2a53-4d39-8b7d-32c7bb3cb0ed/2714add3-2889-4ca2-9511-f797ac8197f4"
+					(reference "#PWR0344")
 					(unit 1)
 				)
@@
 		(dnp no)
 		(fields_autoplaced yes)
-		(property "Reference" "C87"
+		(property "Reference" "C68"
 			(at 125.73 99.0599 0)
 			(effects
@@
 		(instances
 			(project "raywatch"
-				(path "/7b654ee8-2a53-4d39-8b7d-32c7bb3cb0ed/6e6a70ea-4db2-4b59-a2d7-c468f9b8b5a6/965e2c2b-77bd-439d-8b14-adaa270f722d"
-					(reference "C87")
+				(path "/7b654ee8-2a53-4d39-8b7d-32c7bb3cb0ed/2714add3-2889-4ca2-9511-f797ac8197f4"
+					(reference "C68")
 					(unit 1)
 				)

Commit message: Changed footprints from 0603 to 0402
Parts:
- C68, C69: footprint Capacitor_SMD:C_0603_1608Metric -> Capacitor_SMD:C_0504_1310Metric
Changed lines of the file:
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@@
 			)
 		)
-		(property "Footprint" "Capacitor_SMD:C_0603_1608Metric"
+		(property "Footprint" "Capacitor_SMD:C_0504_1310Metric"
 			(at 166.0652 104.14 0)
 			(effects
@@
 			)
 		)
-		(property "Footprint" "Capacitor_SMD:C_0603_1608Metric"
+		(property "Footprint" "Capacitor_SMD:C_0504_1310Metric"
 			(at 128.5748 104.14 0)
 			(effects

Commit message: Replaced global labels with pin headers
Parts:
- added J27: Conn_01x02_Pin, symbol Connector:Conn_01x02_Pin
- added J96: Conn_02x08_Top_Bottom, symbol Connector_Generic:Conn_02x08_Top_Bottom
- added J98: Conn_01x01_Pin, symbol Connector:Conn_01x01_Pin
Connections:
- net +3V0: now also J96.1 (Pin_1), J96.2 (Pin_2), J96.3 (Pin_3), J96.4 (Pin_4), J96.5 (Pin_5), J96.6 (Pin_6), J96.7 (Pin_7), J96.8 (Pin_8)
- net 3VEN: now also J98.1 (Pin_1)
- net GND: now also J27.2 (Pin_2), J96.10 (Pin_10), J96.11 (Pin_11), J96.12 (Pin_12), J96.13 (Pin_13), J96.14 (Pin_14), J96.15 (Pin_15), J96.16 (Pin_16), J96.9 (Pin_9)
- net VSYS: now also J27.1 (Pin_1)
