File: src/hardware/3v0_converter.kicad_sch (KiCad schematic)
At the start: 6 parts, among them J27 Conn_01x02_Pin, J96 Conn_02x08_Top_Bottom, J98 Conn_01x01_Pin, U25 TPS7A2030PDQNR

Commit message: Reannotated schematic
Parts:
- renumbered C68 to C63, C69 to C64, J27 to J71, J98 to J72, J96 to J73, U25 to U26
Changed lines of the file:
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@@
 		(dnp no)
 		(fields_autoplaced yes)
-		(property "Reference" "#PWR0458"
+		(property "Reference" "#PWR0372"
 			(at 127 64.77 0)
 			(effects
@@
 			(project "raywatch"
 				(path "/7b654ee8-2a53-4d39-8b7d-32c7bb3cb0ed/2714add3-2889-4ca2-9511-f797ac8197f4"
-					(reference "#PWR0458")
+					(reference "#PWR0372")
 					(unit 1)
 				)
@@
 		(dnp no)
 		(fields_autoplaced yes)
-		(property "Reference" "U25"
+		(property "Reference" "U26"
 			(at 152.4 88.9 0)
 			(effects
@@
 			(project "raywatch"
 				(path "/7b654ee8-2a53-4d39-8b7d-32c7bb3cb0ed/2714add3-2889-4ca2-9511-f797ac8197f4"
-					(reference "U25")
+					(reference "U26")
 					(unit 1)
 				)
@@
 		(dnp no)
 		(fields_autoplaced yes)
-		(property "Reference" "#PWR0345"
+		(property "Reference" "#PWR0374"
 			(at 129.54 110.49 0)
 			(effects
@@
 			(project "raywatch"
 				(path "/7b654ee8-2a53-4d39-8b7d-32c7bb3cb0ed/2714add3-2889-4ca2-9511-f797ac8197f4"
-					(reference "#PWR0345")
+					(reference "#PWR0374")
 					(unit 1)
 				)
@@
 		(dnp no)
 		(fields_autoplaced yes)
-		(property "Reference" "#PWR0347"
+		(property "Reference" "#PWR0377"
 			(at 165.1 113.03 0)
 			(effects
@@
 			(project "raywatch"
 				(path "/7b654ee8-2a53-4d39-8b7d-32c7bb3cb0ed/2714add3-2889-4ca2-9511-f797ac8197f4"
-					(reference "#PWR0347")
+					(reference "#PWR0377")
 					(unit 1)
 				)
@@
 		(dnp no)
 		(fields_autoplaced yes)
-		(property "Reference" "J27"
+		(property "Reference" "J71"
 			(at 114.3 62.2299 0)
 			(effects
@@
 			(project "raywatch"
 				(path "/7b654ee8-2a53-4d39-8b7d-32c7bb3cb0ed/2714add3-2889-4ca2-9511-f797ac8197f4"
-					(reference "J27")
+					(reference "J71")
 					(unit 1)
 				)
@@
 		(dnp no)
 		(fields_autoplaced yes)
-		(property "Reference" "C69"
+		(property "Reference" "C64"
 			(at 168.91 99.0599 0)
 			(effects
@@
 			(project "raywatch"
 				(path "/7b654ee8-2a53-4d39-8b7d-32c7bb3cb0ed/2714add3-2889-4ca2-9511-f797ac8197f4"
-					(reference "C69")
+					(reference "C64")
 					(unit 1)
 				)
@@
 		(dnp no)
 		(fields_autoplaced yes)
-		(property "Reference" "#PWR0457"
+		(property "Reference" "#PWR0371"
 			(at 116.84 62.23 0)
 			(effects
@@
 			(project "raywatch"
 				(path "/7b654ee8-2a53-4d39-8b7d-32c7bb3cb0ed/2714add3-2889-4ca2-9511-f797ac8197f4"
-					(reference "#PWR0457")
+					(reference "#PWR0371")
 					(unit 1)
 				)
@@
 		(dnp no)
 		(fields_autoplaced yes)
-		(property "Reference" "#PWR064"
+		(property "Reference" "#PWR0378"
 			(at 166.37 77.47 0)
 			(effects
@@
 			(project "raywatch"
 				(path "/7b654ee8-2a53-4d39-8b7d-32c7bb3cb0ed/2714add3-2889-4ca2-9511-f797ac8197f4"
-					(reference "#PWR064")
+					(reference "#PWR0378")
 					(unit 1)
 				)
@@
 		(dnp no)
 		(fields_autoplaced yes)
-		(property "Reference" "J96"
+		(property "Reference" "J73"
 			(at 160.02 46.99 0)
 			(effects
@@
 			(project "raywatch"
 				(path "/7b654ee8-2a53-4d39-8b7d-32c7bb3cb0ed/2714add3-2889-4ca2-9511-f797ac8197f4"
-					(reference "J96")
+					(reference "J73")
 					(unit 1)
 				)
@@
 		(dnp no)
 		(fields_autoplaced yes)
-		(property "Reference" "#PWR063"
+		(property "Reference" "#PWR0375"
 			(at 153.67 67.31 0)
 			(effects
@@
 			(project "raywatch"
 				(path "/7b654ee8-2a53-4d39-8b7d-32c7bb3cb0ed/2714add3-2889-4ca2-9511-f797ac8197f4"
-					(reference "#PWR063")
+					(reference "#PWR0375")
 					(unit 1)
 				)
@@
 		(dnp no)
 		(fields_autoplaced yes)
-		(property "Reference" "J98"
+		(property "Reference" "J72"
 			(at 116.205 71.12 0)
 			(effects
@@
 			(project "raywatch"
 				(path "/7b654ee8-2a53-4d39-8b7d-32c7bb3cb0ed/2714add3-2889-4ca2-9511-f797ac8197f4"
-					(reference "J98")
+					(reference "J72")
 					(unit 1)
 				)
@@
 		(dnp no)
 		(fields_autoplaced yes)
-		(property "Reference" "#PWR0346"
+		(property "Reference" "#PWR0376"
 			(at 165.1 100.33 0)
 			(effects
@@
 			(project "raywatch"
 				(path "/7b654ee8-2a53-4d39-8b7d-32c7bb3cb0ed/2714add3-2889-4ca2-9511-f797ac8197f4"
-					(reference "#PWR0346")
+					(reference "#PWR0376")
 					(unit 1)
 				)
@@
 		(dnp no)
 		(fields_autoplaced yes)
-		(property "Reference" "#PWR0344"
+		(property "Reference" "#PWR0373"
 			(at 129.54 100.33 0)
 			(effects
@@
 			(project "raywatch"
 				(path "/7b654ee8-2a53-4d39-8b7d-32c7bb3cb0ed/2714add3-2889-4ca2-9511-f797ac8197f4"
-					(reference "#PWR0344")
+					(reference "#PWR0373")
 					(unit 1)
 				)
@@
 		(dnp no)
 		(fields_autoplaced yes)
-		(property "Reference" "C68"
+		(property "Reference" "C63"
 			(at 125.73 99.0599 0)
 			(effects
@@
 			(project "raywatch"
 				(path "/7b654ee8-2a53-4d39-8b7d-32c7bb3cb0ed/2714add3-2889-4ca2-9511-f797ac8197f4"
-					(reference "C68")
-					(unit 1)
-				)
+					(reference "C63")
+					(unit 1)
+				)

Commit message: Assigned pin header footprints
Parts:
- J71: footprint (none) -> Connector_PinHeader_2.54mm:PinHeader_1x02_P2.54mm_Horizontal
- J72: footprint (none) -> Connector_PinHeader_2.54mm:PinHeader_1x01_P2.54mm_Horizontal
- J73: footprint (none) -> Connector_PinHeader_2.54mm:PinHeader_1x16_P2.54mm_Vertical
Changed lines of the file:
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@@
 			)
 		)
-		(property "Footprint" ""
+		(property "Footprint" "Connector_PinHeader_2.54mm:PinHeader_1x02_P2.54mm_Horizontal"
 			(at 115.57 62.23 0)
 			(effects
@@
 			)
 		)
-		(property "Footprint" ""
+		(property "Footprint" "Connector_PinHeader_2.54mm:PinHeader_1x16_P2.54mm_Vertical"
 			(at 158.75 60.96 0)
 			(effects
@@
 			)
 		)
-		(property "Footprint" ""
+		(property "Footprint" "Connector_PinHeader_2.54mm:PinHeader_1x01_P2.54mm_Horizontal"
 			(at 115.57 76.2 0)
 			(effects

Commit message: Fixed footprints
Parts:
- J73: footprint Connector_PinHeader_2.54mm:PinHeader_1x16_P2.54mm_Vertical -> Connector_PinHeader_2.54mm:PinHeader_2x08_P2.54mm_Vertical
Changed lines of the file:
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@@
 			)
 		)
-		(property "Footprint" "Connector_PinHeader_2.54mm:PinHeader_1x16_P2.54mm_Vertical"
+		(property "Footprint" "Connector_PinHeader_2.54mm:PinHeader_2x08_P2.54mm_Vertical"
 			(at 158.75 60.96 0)
 			(effects

Commit message: Changed pin headers to vertical
Parts:
- J71: footprint Connector_PinHeader_2.54mm:PinHeader_1x02_P2.54mm_Horizontal -> Connector_PinHeader_2.54mm:PinHeader_1x04_P2.54mm_Vertical
- J72: footprint Connector_PinHeader_2.54mm:PinHeader_1x01_P2.54mm_Horizontal -> Connector_PinHeader_2.54mm:PinHeader_1x04_P2.54mm_Vertical
Changed lines of the file:
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@@
 			)
 		)
-		(property "Footprint" "Connector_PinHeader_2.54mm:PinHeader_1x02_P2.54mm_Horizontal"
+		(property "Footprint" "Connector_PinHeader_2.54mm:PinHeader_1x04_P2.54mm_Vertical"
 			(at 115.57 62.23 0)
 			(effects
@@
 			)
 		)
-		(property "Footprint" "Connector_PinHeader_2.54mm:PinHeader_1x01_P2.54mm_Horizontal"
+		(property "Footprint" "Connector_PinHeader_2.54mm:PinHeader_1x04_P2.54mm_Vertical"
 			(at 115.57 76.2 0)
 			(effects

Commit message: Fixed connector footprints; Changed conectors from 2.54 to 1.27
Parts:
- J69: renamed from J71; footprint Connector_PinHeader_2.54mm:PinHeader_1x04_P2.54mm_Vertical -> Connector_PinHeader_1.27mm:PinHeader_1x02_P1.27mm_Vertical
- J70: renamed from J72; footprint Connector_PinHeader_2.54mm:PinHeader_1x04_P2.54mm_Vertical -> Connector_PinHeader_1.27mm:PinHeader_1x01_P1.27mm_Vertical
- J71: renamed from J73; footprint Connector_PinHeader_2.54mm:PinHeader_2x08_P2.54mm_Vertical -> Connector_PinHeader_1.27mm:PinHeader_2x08_P1.27mm_Vertical
Changed lines of the file:
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@@
 		(dnp no)
 		(fields_autoplaced yes)
-		(property "Reference" "#PWR0374"
+		(property "Reference" "#PWR0376"
 			(at 127 64.77 0)
 			(effects
@@
 			(project "raywatch"
 				(path "/7b654ee8-2a53-4d39-8b7d-32c7bb3cb0ed/2714add3-2889-4ca2-9511-f797ac8197f4"
-					(reference "#PWR0374")
+					(reference "#PWR0376")
 					(unit 1)
 				)
@@
 		(dnp no)
 		(fields_autoplaced yes)
-		(property "Reference" "#PWR0376"
+		(property "Reference" "#PWR0378"
 			(at 129.54 110.49 0)
 			(effects
@@
 			(project "raywatch"
 				(path "/7b654ee8-2a53-4d39-8b7d-32c7bb3cb0ed/2714add3-2889-4ca2-9511-f797ac8197f4"
-					(reference "#PWR0376")
+					(reference "#PWR0378")
 					(unit 1)
 				)
@@
 		(dnp no)
 		(fields_autoplaced yes)
-		(property "Reference" "#PWR0379"
+		(property "Reference" "#PWR0381"
 			(at 165.1 113.03 0)
 			(effects
@@
 			(project "raywatch"
 				(path "/7b654ee8-2a53-4d39-8b7d-32c7bb3cb0ed/2714add3-2889-4ca2-9511-f797ac8197f4"
-					(reference "#PWR0379")
+					(reference "#PWR0381")
 					(unit 1)
 				)
@@
 		(dnp no)
 		(fields_autoplaced yes)
-		(property "Reference" "J71"
+		(property "Reference" "J69"
 			(at 114.3 62.2299 0)
 			(effects
@@
 			)
 		)
-		(property "Footprint" "Connector_PinHeader_2.54mm:PinHeader_1x04_P2.54mm_Vertical"
+		(property "Footprint" "Connector_PinHeader_1.27mm:PinHeader_1x02_P1.27mm_Vertical"
 			(at 115.57 62.23 0)
 			(effects
@@
 			(project "raywatch"
 				(path "/7b654ee8-2a53-4d39-8b7d-32c7bb3cb0ed/2714add3-2889-4ca2-9511-f797ac8197f4"
-					(reference "J71")
+					(reference "J69")
 					(unit 1)
 				)
@@
 		(dnp no)
 		(fields_autoplaced yes)
-		(property "Reference" "#PWR0373"
+		(property "Reference" "#PWR0375"
 			(at 116.84 62.23 0)
 			(effects
@@
 			(project "raywatch"
 				(path "/7b654ee8-2a53-4d39-8b7d-32c7bb3cb0ed/2714add3-2889-4ca2-9511-f797ac8197f4"
-					(reference "#PWR0373")
+					(reference "#PWR0375")
 					(unit 1)
 				)
@@
 		(dnp no)
 		(fields_autoplaced yes)
-		(property "Reference" "#PWR0380"
+		(property "Reference" "#PWR0382"
 			(at 166.37 77.47 0)
 			(effects
@@
 			(project "raywatch"
 				(path "/7b654ee8-2a53-4d39-8b7d-32c7bb3cb0ed/2714add3-2889-4ca2-9511-f797ac8197f4"
-					(reference "#PWR0380")
+					(reference "#PWR0382")
 					(unit 1)
 				)
@@
 		(dnp no)
 		(fields_autoplaced yes)
-		(property "Reference" "J73"
+		(property "Reference" "J71"
 			(at 160.02 46.99 0)
 			(effects
@@
 			)
 		)
-		(property "Footprint" "Connector_PinHeader_2.54mm:PinHeader_2x08_P2.54mm_Vertical"
+		(property "Footprint" "Connector_PinHeader_1.27mm:PinHeader_2x08_P1.27mm_Vertical"
 			(at 158.75 60.96 0)
 			(effects
@@
 			(project "raywatch"
 				(path "/7b654ee8-2a53-4d39-8b7d-32c7bb3cb0ed/2714add3-2889-4ca2-9511-f797ac8197f4"
-					(reference "J73")
+					(reference "J71")
 					(unit 1)
 				)
@@
 		(dnp no)
 		(fields_autoplaced yes)
-		(property "Reference" "#PWR0377"
+		(property "Reference" "#PWR0379"
 			(at 153.67 67.31 0)
 			(effects
@@
 			(project "raywatch"
 				(path "/7b654ee8-2a53-4d39-8b7d-32c7bb3cb0ed/2714add3-2889-4ca2-9511-f797ac8197f4"
-					(reference "#PWR0377")
+					(reference "#PWR0379")
 					(unit 1)
 				)
@@
 		(dnp no)
 		(fields_autoplaced yes)
-		(property "Reference" "J72"
+		(property "Reference" "J70"
 			(at 116.205 71.12 0)
 			(effects
@@
 			)
 		)
-		(property "Footprint" "Connector_PinHeader_2.54mm:PinHeader_1x04_P2.54mm_Vertical"
+		(property "Footprint" "Connector_PinHeader_1.27mm:PinHeader_1x01_P1.27mm_Vertical"
 			(at 115.57 76.2 0)
 			(effects
@@
 			(project "raywatch"
 				(path "/7b654ee8-2a53-4d39-8b7d-32c7bb3cb0ed/2714add3-2889-4ca2-9511-f797ac8197f4"
-					(reference "J72")
+					(reference "J70")
 					(unit 1)
 				)
@@
 		(dnp no)
 		(fields_autoplaced yes)
-		(property "Reference" "#PWR0378"
+		(property "Reference" "#PWR0380"
 			(at 165.1 100.33 0)
 			(effects
@@
 			(project "raywatch"
 				(path "/7b654ee8-2a53-4d39-8b7d-32c7bb3cb0ed/2714add3-2889-4ca2-9511-f797ac8197f4"
-					(reference "#PWR0378")
+					(reference "#PWR0380")
 					(unit 1)
 				)
@@
 		(dnp no)
 		(fields_autoplaced yes)
-		(property "Reference" "#PWR0375"
+		(property "Reference" "#PWR0377"
 			(at 129.54 100.33 0)
 			(effects
@@
 			(project "raywatch"
 				(path "/7b654ee8-2a53-4d39-8b7d-32c7bb3cb0ed/2714add3-2889-4ca2-9511-f797ac8197f4"
-					(reference "#PWR0375")
-					(unit 1)
-				)
+					(reference "#PWR0377")
+					(unit 1)
+				)

Commit message: Fixes; Added TPM PCB
Parts:
- C63, C64: footprint Capacitor_SMD:C_0504_1310Metric -> Capacitor_SMD:C_0402_1005Metric
Changed lines of the file:
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@@
 			)
 		)
-		(property "Footprint" "Capacitor_SMD:C_0504_1310Metric"
+		(property "Footprint" "Capacitor_SMD:C_0402_1005Metric"
 			(at 166.0652 104.14 0)
 			(effects
@@
 			)
 		)
-		(property "Footprint" "Capacitor_SMD:C_0504_1310Metric"
+		(property "Footprint" "Capacitor_SMD:C_0402_1005Metric"
 			(at 128.5748 104.14 0)
 			(effects

Commit message: Fixed 02x08 connector symbol
Parts:
- removed J71: Conn_02x08_Top_Bottom, Connector_PinHeader_1.27mm:PinHeader_2x08_P1.27mm_Vertical, symbol Connector_Generic:Conn_02x08_Top_Bottom
- added J71: Conn_02x08_Odd_Even, symbol Connector_Generic:Conn_02x08_Odd_Even
Connections:
- net +3V0: now also J71.1 (Pin_1), J71.11 (Pin_11), J71.13 (Pin_13), J71.15 (Pin_15), J71.3 (Pin_3), J71.5 (Pin_5), J71.7 (Pin_7), J71.9 (Pin_9)
- net GND: now also J71.10 (Pin_10), J71.12 (Pin_12), J71.14 (Pin_14), J71.16 (Pin_16), J71.2 (Pin_2), J71.4 (Pin_4), J71.6 (Pin_6), J71.8 (Pin_8)
