File: src/hardware/tpm.kicad_sch (KiCad schematic)
At the start: 2 parts

Commit message: Selected GPIO
Changed lines of the file:
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@@
 		)
 		(property "Value" "GND"
-			(at 134.62 118.11 0)
+			(at 137.16 114.2999 0)
 			(effects
 				(font
 					(size 1.27 1.27)
 				)
+				(justify left)
 			)
 		)

Commit message: Cleanup & Fixes; Added footprints; Removed Light sensors
Parts:
- C33: renamed from C?; footprint (none) -> Capacitor_SMD:C_0603_1608Metric
- U9: renamed from U?; footprint UDFN8_2x3MC_MCH -> Project:SON50P200X300X60-9N
Changed lines of the file:
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@@
 		(dnp no)
 		(fields_autoplaced yes)
-		(property "Reference" "#PWR0246"
+		(property "Reference" "#PWR0249"
 			(at 121.92 121.92 0)
 			(effects
@@
 			(project "raywatch"
 				(path "/7b654ee8-2a53-4d39-8b7d-32c7bb3cb0ed/fa39c797-7f88-47af-b50c-765e69cbd658/c4ab4722-2dd5-484a-86b3-dc6635eabcb4"
-					(reference "#PWR0246")
+					(reference "#PWR0249")
 					(unit 1)
 				)
@@
 		(dnp no)
 		(fields_autoplaced yes)
-		(property "Reference" "#PWR0245"
+		(property "Reference" "#PWR0250"
 			(at 134.62 119.38 0)
 			(effects
@@
 		)
 		(property "Value" "GND"
-			(at 137.16 114.2999 0)
-			(effects
-				(font
-					(size 1.27 1.27)
-				)
-				(justify left)
+			(at 134.62 118.11 0)
+			(effects
+				(font
+					(size 1.27 1.27)
+				)
 			)
 		)
@@
 			(project "raywatch"
 				(path "/7b654ee8-2a53-4d39-8b7d-32c7bb3cb0ed/fa39c797-7f88-47af-b50c-765e69cbd658/c4ab4722-2dd5-484a-86b3-dc6635eabcb4"
-					(reference "#PWR0245")
+					(reference "#PWR0250")
 					(unit 1)
 				)
@@
 		(dnp no)
 		(fields_autoplaced yes)
-		(property "Reference" "C?"
+		(property "Reference" "C33"
 			(at 125.73 110.4899 0)
 			(effects
@@
 			)
 		)
-		(property "Footprint" ""
+		(property "Footprint" "Capacitor_SMD:C_0603_1608Metric"
 			(at 122.8852 115.57 0)
 			(effects
@@
 			(project "raywatch"
 				(path "/7b654ee8-2a53-4d39-8b7d-32c7bb3cb0ed/fa39c797-7f88-47af-b50c-765e69cbd658/c4ab4722-2dd5-484a-86b3-dc6635eabcb4"
-					(reference "C?")
+					(reference "C33")
 					(unit 1)
 				)
@@
 		(dnp no)
 		(fields_autoplaced yes)
-		(property "Reference" "#PWR0244"
+		(property "Reference" "#PWR0248"
 			(at 121.92 111.76 0)
 			(effects
@@
 			(project "raywatch"
 				(path "/7b654ee8-2a53-4d39-8b7d-32c7bb3cb0ed/fa39c797-7f88-47af-b50c-765e69cbd658/c4ab4722-2dd5-484a-86b3-dc6635eabcb4"
-					(reference "#PWR0244")
+					(reference "#PWR0248")
 					(unit 1)
 				)
@@
 		(dnp no)
 		(fields_autoplaced yes)
-		(property "Reference" "U?"
+		(property "Reference" "U9"
 			(at 154.94 85.09 0)
 			(effects
@@
 			)
 		)
-		(property "Footprint" "UDFN8_2x3MC_MCH"
+		(property "Footprint" "Project:SON50P200X300X60-9N"
 			(at 134.62 97.79 0)
 			(effects
@@
 			(project "raywatch"
 				(path "/7b654ee8-2a53-4d39-8b7d-32c7bb3cb0ed/fa39c797-7f88-47af-b50c-765e69cbd658/c4ab4722-2dd5-484a-86b3-dc6635eabcb4"
-					(reference "U?")
-					(unit 1)
-				)
+					(reference "U9")
+					(unit 1)
+				)

Commit message: Cleanup & Fixes; Changed GPIO; Added Camera; Added Microphone
Parts:
- renumbered C33 to C31
Changed lines of the file:
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@@
 		(dnp no)
 		(fields_autoplaced yes)
-		(property "Reference" "#PWR0249"
+		(property "Reference" "#PWR0245"
 			(at 121.92 121.92 0)
 			(effects
@@
 			(project "raywatch"
 				(path "/7b654ee8-2a53-4d39-8b7d-32c7bb3cb0ed/fa39c797-7f88-47af-b50c-765e69cbd658/c4ab4722-2dd5-484a-86b3-dc6635eabcb4"
-					(reference "#PWR0249")
+					(reference "#PWR0245")
 					(unit 1)
 				)
@@
 		(dnp no)
 		(fields_autoplaced yes)
-		(property "Reference" "#PWR0250"
+		(property "Reference" "#PWR0246"
 			(at 134.62 119.38 0)
 			(effects
@@
 			(project "raywatch"
 				(path "/7b654ee8-2a53-4d39-8b7d-32c7bb3cb0ed/fa39c797-7f88-47af-b50c-765e69cbd658/c4ab4722-2dd5-484a-86b3-dc6635eabcb4"
-					(reference "#PWR0250")
+					(reference "#PWR0246")
 					(unit 1)
 				)
@@
 		(dnp no)
 		(fields_autoplaced yes)
-		(property "Reference" "C33"
+		(property "Reference" "C31"
 			(at 125.73 110.4899 0)
 			(effects
@@
 			(project "raywatch"
 				(path "/7b654ee8-2a53-4d39-8b7d-32c7bb3cb0ed/fa39c797-7f88-47af-b50c-765e69cbd658/c4ab4722-2dd5-484a-86b3-dc6635eabcb4"
-					(reference "C33")
+					(reference "C31")
 					(unit 1)
 				)
@@
 		(dnp no)
 		(fields_autoplaced yes)
-		(property "Reference" "#PWR0248"
+		(property "Reference" "#PWR0244"
 			(at 121.92 111.76 0)
 			(effects
@@
 			(project "raywatch"
 				(path "/7b654ee8-2a53-4d39-8b7d-32c7bb3cb0ed/fa39c797-7f88-47af-b50c-765e69cbd658/c4ab4722-2dd5-484a-86b3-dc6635eabcb4"
-					(reference "#PWR0248")
-					(unit 1)
-				)
+					(reference "#PWR0244")
+					(unit 1)
+				)

Commit message: Add Light Sensor and Proximity & Gesture Sensor; Changed GPIO
Parts:
- renumbered U9 to U10
Changed lines of the file:
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@@
 		(dnp no)
 		(fields_autoplaced yes)
-		(property "Reference" "#PWR0245"
+		(property "Reference" "#PWR0249"
 			(at 121.92 121.92 0)
 			(effects
@@
 			(project "raywatch"
 				(path "/7b654ee8-2a53-4d39-8b7d-32c7bb3cb0ed/fa39c797-7f88-47af-b50c-765e69cbd658/c4ab4722-2dd5-484a-86b3-dc6635eabcb4"
-					(reference "#PWR0245")
+					(reference "#PWR0249")
 					(unit 1)
 				)
@@
 		(dnp no)
 		(fields_autoplaced yes)
-		(property "Reference" "#PWR0246"
+		(property "Reference" "#PWR0250"
 			(at 134.62 119.38 0)
 			(effects
@@
 			(project "raywatch"
 				(path "/7b654ee8-2a53-4d39-8b7d-32c7bb3cb0ed/fa39c797-7f88-47af-b50c-765e69cbd658/c4ab4722-2dd5-484a-86b3-dc6635eabcb4"
-					(reference "#PWR0246")
+					(reference "#PWR0250")
 					(unit 1)
 				)
@@
 		(dnp no)
 		(fields_autoplaced yes)
-		(property "Reference" "#PWR0244"
+		(property "Reference" "#PWR0248"
 			(at 121.92 111.76 0)
 			(effects
@@
 			(project "raywatch"
 				(path "/7b654ee8-2a53-4d39-8b7d-32c7bb3cb0ed/fa39c797-7f88-47af-b50c-765e69cbd658/c4ab4722-2dd5-484a-86b3-dc6635eabcb4"
-					(reference "#PWR0244")
+					(reference "#PWR0248")
 					(unit 1)
 				)
@@
 		(dnp no)
 		(fields_autoplaced yes)
-		(property "Reference" "U9"
+		(property "Reference" "U10"
 			(at 154.94 85.09 0)
 			(effects
@@
 			(project "raywatch"
 				(path "/7b654ee8-2a53-4d39-8b7d-32c7bb3cb0ed/fa39c797-7f88-47af-b50c-765e69cbd658/c4ab4722-2dd5-484a-86b3-dc6635eabcb4"
-					(reference "U9")
-					(unit 1)
-				)
+					(reference "U10")
+					(unit 1)
+				)

Commit message: Changed footprints from 0603 to 0402
Parts:
- C31: footprint Capacitor_SMD:C_0603_1608Metric -> Capacitor_SMD:C_0504_1310Metric
Changed lines of the file:
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@@
 			)
 		)
-		(property "Footprint" "Capacitor_SMD:C_0603_1608Metric"
+		(property "Footprint" "Capacitor_SMD:C_0504_1310Metric"
 			(at 122.8852 115.57 0)
 			(effects

Commit message: Replaced global labels with pin headers
Parts:
- added J61, J62: Conn_01x02_Pin, symbol Connector:Conn_01x02_Pin
Connections:
- net +3V3: now also J61.1 (Pin_1)
- net GND: now also J61.2 (Pin_2)
- net SCL: now also J62.1 (Pin_1)
- net SDA: now also J62.2 (Pin_2)
