File: src/hardware/tpm.kicad_sch (KiCad schematic)
At the start: 4 parts, among them J61 Conn_01x02_Pin, J62 Conn_01x02_Pin, U10 ATECC608A-MAHDA-S

Commit message: Reannotated schematic
Parts:
- renumbered C31 to C25, J61 to J37, J62 to J38
Changed lines of the file:
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@@
 		(dnp no)
 		(fields_autoplaced yes)
-		(property "Reference" "#PWR0249"
+		(property "Reference" "#PWR0248"
 			(at 121.92 121.92 0)
 			(effects
@@
 			(project "raywatch"
 				(path "/7b654ee8-2a53-4d39-8b7d-32c7bb3cb0ed/f081a1f8-fc4b-4b06-b900-3123b3d09078"
-					(reference "#PWR0249")
+					(reference "#PWR0248")
 					(unit 1)
 				)
@@
 		(dnp no)
 		(fields_autoplaced yes)
-		(property "Reference" "#PWR0250"
+		(property "Reference" "#PWR0249"
 			(at 134.62 119.38 0)
 			(effects
@@
 			(project "raywatch"
 				(path "/7b654ee8-2a53-4d39-8b7d-32c7bb3cb0ed/f081a1f8-fc4b-4b06-b900-3123b3d09078"
-					(reference "#PWR0250")
+					(reference "#PWR0249")
 					(unit 1)
 				)
@@
 		(dnp no)
 		(fields_autoplaced yes)
-		(property "Reference" "J61"
+		(property "Reference" "J37"
 			(at 97.155 59.69 0)
 			(effects
@@
 			(project "raywatch"
 				(path "/7b654ee8-2a53-4d39-8b7d-32c7bb3cb0ed/f081a1f8-fc4b-4b06-b900-3123b3d09078"
-					(reference "J61")
+					(reference "J37")
 					(unit 1)
 				)
@@
 		(dnp no)
 		(fields_autoplaced yes)
-		(property "Reference" "#PWR0491"
+		(property "Reference" "#PWR0245"
 			(at 97.79 64.77 0)
 			(effects
@@
 			(project "raywatch"
 				(path "/7b654ee8-2a53-4d39-8b7d-32c7bb3cb0ed/f081a1f8-fc4b-4b06-b900-3123b3d09078"
-					(reference "#PWR0491")
+					(reference "#PWR0245")
 					(unit 1)
 				)
@@
 		(dnp no)
 		(fields_autoplaced yes)
-		(property "Reference" "C31"
+		(property "Reference" "C25"
 			(at 125.73 110.4899 0)
 			(effects
@@
 			(project "raywatch"
 				(path "/7b654ee8-2a53-4d39-8b7d-32c7bb3cb0ed/f081a1f8-fc4b-4b06-b900-3123b3d09078"
-					(reference "C31")
+					(reference "C25")
 					(unit 1)
 				)
@@
 		(dnp no)
 		(fields_autoplaced yes)
-		(property "Reference" "#PWR0248"
+		(property "Reference" "#PWR0247"
 			(at 121.92 111.76 0)
 			(effects
@@
 			(project "raywatch"
 				(path "/7b654ee8-2a53-4d39-8b7d-32c7bb3cb0ed/f081a1f8-fc4b-4b06-b900-3123b3d09078"
-					(reference "#PWR0248")
+					(reference "#PWR0247")
 					(unit 1)
 				)
@@
 		(dnp no)
 		(fields_autoplaced yes)
-		(property "Reference" "#PWR0492"
+		(property "Reference" "#PWR0246"
 			(at 107.95 67.31 0)
 			(effects
@@
 			(project "raywatch"
 				(path "/7b654ee8-2a53-4d39-8b7d-32c7bb3cb0ed/f081a1f8-fc4b-4b06-b900-3123b3d09078"
-					(reference "#PWR0492")
+					(reference "#PWR0246")
 					(unit 1)
 				)
@@
 		(dnp no)
 		(fields_autoplaced yes)
-		(property "Reference" "J62"
+		(property "Reference" "J38"
 			(at 97.155 69.85 0)
 			(effects
@@
 			(project "raywatch"
 				(path "/7b654ee8-2a53-4d39-8b7d-32c7bb3cb0ed/f081a1f8-fc4b-4b06-b900-3123b3d09078"
-					(reference "J62")
-					(unit 1)
-				)
+					(reference "J38")
+					(unit 1)
+				)

Commit message: Assigned pin header footprints
Parts:
- J37, J38: footprint (none) -> Connector_PinHeader_2.54mm:PinHeader_1x02_P2.54mm_Horizontal
Changed lines of the file:
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@@
 			)
 		)
-		(property "Footprint" ""
+		(property "Footprint" "Connector_PinHeader_2.54mm:PinHeader_1x02_P2.54mm_Horizontal"
 			(at 96.52 64.77 0)
 			(effects
@@
 			)
 		)
-		(property "Footprint" ""
+		(property "Footprint" "Connector_PinHeader_2.54mm:PinHeader_1x02_P2.54mm_Horizontal"
 			(at 96.52 74.93 0)
 			(effects

Commit message: Fixed symbol of ATECC608A-MAHDA-S
Parts:
- U10: footprint Project:SON50P200X300X60-9N -> SON50P200X300X60-9N
Connections:
- net GND: now also U10.9 (GND_PAD)
Changed lines of the file:
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@@
 	)
 	(no_connect
-		(at 175.26 107.95)
+		(at 175.26 99.06)
 	)
 	(no_connect
-		(at 175.26 110.49)
+		(at 175.26 104.14)
 	)
 	(no_connect
-		(at 175.26 105.41)
+		(at 175.26 101.6)
 	)
 	(no_connect
-		(at 175.26 102.87)
+		(at 175.26 106.68)
 	)
 	(wire
@@
 	(symbol
 		(lib_id "power:GND")
+		(at 175.26 111.76 0)
+		(unit 1)
+		(exclude_from_sim no)
+		(in_bom yes)
+		(on_board yes)
+		(dnp no)
+		(fields_autoplaced yes)
+		(property "Reference" "#PWR0498"
+			(at 175.26 118.11 0)
+			(effects
+				(font
+					(size 1.27 1.27)
+				)
+				(hide yes)
+			)
+		)
+		(property "Value" "GND"
+			(at 175.26 116.84 0)
+			(effects
+				(font
+					(size 1.27 1.27)
+				)
+			)
+		)
+		(property "Footprint" ""
+			(at 175.26 111.76 0)
+			(effects
+				(font
+					(size 1.27 1.27)
+				)
+				(hide yes)
+			)
+		)
+		(property "Datasheet" ""
+			(at 175.26 111.76 0)
+			(effects
+				(font
+					(size 1.27 1.27)
+				)
+				(hide yes)
+			)
+		)
+		(property "Description" "Power symbol creates a global label with name \"GND\" , ground"
+			(at 175.26 111.76 0)
+			(effects
+				(font
+					(size 1.27 1.27)
+				)
+				(hide yes)
+			)
+		)
+		(pin "1"
+		)
+		(instances
+			(project "raywatch"
+				(path "/7b654ee8-2a53-4d39-8b7d-32c7bb3cb0ed/f081a1f8-fc4b-4b06-b900-3123b3d09078"
+					(reference "#PWR0498")
+					(unit 1)
+				)
+			)
+		)
+	)
+	(symbol
+		(lib_id "power:GND")
 		(at 134.62 113.03 0)
 		(unit 1)
@@
 			)
 		)
-		(property "Footprint" "Project:SON50P200X300X60-9N"
+		(property "Footprint" "SON50P200X300X60-9N"
 			(at 134.62 97.79 0)
 			(effects
@@
 			)
 		)
-		(property "Datasheet" "ATECC608A-MAHDA-S"
+		(property "Datasheet" "https://ww1.microchip.com/downloads/en/DeviceDoc/ATECC608A-CryptoAuthentication-Device-Summary-Data-Sheet-DS40001977B.pdf"
 			(at 134.62 97.79 0)
 			(effects
@@
 		(pin "2"
 		)
-		(instances
+		(pin "9"
+		)
+		(instances

Commit message: Reannotate
Parts:
- renumbered U10 to U9
Changed lines of the file:
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@@
 		(dnp no)
 		(fields_autoplaced yes)
-		(property "Reference" "#PWR0498"
+		(property "Reference" "#PWR0250"
 			(at 175.26 118.11 0)
 			(effects
@@
 			(project "raywatch"
 				(path "/7b654ee8-2a53-4d39-8b7d-32c7bb3cb0ed/f081a1f8-fc4b-4b06-b900-3123b3d09078"
-					(reference "#PWR0498")
+					(reference "#PWR0250")
 					(unit 1)
 				)
@@
 		(dnp no)
 		(fields_autoplaced yes)
-		(property "Reference" "U10"
+		(property "Reference" "U9"
 			(at 154.94 85.09 0)
 			(effects
@@
 			(project "raywatch"
 				(path "/7b654ee8-2a53-4d39-8b7d-32c7bb3cb0ed/f081a1f8-fc4b-4b06-b900-3123b3d09078"
-					(reference "U10")
-					(unit 1)
-				)
+					(reference "U9")
+					(unit 1)
+				)

Commit message: Fixed U9
Parts:
- U9: footprint SON50P200X300X60-9N -> Project:SON50P200X300X60-9N
Changed lines of the file:
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@@
 			)
 		)
-		(property "Footprint" "SON50P200X300X60-9N"
+		(property "Footprint" "Project:SON50P200X300X60-9N"
 			(at 134.62 97.79 0)
 			(effects

Commit message: Changed pin headers to vertical
Parts:
- J37, J38: footprint Connector_PinHeader_2.54mm:PinHeader_1x02_P2.54mm_Horizontal -> Connector_PinHeader_2.54mm:PinHeader_1x02_P2.54mm_Vertical
Changed lines of the file:
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@@
 			)
 		)
-		(property "Footprint" "Connector_PinHeader_2.54mm:PinHeader_1x02_P2.54mm_Horizontal"
+		(property "Footprint" "Connector_PinHeader_2.54mm:PinHeader_1x02_P2.54mm_Vertical"
 			(at 96.52 64.77 0)
 			(effects
@@
 			)
 		)
-		(property "Footprint" "Connector_PinHeader_2.54mm:PinHeader_1x02_P2.54mm_Horizontal"
+		(property "Footprint" "Connector_PinHeader_2.54mm:PinHeader_1x02_P2.54mm_Vertical"
 			(at 96.52 74.93 0)
 			(effects

Commit message: Fixed connector footprints; Changed conectors from 2.54 to 1.27
Parts:
- J35: renamed from J37; footprint Connector_PinHeader_2.54mm:PinHeader_1x02_P2.54mm_Vertical -> Connector_PinHeader_1.27mm:PinHeader_1x02_P1.27mm_Vertical
- J36: renamed from J38; footprint Connector_PinHeader_2.54mm:PinHeader_1x02_P2.54mm_Vertical -> Connector_PinHeader_1.27mm:PinHeader_1x02_P1.27mm_Vertical
Changed lines of the file:
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@@
 		(dnp no)
 		(fields_autoplaced yes)
-		(property "Reference" "#PWR0248"
+		(property "Reference" "#PWR0250"
 			(at 121.92 121.92 0)
 			(effects
@@
 			(project "raywatch"
 				(path "/7b654ee8-2a53-4d39-8b7d-32c7bb3cb0ed/f081a1f8-fc4b-4b06-b900-3123b3d09078"
-					(reference "#PWR0248")
+					(reference "#PWR0250")
 					(unit 1)
 				)
@@
 		(dnp no)
 		(fields_autoplaced yes)
-		(property "Reference" "#PWR0250"
+		(property "Reference" "#PWR0252"
 			(at 175.26 118.11 0)
 			(effects
@@
 			(project "raywatch"
 				(path "/7b654ee8-2a53-4d39-8b7d-32c7bb3cb0ed/f081a1f8-fc4b-4b06-b900-3123b3d09078"
-					(reference "#PWR0250")
+					(reference "#PWR0252")
 					(unit 1)
 				)
@@
 		(dnp no)
 		(fields_autoplaced yes)
-		(property "Reference" "#PWR0249"
+		(property "Reference" "#PWR0251"
 			(at 134.62 119.38 0)
 			(effects
@@
 			(project "raywatch"
 				(path "/7b654ee8-2a53-4d39-8b7d-32c7bb3cb0ed/f081a1f8-fc4b-4b06-b900-3123b3d09078"
-					(reference "#PWR0249")
+					(reference "#PWR0251")
 					(unit 1)
 				)
@@
 		(dnp no)
 		(fields_autoplaced yes)
-		(property "Reference" "J37"
+		(property "Reference" "J35"
 			(at 97.155 59.69 0)
 			(effects
@@
 			)
 		)
-		(property "Footprint" "Connector_PinHeader_2.54mm:PinHeader_1x02_P2.54mm_Vertical"
+		(property "Footprint" "Connector_PinHeader_1.27mm:PinHeader_1x02_P1.27mm_Vertical"
 			(at 96.52 64.77 0)
 			(effects
@@
 			(project "raywatch"
 				(path "/7b654ee8-2a53-4d39-8b7d-32c7bb3cb0ed/f081a1f8-fc4b-4b06-b900-3123b3d09078"
-					(reference "J37")
+					(reference "J35")
 					(unit 1)
 				)
@@
 		(dnp no)
 		(fields_autoplaced yes)
-		(property "Reference" "#PWR0245"
+		(property "Reference" "#PWR0247"
 			(at 97.79 64.77 0)
 			(effects
@@
 			(project "raywatch"
 				(path "/7b654ee8-2a53-4d39-8b7d-32c7bb3cb0ed/f081a1f8-fc4b-4b06-b900-3123b3d09078"
-					(reference "#PWR0245")
+					(reference "#PWR0247")
 					(unit 1)
 				)
@@
 		(dnp no)
 		(fields_autoplaced yes)
-		(property "Reference" "#PWR0247"
+		(property "Reference" "#PWR0249"
 			(at 121.92 111.76 0)
 			(effects
@@
 			(project "raywatch"
 				(path "/7b654ee8-2a53-4d39-8b7d-32c7bb3cb0ed/f081a1f8-fc4b-4b06-b900-3123b3d09078"
-					(reference "#PWR0247")
+					(reference "#PWR0249")
 					(unit 1)
 				)
@@
 		(dnp no)
 		(fields_autoplaced yes)
-		(property "Reference" "#PWR0246"
+		(property "Reference" "#PWR0248"
 			(at 107.95 67.31 0)
 			(effects
@@
 			(project "raywatch"
 				(path "/7b654ee8-2a53-4d39-8b7d-32c7bb3cb0ed/f081a1f8-fc4b-4b06-b900-3123b3d09078"
-					(reference "#PWR0246")
+					(reference "#PWR0248")
 					(unit 1)
 				)
@@
 		(dnp no)
 		(fields_autoplaced yes)
-		(property "Reference" "J38"
+		(property "Reference" "J36"
 			(at 97.155 69.85 0)
 			(effects
@@
 			)
 		)
-		(property "Footprint" "Connector_PinHeader_2.54mm:PinHeader_1x02_P2.54mm_Vertical"
+		(property "Footprint" "Connector_PinHeader_1.27mm:PinHeader_1x02_P1.27mm_Vertical"
 			(at 96.52 74.93 0)
 			(effects
@@
 			(project "raywatch"
 				(path "/7b654ee8-2a53-4d39-8b7d-32c7bb3cb0ed/f081a1f8-fc4b-4b06-b900-3123b3d09078"
-					(reference "J38")
-					(unit 1)
-				)
+					(reference "J36")
+					(unit 1)
+				)

Commit message: Fixes; Added TPM PCB
Parts:
- C25: footprint Capacitor_SMD:C_0504_1310Metric -> Capacitor_SMD:C_0402_1005Metric
Changed lines of the file:
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@@
 			)
 		)
-		(property "Footprint" "Capacitor_SMD:C_0504_1310Metric"
+		(property "Footprint" "Capacitor_SMD:C_0402_1005Metric"
 			(at 122.8852 115.57 0)
 			(effects
