File: src/hardware/microphone.kicad_sch (KiCad schematic)
At the start: 0 parts

Commit message: Added Microphone
Parts:
- added C101: 100nF, symbol Device:C
- added U35: IM72D128V01XTMA1, PG-LLGA-5-3_INF, symbol IM72D128V01XTMA1:IM72D128V01XTMA1
Connections:
- new net +3V3: C101.1, U35.2 (VDD)
- new net GND: C101.2, U35.4 (SELECT), U35.5 (GND)
- new net PDKCLK: U35.3 (CLOCK)
- new net PDMDATA: U35.1 (DATA)

Commit message: Added 1.8V GPIO Extender
Parts:
- U35: footprint PG-LLGA-5-3_INF -> Project:PG-LLGA-5-3_INF
Changed lines of the file:
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@@
 			)
 		)
-		(property "Footprint" "PG-LLGA-5-3_INF"
+		(property "Footprint" "Project:PG-LLGA-5-3_INF"
 			(at 133.35 91.44 0)
 			(effects

Commit message: Selected S1..10 & TR1
Parts:
- C101: footprint (none) -> Capacitor_SMD:C_0603_1608Metric
Changed lines of the file:
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@@
 			)
 		)
-		(property "Footprint" ""
+		(property "Footprint" "Capacitor_SMD:C_0603_1608Metric"
 			(at 122.8852 111.76 0)
 			(effects

Commit message: Changed footprints from 0603 to 0402
Parts:
- C101: footprint Capacitor_SMD:C_0603_1608Metric -> Capacitor_SMD:C_0504_1310Metric
Changed lines of the file:
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@@
 			)
 		)
-		(property "Footprint" "Capacitor_SMD:C_0603_1608Metric"
+		(property "Footprint" "Capacitor_SMD:C_0504_1310Metric"
 			(at 122.8852 111.76 0)
 			(effects

Commit message: Replaced global labels with pin headers
Parts:
- added J5, J6: Conn_01x02_Pin, symbol Connector:Conn_01x02_Pin
Connections:
- net +3V3: now also J5.1 (Pin_1)
- net GND: now also J5.2 (Pin_2)
- net PDMDATA: now also J6.1 (Pin_1)
- net PDKCLK renamed PDMCLK
- net PDMCLK: now also J6.2 (Pin_2)

Commit message: Reannotated schematic
Parts:
- renumbered C101 to C96, J5 to J92, J6 to J93, U35 to U36
Changed lines of the file:
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@@
 		(dnp no)
 		(fields_autoplaced yes)
-		(property "Reference" "J5"
+		(property "Reference" "J92"
 			(at 80.01 86.3599 0)
 			(effects
@@
 			(project "raywatch"
 				(path "/7b654ee8-2a53-4d39-8b7d-32c7bb3cb0ed/f2f5da81-6e74-45e5-9c07-b66eda9b7e5d"
-					(reference "J5")
+					(reference "J92")
 					(unit 1)
 				)
@@
 		(dnp no)
 		(fields_autoplaced yes)
-		(property "Reference" "U35"
+		(property "Reference" "U36"
 			(at 156.21 81.28 0)
 			(effects
@@
 			(project "raywatch"
 				(path "/7b654ee8-2a53-4d39-8b7d-32c7bb3cb0ed/f2f5da81-6e74-45e5-9c07-b66eda9b7e5d"
-					(reference "U35")
+					(reference "U36")
 					(unit 1)
 				)
@@
 		(dnp no)
 		(fields_autoplaced yes)
-		(property "Reference" "#PWR0412"
+		(property "Reference" "#PWR0471"
 			(at 127 96.52 0)
 			(effects
@@
 			(project "raywatch"
 				(path "/7b654ee8-2a53-4d39-8b7d-32c7bb3cb0ed/f2f5da81-6e74-45e5-9c07-b66eda9b7e5d"
-					(reference "#PWR0412")
+					(reference "#PWR0471")
 					(unit 1)
 				)
@@
 		(dnp no)
 		(fields_autoplaced yes)
-		(property "Reference" "#PWR076"
+		(property "Reference" "#PWR0468"
 			(at 92.71 88.9 0)
 			(effects
@@
 			(project "raywatch"
 				(path "/7b654ee8-2a53-4d39-8b7d-32c7bb3cb0ed/f2f5da81-6e74-45e5-9c07-b66eda9b7e5d"
-					(reference "#PWR076")
+					(reference "#PWR0468")
 					(unit 1)
 				)
@@
 		(dnp no)
 		(fields_autoplaced yes)
-		(property "Reference" "#PWR0413"
+		(property "Reference" "#PWR0472"
 			(at 133.35 115.57 0)
 			(effects
@@
 			(project "raywatch"
 				(path "/7b654ee8-2a53-4d39-8b7d-32c7bb3cb0ed/f2f5da81-6e74-45e5-9c07-b66eda9b7e5d"
-					(reference "#PWR0413")
+					(reference "#PWR0472")
 					(unit 1)
 				)
@@
 		(dnp no)
 		(fields_autoplaced yes)
-		(property "Reference" "J6"
+		(property "Reference" "J93"
 			(at 80.01 93.9799 0)
 			(effects
@@
 			(project "raywatch"
 				(path "/7b654ee8-2a53-4d39-8b7d-32c7bb3cb0ed/f2f5da81-6e74-45e5-9c07-b66eda9b7e5d"
-					(reference "J6")
+					(reference "J93")
 					(unit 1)
 				)
@@
 		(dnp no)
 		(fields_autoplaced yes)
-		(property "Reference" "#PWR0411"
+		(property "Reference" "#PWR0470"
 			(at 121.92 118.11 0)
 			(effects
@@
 			(project "raywatch"
 				(path "/7b654ee8-2a53-4d39-8b7d-32c7bb3cb0ed/f2f5da81-6e74-45e5-9c07-b66eda9b7e5d"
-					(reference "#PWR0411")
+					(reference "#PWR0470")
 					(unit 1)
 				)
@@
 		(dnp no)
 		(fields_autoplaced yes)
-		(property "Reference" "#PWR075"
+		(property "Reference" "#PWR0467"
 			(at 82.55 86.36 0)
 			(effects
@@
 			(project "raywatch"
 				(path "/7b654ee8-2a53-4d39-8b7d-32c7bb3cb0ed/f2f5da81-6e74-45e5-9c07-b66eda9b7e5d"
-					(reference "#PWR075")
+					(reference "#PWR0467")
 					(unit 1)
 				)
@@
 		(dnp no)
 		(fields_autoplaced yes)
-		(property "Reference" "C101"
+		(property "Reference" "C96"
 			(at 125.73 106.6799 0)
 			(effects
@@
 			(project "raywatch"
 				(path "/7b654ee8-2a53-4d39-8b7d-32c7bb3cb0ed/f2f5da81-6e74-45e5-9c07-b66eda9b7e5d"
-					(reference "C101")
+					(reference "C96")
 					(unit 1)
 				)
@@
 		(dnp no)
 		(fields_autoplaced yes)
-		(property "Reference" "#PWR0410"
+		(property "Reference" "#PWR0469"
 			(at 121.92 107.95 0)
 			(effects
@@
 			(project "raywatch"
 				(path "/7b654ee8-2a53-4d39-8b7d-32c7bb3cb0ed/f2f5da81-6e74-45e5-9c07-b66eda9b7e5d"
-					(reference "#PWR0410")
-					(unit 1)
-				)
+					(reference "#PWR0469")
+					(unit 1)
+				)
