File: src/hardware/microphone.kicad_sch (KiCad schematic)
At the start: 4 parts, among them J92 Conn_01x02_Pin, J93 Conn_01x02_Pin, U36 IM72D128V01XTMA1

Commit message: Assigned pin header footprints
Parts:
- J92, J93: footprint (none) -> Connector_PinHeader_2.54mm:PinHeader_1x02_P2.54mm_Horizontal
Changed lines of the file:
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@@
 			)
 		)
-		(property "Footprint" ""
+		(property "Footprint" "Connector_PinHeader_2.54mm:PinHeader_1x02_P2.54mm_Horizontal"
 			(at 81.28 86.36 0)
 			(effects
@@
 			)
 		)
-		(property "Footprint" ""
+		(property "Footprint" "Connector_PinHeader_2.54mm:PinHeader_1x02_P2.54mm_Horizontal"
 			(at 81.28 93.98 0)
 			(effects

Commit message: Changed pin headers to vertical
Parts:
- J92, J93: footprint Connector_PinHeader_2.54mm:PinHeader_1x02_P2.54mm_Horizontal -> Connector_PinHeader_2.54mm:PinHeader_1x02_P2.54mm_Vertical
Changed lines of the file:
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@@
 			)
 		)
-		(property "Footprint" "Connector_PinHeader_2.54mm:PinHeader_1x02_P2.54mm_Horizontal"
+		(property "Footprint" "Connector_PinHeader_2.54mm:PinHeader_1x02_P2.54mm_Vertical"
 			(at 81.28 86.36 0)
 			(effects
@@
 			)
 		)
-		(property "Footprint" "Connector_PinHeader_2.54mm:PinHeader_1x02_P2.54mm_Horizontal"
+		(property "Footprint" "Connector_PinHeader_2.54mm:PinHeader_1x02_P2.54mm_Vertical"
 			(at 81.28 93.98 0)
 			(effects

Commit message: Fixed connector footprints; Changed conectors from 2.54 to 1.27
Parts:
- J90: renamed from J92; footprint Connector_PinHeader_2.54mm:PinHeader_1x02_P2.54mm_Vertical -> Connector_PinHeader_1.27mm:PinHeader_1x02_P1.27mm_Vertical
- J91: renamed from J93; footprint Connector_PinHeader_2.54mm:PinHeader_1x02_P2.54mm_Vertical -> Connector_PinHeader_1.27mm:PinHeader_1x02_P1.27mm_Vertical
Changed lines of the file:
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@@
 		(dnp no)
 		(fields_autoplaced yes)
-		(property "Reference" "J92"
+		(property "Reference" "J90"
 			(at 80.01 86.3599 0)
 			(effects
@@
 			)
 		)
-		(property "Footprint" "Connector_PinHeader_2.54mm:PinHeader_1x02_P2.54mm_Vertical"
+		(property "Footprint" "Connector_PinHeader_1.27mm:PinHeader_1x02_P1.27mm_Vertical"
 			(at 81.28 86.36 0)
 			(effects
@@
 			(project "raywatch"
 				(path "/7b654ee8-2a53-4d39-8b7d-32c7bb3cb0ed/f2f5da81-6e74-45e5-9c07-b66eda9b7e5d"
-					(reference "J92")
+					(reference "J90")
 					(unit 1)
 				)
@@
 		(dnp no)
 		(fields_autoplaced yes)
-		(property "Reference" "#PWR0473"
+		(property "Reference" "#PWR0475"
 			(at 127 96.52 0)
 			(effects
@@
 			(project "raywatch"
 				(path "/7b654ee8-2a53-4d39-8b7d-32c7bb3cb0ed/f2f5da81-6e74-45e5-9c07-b66eda9b7e5d"
-					(reference "#PWR0473")
+					(reference "#PWR0475")
 					(unit 1)
 				)
@@
 		(dnp no)
 		(fields_autoplaced yes)
-		(property "Reference" "#PWR0470"
+		(property "Reference" "#PWR0472"
 			(at 92.71 88.9 0)
 			(effects
@@
 			(project "raywatch"
 				(path "/7b654ee8-2a53-4d39-8b7d-32c7bb3cb0ed/f2f5da81-6e74-45e5-9c07-b66eda9b7e5d"
-					(reference "#PWR0470")
+					(reference "#PWR0472")
 					(unit 1)
 				)
@@
 		(dnp no)
 		(fields_autoplaced yes)
-		(property "Reference" "#PWR0474"
+		(property "Reference" "#PWR0476"
 			(at 133.35 115.57 0)
 			(effects
@@
 			(project "raywatch"
 				(path "/7b654ee8-2a53-4d39-8b7d-32c7bb3cb0ed/f2f5da81-6e74-45e5-9c07-b66eda9b7e5d"
-					(reference "#PWR0474")
+					(reference "#PWR0476")
 					(unit 1)
 				)
@@
 		(dnp no)
 		(fields_autoplaced yes)
-		(property "Reference" "J93"
+		(property "Reference" "J91"
 			(at 80.01 93.9799 0)
 			(effects
@@
 			)
 		)
-		(property "Footprint" "Connector_PinHeader_2.54mm:PinHeader_1x02_P2.54mm_Vertical"
+		(property "Footprint" "Connector_PinHeader_1.27mm:PinHeader_1x02_P1.27mm_Vertical"
 			(at 81.28 93.98 0)
 			(effects
@@
 			(project "raywatch"
 				(path "/7b654ee8-2a53-4d39-8b7d-32c7bb3cb0ed/f2f5da81-6e74-45e5-9c07-b66eda9b7e5d"
-					(reference "J93")
+					(reference "J91")
 					(unit 1)
 				)
@@
 		(dnp no)
 		(fields_autoplaced yes)
-		(property "Reference" "#PWR0472"
+		(property "Reference" "#PWR0474"
 			(at 121.92 118.11 0)
 			(effects
@@
 			(project "raywatch"
 				(path "/7b654ee8-2a53-4d39-8b7d-32c7bb3cb0ed/f2f5da81-6e74-45e5-9c07-b66eda9b7e5d"
-					(reference "#PWR0472")
+					(reference "#PWR0474")
 					(unit 1)
 				)
@@
 		(dnp no)
 		(fields_autoplaced yes)
-		(property "Reference" "#PWR0469"
+		(property "Reference" "#PWR0471"
 			(at 82.55 86.36 0)
 			(effects
@@
 			(project "raywatch"
 				(path "/7b654ee8-2a53-4d39-8b7d-32c7bb3cb0ed/f2f5da81-6e74-45e5-9c07-b66eda9b7e5d"
-					(reference "#PWR0469")
+					(reference "#PWR0471")
 					(unit 1)
 				)
@@
 		(dnp no)
 		(fields_autoplaced yes)
-		(property "Reference" "#PWR0471"
+		(property "Reference" "#PWR0473"
 			(at 121.92 107.95 0)
 			(effects
@@
 			(project "raywatch"
 				(path "/7b654ee8-2a53-4d39-8b7d-32c7bb3cb0ed/f2f5da81-6e74-45e5-9c07-b66eda9b7e5d"
-					(reference "#PWR0471")
-					(unit 1)
-				)
+					(reference "#PWR0473")
+					(unit 1)
+				)

Commit message: Fixes; Added TPM PCB
Parts:
- C96: footprint Capacitor_SMD:C_0504_1310Metric -> Capacitor_SMD:C_0402_1005Metric
Changed lines of the file:
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@@
 			)
 		)
-		(property "Footprint" "Capacitor_SMD:C_0504_1310Metric"
+		(property "Footprint" "Capacitor_SMD:C_0402_1005Metric"
 			(at 122.8852 111.76 0)
 			(effects
