File: src/hardware/wireless_charging.kicad_sch (KiCad schematic)
At the start: 24 parts, among them U24 CSD83325L, U25 BQ51013BRHLR

Commit message: Cleanup & Fixes; Changed GPIO; Added Camera; Added Microphone
Parts:
- renumbered C71 to C69, C72 to C70, C73 to C71, C74 to C72, C75 to C73, C76 to C74, C77 to C75, C78 to C76, C79 to C77, C80 to C78, C81 to C79, C82 to C80, C83 to C81, C84 to C82, C85 to C83, C86 to C84, R37 to R35, R38 to R36, R39 to R37, R40 to R38, R41 to R39

Commit message: Add Light Sensor and Proximity & Gesture Sensor; Changed GPIO
Parts:
- renumbered R35 to R36, R36 to R37, R37 to R38, R38 to R39, R39 to R40, U24 to U25, U25 to U26
Changed lines of the file:
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@@
 		(dnp no)
 		(fields_autoplaced yes)
-		(property "Reference" "R37"
+		(property "Reference" "R38"
 			(at 116.84 114.3 90)
 			(effects
@@
 			(project "raywatch"
 				(path "/7b654ee8-2a53-4d39-8b7d-32c7bb3cb0ed/6e6a70ea-4db2-4b59-a2d7-c468f9b8b5a6/d00e072b-2be1-497b-8423-3eead973d996"
-					(reference "R37")
+					(reference "R38")
 					(unit 1)
 				)
@@
 		(dnp no)
 		(fields_autoplaced yes)
-		(property "Reference" "#PWR0352"
+		(property "Reference" "#PWR0356"
 			(at 156.21 127 0)
 			(effects
@@
 			(project "raywatch"
 				(path "/7b654ee8-2a53-4d39-8b7d-32c7bb3cb0ed/6e6a70ea-4db2-4b59-a2d7-c468f9b8b5a6/d00e072b-2be1-497b-8423-3eead973d996"
-					(reference "#PWR0352")
+					(reference "#PWR0356")
 					(unit 1)
 				)
@@
 		(dnp no)
 		(fields_autoplaced yes)
-		(property "Reference" "#PWR0354"
+		(property "Reference" "#PWR0358"
 			(at 181.61 106.68 0)
 			(effects
@@
 			(project "raywatch"
 				(path "/7b654ee8-2a53-4d39-8b7d-32c7bb3cb0ed/6e6a70ea-4db2-4b59-a2d7-c468f9b8b5a6/d00e072b-2be1-497b-8423-3eead973d996"
-					(reference "#PWR0354")
+					(reference "#PWR0358")
 					(unit 1)
 				)
@@
 		(dnp no)
 		(fields_autoplaced yes)
-		(property "Reference" "#PWR0344"
+		(property "Reference" "#PWR0348"
 			(at 43.18 109.22 0)
 			(effects
@@
 			(project "raywatch"
 				(path "/7b654ee8-2a53-4d39-8b7d-32c7bb3cb0ed/6e6a70ea-4db2-4b59-a2d7-c468f9b8b5a6/d00e072b-2be1-497b-8423-3eead973d996"
-					(reference "#PWR0344")
+					(reference "#PWR0348")
 					(unit 1)
 				)
@@
 		(dnp no)
 		(fields_autoplaced yes)
-		(property "Reference" "#PWR0355"
+		(property "Reference" "#PWR0359"
 			(at 181.61 116.84 0)
 			(effects
@@
 			(project "raywatch"
 				(path "/7b654ee8-2a53-4d39-8b7d-32c7bb3cb0ed/6e6a70ea-4db2-4b59-a2d7-c468f9b8b5a6/d00e072b-2be1-497b-8423-3eead973d996"
-					(reference "#PWR0355")
+					(reference "#PWR0359")
 					(unit 1)
 				)
@@
 		(dnp no)
 		(fields_autoplaced yes)
-		(property "Reference" "U24"
+		(property "Reference" "U25"
 			(at 53.34 83.8199 90)
 			(effects
@@
 			(project "raywatch"
 				(path "/7b654ee8-2a53-4d39-8b7d-32c7bb3cb0ed/6e6a70ea-4db2-4b59-a2d7-c468f9b8b5a6/d00e072b-2be1-497b-8423-3eead973d996"
-					(reference "U24")
+					(reference "U25")
 					(unit 1)
 				)
@@
 		(dnp no)
 		(fields_autoplaced yes)
-		(property "Reference" "#PWR0353"
+		(property "Reference" "#PWR0357"
 			(at 168.91 116.84 0)
 			(effects
@@
 			(project "raywatch"
 				(path "/7b654ee8-2a53-4d39-8b7d-32c7bb3cb0ed/6e6a70ea-4db2-4b59-a2d7-c468f9b8b5a6/d00e072b-2be1-497b-8423-3eead973d996"
-					(reference "#PWR0353")
+					(reference "#PWR0357")
 					(unit 1)
 				)
@@
 		(dnp no)
 		(fields_autoplaced yes)
-		(property "Reference" "#PWR0347"
+		(property "Reference" "#PWR0351"
 			(at 57.15 68.58 0)
 			(effects
@@
 			(project "raywatch"
 				(path "/7b654ee8-2a53-4d39-8b7d-32c7bb3cb0ed/6e6a70ea-4db2-4b59-a2d7-c468f9b8b5a6/d00e072b-2be1-497b-8423-3eead973d996"
-					(reference "#PWR0347")
+					(reference "#PWR0351")
 					(unit 1)
 				)
@@
 		(dnp no)
 		(fields_autoplaced yes)
-		(property "Reference" "#PWR0351"
+		(property "Reference" "#PWR0355"
 			(at 114.3 92.71 0)
 			(effects
@@
 			(project "raywatch"
 				(path "/7b654ee8-2a53-4d39-8b7d-32c7bb3cb0ed/6e6a70ea-4db2-4b59-a2d7-c468f9b8b5a6/d00e072b-2be1-497b-8423-3eead973d996"
-					(reference "#PWR0351")
+					(reference "#PWR0355")
 					(unit 1)
 				)
@@
 		(dnp no)
 		(fields_autoplaced yes)
-		(property "Reference" "R38"
+		(property "Reference" "R39"
 			(at 167.64 69.85 90)
 			(effects
@@
 			(project "raywatch"
 				(path "/7b654ee8-2a53-4d39-8b7d-32c7bb3cb0ed/6e6a70ea-4db2-4b59-a2d7-c468f9b8b5a6/d00e072b-2be1-497b-8423-3eead973d996"
-					(reference "R38")
+					(reference "R39")
 					(unit 1)
 				)
@@
 		(dnp no)
 		(fields_autoplaced yes)
-		(property "Reference" "#PWR0349"
+		(property "Reference" "#PWR0353"
 			(at 113.03 110.49 0)
 			(effects
@@
 			(project "raywatch"
 				(path "/7b654ee8-2a53-4d39-8b7d-32c7bb3cb0ed/6e6a70ea-4db2-4b59-a2d7-c468f9b8b5a6/d00e072b-2be1-497b-8423-3eead973d996"
-					(reference "#PWR0349")
+					(reference "#PWR0353")
 					(unit 1)
 				)
@@
 		(dnp no)
 		(fields_autoplaced yes)
-		(property "Reference" "R39"
+		(property "Reference" "R40"
 			(at 167.64 78.74 90)
 			(effects
@@
 			(project "raywatch"
 				(path "/7b654ee8-2a53-4d39-8b7d-32c7bb3cb0ed/6e6a70ea-4db2-4b59-a2d7-c468f9b8b5a6/d00e072b-2be1-497b-8423-3eead973d996"
-					(reference "R39")
+					(reference "R40")
 					(unit 1)
 				)
@@
 		(dnp no)
 		(fields_autoplaced yes)
-		(property "Reference" "R35"
+		(property "Reference" "R36"
 			(at 99.06 88.9 90)
 			(effects
@@
 			(project "raywatch"
 				(path "/7b654ee8-2a53-4d39-8b7d-32c7bb3cb0ed/6e6a70ea-4db2-4b59-a2d7-c468f9b8b5a6/d00e072b-2be1-497b-8423-3eead973d996"
-					(reference "R35")
+					(reference "R36")
 					(unit 1)
 				)
@@
 		(dnp no)
 		(fields_autoplaced yes)
-		(property "Reference" "#PWR0346"
+		(property "Reference" "#PWR0350"
 			(at 48.26 119.38 0)
 			(effects
@@
 			(project "raywatch"
 				(path "/7b654ee8-2a53-4d39-8b7d-32c7bb3cb0ed/6e6a70ea-4db2-4b59-a2d7-c468f9b8b5a6/d00e072b-2be1-497b-8423-3eead973d996"
-					(reference "#PWR0346")
+					(reference "#PWR0350")
 					(unit 1)
 				)
@@
 		(dnp no)
 		(fields_autoplaced yes)
-		(property "Reference" "#PWR0348"
+		(property "Reference" "#PWR0352"
 			(at 95.25 104.14 0)
 			(effects
@@
 			(project "raywatch"
 				(path "/7b654ee8-2a53-4d39-8b7d-32c7bb3cb0ed/6e6a70ea-4db2-4b59-a2d7-c468f9b8b5a6/d00e072b-2be1-497b-8423-3eead973d996"
-					(reference "#PWR0348")
+					(reference "#PWR0352")
 					(unit 1)
 				)
@@
 		(dnp no)
 		(fields_autoplaced yes)
-		(property "Reference" "U25"
+		(property "Reference" "U26"
 			(at 138.43 74.93 0)
 			(effects
@@
 			(project "raywatch"
 				(path "/7b654ee8-2a53-4d39-8b7d-32c7bb3cb0ed/6e6a70ea-4db2-4b59-a2d7-c468f9b8b5a6/d00e072b-2be1-497b-8423-3eead973d996"
-					(reference "U25")
+					(reference "U26")
 					(unit 1)
 				)
@@
 		(dnp no)
 		(fields_autoplaced yes)
-		(property "Reference" "R36"
+		(property "Reference" "R37"
 			(at 116.84 96.52 90)
 			(effects
@@
 			(project "raywatch"
 				(path "/7b654ee8-2a53-4d39-8b7d-32c7bb3cb0ed/6e6a70ea-4db2-4b59-a2d7-c468f9b8b5a6/d00e072b-2be1-497b-8423-3eead973d996"
-					(reference "R36")
+					(reference "R37")
 					(unit 1)
 				)
@@
 		(dnp no)
 		(fields_autoplaced yes)
-		(property "Reference" "#PWR0350"
+		(property "Reference" "#PWR0354"
 			(at 114.3 90.17 0)
 			(effects
@@
 			(project "raywatch"
 				(path "/7b654ee8-2a53-4d39-8b7d-32c7bb3cb0ed/6e6a70ea-4db2-4b59-a2d7-c468f9b8b5a6/d00e072b-2be1-497b-8423-3eead973d996"
-					(reference "#PWR0350")
+					(reference "#PWR0354")
 					(unit 1)
 				)
@@
 		(dnp no)
 		(fields_autoplaced yes)
-		(property "Reference" "#PWR0345"
+		(property "Reference" "#PWR0349"
 			(at 43.18 119.38 0)
 			(effects
@@
 			(project "raywatch"
 				(path "/7b654ee8-2a53-4d39-8b7d-32c7bb3cb0ed/6e6a70ea-4db2-4b59-a2d7-c468f9b8b5a6/d00e072b-2be1-497b-8423-3eead973d996"
-					(reference "#PWR0345")
-					(unit 1)
-				)
+					(reference "#PWR0349")
+					(unit 1)
+				)

Commit message: Flattend hirachy
Parts:
- renumbered C84 to C100, C69 to C85, C70 to C86, C71 to C87, C72 to C88, C73 to C89, C74 to C90, C75 to C91, C76 to C92, C77 to C93, C78 to C94, C79 to C95, C80 to C96, C81 to C97, C82 to C98, C83 to C99, R36 to R46, R37 to R47, R38 to R48, R39 to R49, R40 to R50, U25 to U33, U26 to U34

Commit message: Assigned components
Parts:
- R46: value 200 -> 200Ω
Changed lines of the file:
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@@
+			)
+		)
+		(property "β(25/85)" ""
+			(at 201.93 86.36 0)
+			(effects
+				(font
+					(size 1.27 1.27)
+				)
+				(hide yes)
 			)
 		)
@@
 		)
 		(property "Max Voltage" "25V"
+			(at 234.95 115.57 90)
+			(effects
+				(font
+					(size 1.27 1.27)
+				)
+				(hide yes)
+			)
+		)
+		(property "β(25/85)" ""
 			(at 234.95 115.57 90)
 			(effects
@@
 			)
 		)
+		(property "β(25/85)" ""
+			(at 116.84 110.49 90)
+			(effects
+				(font
+					(size 1.27 1.27)
+				)
+				(hide yes)
+			)
+		)
 		(pin "1"
 		)
@@
 			)
 		)
+		(property "β(25/85)" ""
+			(at 242.57 102.87 90)
+			(effects
+				(font
+					(size 1.27 1.27)
+				)
+				(hide yes)
+			)
+		)
 		(pin "1"
 		)
@@
 		)
 		(property "Max Voltage " "25V"
+			(at 234.95 102.87 90)
+			(effects
+				(font
+					(size 1.27 1.27)
+				)
+				(hide yes)
+			)
+		)
+		(property "β(25/85)" ""
 			(at 234.95 102.87 90)
 			(effects
@@
 			)
 		)
+		(property "β(25/85)" ""
+			(at 48.26 109.22 0)
+			(effects
+				(font
+					(size 1.27 1.27)
+				)
+				(hide yes)
+			)
+		)
 		(pin "2"
 		)
@@
 		)
 		(property "Max Volt" "25V"
+			(at 242.57 97.79 90)
+			(effects
+				(font
+					(size 1.27 1.27)
+				)
+				(hide yes)
+			)
+		)
+		(property "β(25/85)" ""
 			(at 242.57 97.79 90)
 			(effects
@@
 			)
 		)
+		(property "β(25/85)" ""
+			(at 250.19 115.57 90)
+			(effects
+				(font
+					(size 1.27 1.27)
+				)
+				(hide yes)
+			)
+		)
 		(pin "1"
 		)
@@
 		)
 		(property "Description" "Unpolarized capacitor"
+			(at 168.91 106.68 0)
+			(effects
+				(font
+					(size 1.27 1.27)
+				)
+				(hide yes)
+			)
+		)
+		(property "β(25/85)" ""
 			(at 168.91 106.68 0)
 			(effects
@@
 			)
 		)
+		(property "β(25/85)" ""
+			(at 250.19 128.27 90)
+			(effects
+				(font
+					(size 1.27 1.27)
+				)
+				(hide yes)
+			)
+		)
 		(pin "1"
 		)
@@
 			)
 		)
+		(property "β(25/85)" ""
+			(at 224.79 86.36 0)
+			(effects
+				(font
+					(size 1.27 1.27)
+				)
+				(hide yes)
+			)
+		)
 		(pin "1"
 		)
@@
 			)
 		)
+		(property "β(25/85)" ""
+			(at 242.57 69.85 0)
+			(effects
+				(font
+					(size 1.27 1.27)
+				)
+				(hide yes)
+			)
+		)
 		(pin "2"
 		)
@@
 			)
 		)
+		(property "β(25/85)" ""
+			(at 237.49 86.36 0)
+			(effects
+				(font
+					(size 1.27 1.27)
+				)
+				(hide yes)
+			)
+		)
 		(pin "1"
 		)
@@
 			)
 		)
+		(property "β(25/85)" ""
+			(at 58.42 85.09 90)
+			(effects
+				(font
+					(size 1.27 1.27)
+				)
+				(hide yes)
+			)
+		)
 		(pin "C1"
 		)
@@
 			)
 		)
+		(property "β(25/85)" ""
+			(at 181.61 106.68 0)
+			(effects
+				(font
+					(size 1.27 1.27)
+				)
+				(hide yes)
+			)
+		)
 		(pin "2"
 		)
@@
 		)
 		(property "Max Voltage" "25V"
+			(at 234.95 128.27 90)
+			(effects
+				(font
+					(size 1.27 1.27)
+				)
+				(hide yes)
+			)
+		)
+		(property "β(25/85)" ""
 			(at 234.95 128.27 90)
 			(effects
@@
 			)
 		)
+		(property "β(25/85)" ""
+			(at 167.64 76.2 90)
+			(effects
+				(font
+					(size 1.27 1.27)
+				)
+				(hide yes)
+			)
+		)
 		(pin "1"
 		)
@@
 			)
 		)
+		(property "β(25/85)" ""
+			(at 250.19 102.87 90)
+			(effects
+				(font
+					(size 1.27 1.27)
+				)
+				(hide yes)
+			)
+		)
 		(pin "1"
 		)
@@
 			)
 		)
+		(property "β(25/85)" ""
+			(at 43.18 109.22 0)
+			(effects
+				(font
+					(size 1.27 1.27)
+				)
+				(hide yes)
+			)
+		)
 		(pin "2"
 		)
@@
 			)
 		)
+		(property "β(25/85)" ""
+			(at 167.64 85.09 90)
+			(effects
+				(font
+					(size 1.27 1.27)
+				)
+				(hide yes)
+			)
+		)
 		(pin "1"
 		)
@@
 			)
 		)
-		(property "Value" "200"
+		(property "Value" "200Ω"
 			(at 99.06 91.44 90)
 			(effects
@@
 		(property "Description" "Resistor"
 			(at 99.06 95.25 0)
+			(effects
+				(font
+					(size 1.27 1.27)
+				)
+				(hide yes)
+			)
+		)
+		(property "β(25/85)" ""
+			(at 99.06 95.25 90)
 			(effects
 				(font
@@
 			)
 		)
+		(property "β(25/85)" ""
+			(at 213.36 86.36 0)
+			(effects
+				(font
+					(size 1.27 1.27)
+				)
+				(hide yes)
+			)
+		)
 		(pin "1"
 		)
@@
 			)
 		)
+		(property "β(25/85)" ""
+			(at 138.43 102.87 0)
+			(effects
+				(font
+					(size 1.27 1.27)
+				)
+				(hide yes)
+			)
+		)
 		(pin "28"
 		)
@@
 			(effects
 				(font
+					(size 1.27 1.27)
+				)
+				(hide yes)
+			)
+		)
+		(property "β(25/85)" ""
+			(at 116.84 102.87 90)
+			(effects
+				(font

Commit message: Changed footprints from 0603 to 0402
Parts:
- C100, C85, C86, C87, C88, C89, C90, C91, C92, C93, C94, C95, C96, C97, C98, C99: footprint Capacitor_SMD:C_0603_1608Metric -> Capacitor_SMD:C_0504_1310Metric
- R46, R47, R48, R49, R50: footprint Resistor_SMD:R_0603_1608Metric -> Resistor_SMD:R_0402_1005Metric
Changed lines of the file:
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@@
 			)
 		)
-		(property "Footprint" "Capacitor_SMD:C_0603_1608Metric"
+		(property "Footprint" "Capacitor_SMD:C_0504_1310Metric"
 			(at 200.9648 82.55 0)
 			(effects
@@
 			)
 		)
-		(property "Footprint" "Capacitor_SMD:C_0603_1608Metric"
+		(property "Footprint" "Capacitor_SMD:C_0504_1310Metric"
 			(at 238.76 114.6048 0)
 			(effects
@@
 			)
 		)
-		(property "Footprint" "Resistor_SMD:R_0603_1608Metric"
+		(property "Footprint" "Resistor_SMD:R_0402_1005Metric"
 			(at 116.84 112.268 90)
 			(effects
@@
 			)
 		)
-		(property "Footprint" "Capacitor_SMD:C_0603_1608Metric"
+		(property "Footprint" "Capacitor_SMD:C_0504_1310Metric"
 			(at 246.38 101.9048 0)
 			(effects
@@
 			)
 		)
-		(property "Footprint" "Capacitor_SMD:C_0603_1608Metric"
+		(property "Footprint" "Capacitor_SMD:C_0504_1310Metric"
 			(at 238.76 101.9048 0)
 			(effects
@@
 			)
 		)
-		(property "Footprint" "Capacitor_SMD:C_0603_1608Metric"
+		(property "Footprint" "Capacitor_SMD:C_0504_1310Metric"
 			(at 49.2252 105.41 0)
 			(effects
@@
 			)
 		)
-		(property "Footprint" "Capacitor_SMD:C_0603_1608Metric"
+		(property "Footprint" "Capacitor_SMD:C_0504_1310Metric"
 			(at 246.38 96.8248 0)
 			(effects
@@
 			)
 		)
-		(property "Footprint" "Capacitor_SMD:C_0603_1608Metric"
+		(property "Footprint" "Capacitor_SMD:C_0504_1310Metric"
 			(at 246.38 114.6048 0)
 			(effects
@@
 			)
 		)
-		(property "Footprint" "Capacitor_SMD:C_0603_1608Metric"
+		(property "Footprint" "Capacitor_SMD:C_0504_1310Metric"
 			(at 169.8752 110.49 0)
 			(effects
@@
 			)
 		)
-		(property "Footprint" "Capacitor_SMD:C_0603_1608Metric"
+		(property "Footprint" "Capacitor_SMD:C_0504_1310Metric"
 			(at 246.38 127.3048 0)
 			(effects
@@
 			)
 		)
-		(property "Footprint" "Capacitor_SMD:C_0603_1608Metric"
+		(property "Footprint" "Capacitor_SMD:C_0504_1310Metric"
 			(at 223.8248 82.55 0)
 			(effects
@@
 			)
 		)
-		(property "Footprint" "Capacitor_SMD:C_0603_1608Metric"
+		(property "Footprint" "Capacitor_SMD:C_0504_1310Metric"
 			(at 236.5248 82.55 0)
 			(effects
@@
 			)
 		)
-		(property "Footprint" "Capacitor_SMD:C_0603_1608Metric"
+		(property "Footprint" "Capacitor_SMD:C_0504_1310Metric"
 			(at 182.5752 110.49 0)
 			(effects
@@
 			)
 		)
-		(property "Footprint" "Capacitor_SMD:C_0603_1608Metric"
+		(property "Footprint" "Capacitor_SMD:C_0504_1310Metric"
 			(at 238.76 127.3048 0)
 			(effects
@@
 			)
 		)
-		(property "Footprint" "Resistor_SMD:R_0603_1608Metric"
+		(property "Footprint" "Resistor_SMD:R_0402_1005Metric"
 			(at 167.64 77.978 90)
 			(effects
@@
 			)
 		)
-		(property "Footprint" "Capacitor_SMD:C_0603_1608Metric"
+		(property "Footprint" "Capacitor_SMD:C_0504_1310Metric"
 			(at 246.38 101.9048 0)
 			(effects
@@
 			)
 		)
-		(property "Footprint" "Capacitor_SMD:C_0603_1608Metric"
+		(property "Footprint" "Capacitor_SMD:C_0504_1310Metric"
 			(at 44.1452 105.41 0)
 			(effects
@@
 			)
 		)
-		(property "Footprint" "Resistor_SMD:R_0603_1608Metric"
+		(property "Footprint" "Resistor_SMD:R_0402_1005Metric"
 			(at 167.64 86.868 90)
 			(effects
@@
 			)
 		)
-		(property "Footprint" "Resistor_SMD:R_0603_1608Metric"
+		(property "Footprint" "Resistor_SMD:R_0402_1005Metric"
 			(at 99.06 93.472 90)
 			(effects
@@
 			)
 		)
-		(property "Footprint" "Capacitor_SMD:C_0603_1608Metric"
+		(property "Footprint" "Capacitor_SMD:C_0504_1310Metric"
 			(at 212.3948 82.55 0)
 			(effects
@@
 			)
 		)
-		(property "Footprint" "Resistor_SMD:R_0603_1608Metric"
+		(property "Footprint" "Resistor_SMD:R_0402_1005Metric"
 			(at 116.84 101.092 90)
 			(effects

Commit message: Replaced global labels with pin headers
Parts:
- added J12, J13, J4: Conn_01x02_Pin, symbol Connector:Conn_01x02_Pin
Connections:
- net EXP: now also J12.2 (Pin_2), J4.2 (Pin_2)
- net SOLARSTAT: now also J13.1 (Pin_1)
- net VIN: now also J12.1 (Pin_1)
- net VSOLAR: now also J4.1 (Pin_1)
- net WCDET: now also J13.2 (Pin_2)

Commit message: Reannotated schematic
Parts:
- renumbered C85 to C80, C86 to C81, C87 to C82, C88 to C83, C89 to C84, C90 to C85, C91 to C86, C92 to C87, C93 to C88, C94 to C89, C95 to C90, C96 to C91, C97 to C92, C98 to C93, C99 to C94, C100 to C95, J4 to J89, J12 to J90, J13 to J91, R46 to R40, R47 to R41, R48 to R42, R49 to R43, R50 to R44, U33 to U34, U34 to U35

Commit message: Assigned pin header footprints
Parts:
- J89, J90, J91: footprint (none) -> Connector_PinHeader_2.54mm:PinHeader_1x02_P2.54mm_Horizontal
Changed lines of the file:
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@@
 			)
 		)
-		(property "Footprint" ""
+		(property "Footprint" "Connector_PinHeader_2.54mm:PinHeader_1x02_P2.54mm_Horizontal"
 			(at 99.06 39.37 0)
 			(effects
@@
 			)
 		)
-		(property "Footprint" ""
+		(property "Footprint" "Connector_PinHeader_2.54mm:PinHeader_1x02_P2.54mm_Horizontal"
 			(at 99.06 48.26 0)
 			(effects
@@
 			)
 		)
-		(property "Footprint" ""
+		(property "Footprint" "Connector_PinHeader_2.54mm:PinHeader_1x02_P2.54mm_Horizontal"
 			(at 99.06 31.75 0)
 			(effects
