File: src/hardware/proximity_gesture.kicad_sch (KiCad schematic)
At the start: 16 parts, among them U37 APDS-9500, Y5 SG-210STF_24.0000ML0

Commit message: Selected S1..10 & TR1
Parts:
- C103, C104, C105, C106, C107, C108, C109, C110, C111, C112, C113, C114: footprint (none) -> Capacitor_SMD:C_0603_1608Metric
- R51: footprint (none) -> Resistor_SMD:R_0603_1608Metric
Changed lines of the file:
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@@
 			)
 		)
-		(property "Footprint" ""
+		(property "Footprint" "Capacitor_SMD:C_0603_1608Metric"
 			(at 210.5152 107.95 0)
 			(effects
@@
 			)
 		)
-		(property "Footprint" ""
+		(property "Footprint" "Capacitor_SMD:C_0603_1608Metric"
 			(at 193.3448 69.85 0)
 			(effects
@@
 			)
 		)
-		(property "Footprint" ""
+		(property "Footprint" "Capacitor_SMD:C_0603_1608Metric"
 			(at 223.2152 87.63 0)
 			(effects
@@
 			)
 		)
-		(property "Footprint" ""
+		(property "Footprint" "Capacitor_SMD:C_0603_1608Metric"
 			(at 195.2752 138.43 0)
 			(effects
@@
 			)
 		)
-		(property "Footprint" ""
+		(property "Footprint" "Capacitor_SMD:C_0603_1608Metric"
 			(at 221.9452 107.95 0)
 			(effects
@@
 			)
 		)
-		(property "Footprint" ""
+		(property "Footprint" "Capacitor_SMD:C_0603_1608Metric"
 			(at 207.9752 138.43 0)
 			(effects
@@
 			)
 		)
-		(property "Footprint" ""
+		(property "Footprint" "Capacitor_SMD:C_0603_1608Metric"
 			(at 234.6452 87.63 0)
 			(effects
@@
 			)
 		)
-		(property "Footprint" ""
+		(property "Footprint" "Capacitor_SMD:C_0603_1608Metric"
 			(at 165.4048 69.85 0)
 			(effects
@@
 			)
 		)
-		(property "Footprint" ""
+		(property "Footprint" "Capacitor_SMD:C_0603_1608Metric"
 			(at 200.3552 69.85 0)
 			(effects
@@
 			)
 		)
-		(property "Footprint" ""
+		(property "Footprint" "Capacitor_SMD:C_0603_1608Metric"
 			(at 172.4152 69.85 0)
 			(effects
@@
 			)
 		)
-		(property "Footprint" ""
+		(property "Footprint" "Resistor_SMD:R_0603_1608Metric"
 			(at 140.462 93.98 90)
 			(effects
@@
 			)
 		)
-		(property "Footprint" ""
+		(property "Footprint" "Capacitor_SMD:C_0603_1608Metric"
 			(at 182.5752 138.43 0)
 			(effects
@@
 			)
 		)
-		(property "Footprint" ""
+		(property "Footprint" "Capacitor_SMD:C_0603_1608Metric"
 			(at 110.1852 111.76 0)
 			(effects

Commit message: Cleanup
Parts:
- R51: value 10k -> 10kΩ
Changed lines of the file:
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@@
 			)
 		)
-		(property "Value" "10k"
+		(property "Value" "10kΩ"
 			(at 144.78 95.2499 0)
 			(effects

Commit message: Assigned components
Other:
- moved on the sheet: R51
Changed lines of the file:
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@@
 	)
 	(junction
+		(at 140.97 97.79)
+		(diameter 0)
+		(color 0 0 0 0)
+	)
+	(junction
 		(at 194.31 62.23)
 		(diameter 0)
@@
 	)
 	(junction
-		(at 142.24 97.79)
-		(diameter 0)
-		(color 0 0 0 0)
-	)
-	(junction
 		(at 220.98 100.33)
 		(diameter 0)
@@
 	(wire
 		(pts
-			(xy 142.24 97.79) (xy 156.21 97.79)
+			(xy 207.01 128.27) (xy 191.77 128.27)
 		)
 		(stroke
@@
 	(wire
 		(pts
-			(xy 207.01 128.27) (xy 191.77 128.27)
+			(xy 186.69 130.81) (xy 194.31 130.81)
 		)
 		(stroke
@@
 	(wire
 		(pts
-			(xy 186.69 130.81) (xy 194.31 130.81)
+			(xy 140.97 97.79) (xy 156.21 97.79)
 		)
 		(stroke
@@
 	(wire
 		(pts
-			(xy 139.7 97.79) (xy 142.24 97.79)
+			(xy 138.43 97.79) (xy 140.97 97.79)
 		)
 		(stroke
@@
 	(global_label "IRINT"
 		(shape output)
-		(at 139.7 97.79 180)
+		(at 138.43 97.79 180)
 		(fields_autoplaced yes)
 		(effects
@@
 		)
 		(property "Intersheetrefs" "${INTERSHEET_REFS}"
-			(at 131.9371 97.79 0)
+			(at 130.6671 97.79 0)
 			(effects
 				(font
@@
 			)
 		)
+		(property "β(25/85)" ""
+			(at 209.55 104.14 0)
+			(effects
+				(font
+					(size 1.27 1.27)
+				)
+				(hide yes)
+			)
+		)
 		(pin "2"
 		)
@@
 			)
 		)
+		(property "β(25/85)" ""
+			(at 194.31 66.04 0)
+			(effects
+				(font
+					(size 1.27 1.27)
+				)
+				(hide yes)
+			)
+		)
 		(pin "2"
 		)
@@
 			)
 		)
+		(property "β(25/85)" ""
+			(at 222.25 91.44 0)
+			(effects
+				(font
+					(size 1.27 1.27)
+				)
+				(hide yes)
+			)
+		)
 		(pin "2"
 		)
@@
 			)
 		)
+		(property "β(25/85)" ""
+			(at 85.09 109.22 0)
+			(effects
+				(font
+					(size 1.27 1.27)
+				)
+				(hide yes)
+			)
+		)
 		(pin "3"
 		)
@@
 	(symbol
 		(lib_id "power:+3V3")
-		(at 142.24 90.17 0)
+		(at 140.97 90.17 0)
 		(unit 1)
 		(exclude_from_sim no)
@@
 		(fields_autoplaced yes)
 		(property "Reference" "#PWR0419"
-			(at 142.24 93.98 0)
+			(at 140.97 93.98 0)
 			(effects
 				(font
@@
 		)
 		(property "Value" "+3V3"
-			(at 142.24 85.09 0)
+			(at 140.97 85.09 0)
 			(effects
 				(font
@@
 		)
 		(property "Footprint" ""
-			(at 142.24 90.17 0)
+			(at 140.97 90.17 0)
 			(effects
 				(font
@@
 		)
 		(property "Datasheet" ""
-			(at 142.24 90.17 0)
+			(at 140.97 90.17 0)
 			(effects
 				(font
@@
 		)
 		(property "Description" "Power symbol creates a global label with name \"+3V3\""
-			(at 142.24 90.17 0)
+			(at 140.97 90.17 0)
 			(effects
 				(font
@@
 			)
 		)
+		(property "β(25/85)" ""
+			(at 214.63 95.25 0)
+			(effects
+				(font
+					(size 1.27 1.27)
+				)
+				(hide yes)
+			)
+		)
 		(pin "A"
 		)
@@
 			)
 		)
+		(property "β(25/85)" ""
+			(at 194.31 134.62 0)
+			(effects
+				(font
+					(size 1.27 1.27)
+				)
+				(hide yes)
+			)
+		)
 		(pin "2"
 		)
@@
 			)
 		)
+		(property "β(25/85)" ""
+			(at 179.07 105.41 0)
+			(effects
+				(font
+					(size 1.27 1.27)
+				)
+				(hide yes)
+			)
+		)
 		(pin "14"
 		)
@@
 			)
 		)
+		(property "β(25/85)" ""
+			(at 220.98 104.14 0)
+			(effects
+				(font
+					(size 1.27 1.27)
+				)
+				(hide yes)
+			)
+		)
 		(pin "2"
 		)
@@
 			)
 		)
+		(property "β(25/85)" ""
+			(at 207.01 134.62 0)
+			(effects
+				(font
+					(size 1.27 1.27)
+				)
+				(hide yes)
+			)
+		)
 		(pin "2"
 		)
@@
 			)
 		)
+		(property "β(25/85)" ""
+			(at 233.68 91.44 0)
+			(effects
+				(font
+					(size 1.27 1.27)
+				)
+				(hide yes)
+			)
+		)
 		(pin "2"
 		)
@@
 			)
 		)
+		(property "β(25/85)" ""
+			(at 166.37 66.04 0)
+			(effects
+				(font
+					(size 1.27 1.27)
+				)
+				(hide yes)
+			)
+		)
 		(pin "2"
 		)
@@
 			)
 		)
+		(property "β(25/85)" ""
+			(at 199.39 66.04 0)
+			(effects
+				(font
+					(size 1.27 1.27)
+				)
+				(hide yes)
+			)
+		)
 		(pin "2"
 		)
@@
 			)
 		)
+		(property "β(25/85)" ""
+			(at 171.45 66.04 0)
+			(effects
+				(font
+					(size 1.27 1.27)
+				)
+				(hide yes)
+			)
+		)
 		(pin "2"
 		)
@@
 	(symbol
 		(lib_id "Device:R")
-		(at 142.24 93.98 0)
+		(at 140.97 93.98 0)
 		(unit 1)
 		(exclude_from_sim no)
@@
 		(fields_autoplaced yes)
 		(property "Reference" "R51"
-			(at 144.78 92.7099 0)
+			(at 143.51 92.7099 0)
 			(effects
 				(font
@@
 		)
 		(property "Value" "10kΩ"
-			(at 144.78 95.2499 0)
+			(at 143.51 95.2499 0)
 			(effects
 				(font
@@
 		)
 		(property "Footprint" "Resistor_SMD:R_0603_1608Metric"
-			(at 140.462 93.98 90)
+			(at 139.192 93.98 90)
 			(effects
 				(font
@@
 		)
 		(property "Datasheet" "~"
-			(at 142.24 93.98 0)
+			(at 140.97 93.98 0)
 			(effects
 				(font
@@
 		)
 		(property "Description" "Resistor"
-			(at 142.24 93.98 0)
+			(at 140.97 93.98 0)
+			(effects
+				(font
+					(size 1.27 1.27)
+				)
+				(hide yes)
+			)
+		)
+		(property "β(25/85)" ""
+			(at 140.97 93.98 0)
 			(effects
 				(font
@@
 			)
 		)
+		(property "β(25/85)" ""
+			(at 181.61 134.62 0)
+			(effects
+				(font
+					(size 1.27 1.27)
+				)
+				(hide yes)
+			)
+		)
 		(pin "2"
 		)
@@
 			(at 109.22 107.95 0)
 			(effects
+				(font
+					(size 1.27 1.27)
+				)
+				(hide yes)
+			)
+		)
+		(property "β(25/85)" ""
+			(at 109.22 107.95 0)
+			(effects

Commit message: Changed footprints from 0603 to 0402
Parts:
- C103, C104, C105, C106, C107, C108, C109, C110, C111, C112, C113, C114: footprint Capacitor_SMD:C_0603_1608Metric -> Capacitor_SMD:C_0504_1310Metric
- R51: footprint Resistor_SMD:R_0603_1608Metric -> Resistor_SMD:R_0402_1005Metric
Changed lines of the file:
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@@
 			)
 		)
-		(property "Footprint" "Capacitor_SMD:C_0603_1608Metric"
+		(property "Footprint" "Capacitor_SMD:C_0504_1310Metric"
 			(at 210.5152 107.95 0)
 			(effects
@@
 			)
 		)
-		(property "Footprint" "Capacitor_SMD:C_0603_1608Metric"
+		(property "Footprint" "Capacitor_SMD:C_0504_1310Metric"
 			(at 193.3448 69.85 0)
 			(effects
@@
 			)
 		)
-		(property "Footprint" "Capacitor_SMD:C_0603_1608Metric"
+		(property "Footprint" "Capacitor_SMD:C_0504_1310Metric"
 			(at 223.2152 87.63 0)
 			(effects
@@
 			)
 		)
-		(property "Footprint" "Capacitor_SMD:C_0603_1608Metric"
+		(property "Footprint" "Capacitor_SMD:C_0504_1310Metric"
 			(at 195.2752 138.43 0)
 			(effects
@@
 			)
 		)
-		(property "Footprint" "Capacitor_SMD:C_0603_1608Metric"
+		(property "Footprint" "Capacitor_SMD:C_0504_1310Metric"
 			(at 221.9452 107.95 0)
 			(effects
@@
 			)
 		)
-		(property "Footprint" "Capacitor_SMD:C_0603_1608Metric"
+		(property "Footprint" "Capacitor_SMD:C_0504_1310Metric"
 			(at 207.9752 138.43 0)
 			(effects
@@
 			)
 		)
-		(property "Footprint" "Capacitor_SMD:C_0603_1608Metric"
+		(property "Footprint" "Capacitor_SMD:C_0504_1310Metric"
 			(at 234.6452 87.63 0)
 			(effects
@@
 			)
 		)
-		(property "Footprint" "Capacitor_SMD:C_0603_1608Metric"
+		(property "Footprint" "Capacitor_SMD:C_0504_1310Metric"
 			(at 165.4048 69.85 0)
 			(effects
@@
 			)
 		)
-		(property "Footprint" "Capacitor_SMD:C_0603_1608Metric"
+		(property "Footprint" "Capacitor_SMD:C_0504_1310Metric"
 			(at 200.3552 69.85 0)
 			(effects
@@
 			)
 		)
-		(property "Footprint" "Capacitor_SMD:C_0603_1608Metric"
+		(property "Footprint" "Capacitor_SMD:C_0504_1310Metric"
 			(at 172.4152 69.85 0)
 			(effects
@@
 			)
 		)
-		(property "Footprint" "Resistor_SMD:R_0603_1608Metric"
+		(property "Footprint" "Resistor_SMD:R_0402_1005Metric"
 			(at 139.192 93.98 90)
 			(effects
@@
 			)
 		)
-		(property "Footprint" "Capacitor_SMD:C_0603_1608Metric"
+		(property "Footprint" "Capacitor_SMD:C_0504_1310Metric"
 			(at 182.5752 138.43 0)
 			(effects
@@
 			)
 		)
-		(property "Footprint" "Capacitor_SMD:C_0603_1608Metric"
+		(property "Footprint" "Capacitor_SMD:C_0504_1310Metric"
 			(at 110.1852 111.76 0)
 			(effects

Commit message: Replaced global labels with pin headers
Parts:
- added J10, J11, J7, J8: Conn_01x02_Pin, symbol Connector:Conn_01x02_Pin
- added J9: Conn_01x04_Pin, symbol Connector:Conn_01x04_Pin
Connections:
- net +3V3: now also J10.1 (Pin_1)
- net +4V5: now also J11.1 (Pin_1)
- net GND: now also J10.2 (Pin_2), J11.2 (Pin_2)
- net IRCLKEN: now also J8.2 (Pin_2)
- net IRINT: now also J8.1 (Pin_1)
- net MISO: now also J9.3 (Pin_3)
- net SCK: now also J9.1 (Pin_1)
- net SCL: now also J7.1 (Pin_1)
- net SDA: now also J7.2 (Pin_2)
- net IRCS renamed CS
- net CS: now also J9.4 (Pin_4)
- no-connect marks 2 -> 3

Commit message: Reannotated schematic
Parts:
- renumbered C106 to C100, C107 to C101, C108 to C102, C109 to C103, C110 to C104, C111 to C105, C112 to C106, C113 to C107, C114 to C108, C103 to C97, C104 to C98, C105 to C99, J10 to J94, J11 to J95, J8 to J96, J7 to J97, J9 to J98, R51 to R45

Commit message: Assigned pin header footprints
Parts:
- J94, J95, J96, J97: footprint (none) -> Connector_PinHeader_2.54mm:PinHeader_1x02_P2.54mm_Horizontal
- J98: footprint (none) -> Connector_PinHeader_2.54mm:PinHeader_1x04_P2.54mm_Horizontal
Changed lines of the file:
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@@
 			)
 		)
-		(property "Footprint" ""
+		(property "Footprint" "Connector_PinHeader_2.54mm:PinHeader_1x02_P2.54mm_Horizontal"
 			(at 101.6 57.15 0)
 			(effects
@@
 			)
 		)
-		(property "Footprint" ""
+		(property "Footprint" "Connector_PinHeader_2.54mm:PinHeader_1x02_P2.54mm_Horizontal"
 			(at 100.33 34.29 0)
 			(effects
@@
 			)
 		)
-		(property "Footprint" ""
+		(property "Footprint" "Connector_PinHeader_2.54mm:PinHeader_1x02_P2.54mm_Horizontal"
 			(at 100.33 41.91 0)
 			(effects
@@
 			)
 		)
-		(property "Footprint" ""
+		(property "Footprint" "Connector_PinHeader_2.54mm:PinHeader_1x04_P2.54mm_Horizontal"
 			(at 101.6 67.31 0)
 			(effects
@@
 			)
 		)
-		(property "Footprint" ""
+		(property "Footprint" "Connector_PinHeader_2.54mm:PinHeader_1x02_P2.54mm_Horizontal"
 			(at 101.6 49.53 0)
 			(effects
