File: src/hardware/leds.kicad_sch (KiCad schematic)
At the start: 75 parts, among them U8 SN74AHCT1G125DBVR, U9 TPS22916BYFPR

Commit message: Changed footprints from 0603 to 0402
Parts:
- C30: footprint Capacitor_SMD:C_0603_1608Metric -> Capacitor_SMD:C_0504_1310Metric
Changed lines of the file:
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@@
 			)
 		)
-		(property "Footprint" "Capacitor_SMD:C_0603_1608Metric"
+		(property "Footprint" "Capacitor_SMD:C_0504_1310Metric"
 			(at 100.6348 172.72 0)
 			(effects

Commit message: Replaced global labels with pin headers
Parts:
- added J63, J64: Conn_01x02_Pin, symbol Connector:Conn_01x02_Pin
Connections:
- net +4V5: now also J63.1 (Pin_1)
- net GND: now also J63.2 (Pin_2)
- net LEDDIN: now also J64.2 (Pin_2)
- net LEDEN: now also J64.1 (Pin_1)

Commit message: Reannotated schematic
Parts:
- renumbered C30 to C24, J63 to J35, J64 to J36

Commit message: Assigned pin header footprints
Parts:
- J35, J36: footprint (none) -> Connector_PinHeader_2.54mm:PinHeader_1x02_P2.54mm_Horizontal
Changed lines of the file:
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@@
 			)
 		)
-		(property "Footprint" ""
+		(property "Footprint" "Connector_PinHeader_2.54mm:PinHeader_1x02_P2.54mm_Horizontal"
 			(at 83.82 147.32 0)
 			(effects
@@
 			)
 		)
-		(property "Footprint" ""
+		(property "Footprint" "Connector_PinHeader_2.54mm:PinHeader_1x02_P2.54mm_Horizontal"
 			(at 59.69 147.32 0)
 			(effects

Commit message: Reannotate
Parts:
- renumbered U8 to U7, U9 to U8
Changed lines of the file:
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@@
 		(dnp no)
 		(fields_autoplaced yes)
-		(property "Reference" "U8"
+		(property "Reference" "U7"
 			(at 63.5 157.48 0)
 			(effects
@@
 			(project "raywatch"
 				(path "/7b654ee8-2a53-4d39-8b7d-32c7bb3cb0ed/0600b049-21d1-41d4-ba88-3a8142850263"
-					(reference "U8")
+					(reference "U7")
 					(unit 1)
 				)
@@
 		(dnp no)
 		(fields_autoplaced yes)
-		(property "Reference" "U9"
+		(property "Reference" "U8"
 			(at 144.78 162.56 0)
 			(effects
@@
 			(project "raywatch"
 				(path "/7b654ee8-2a53-4d39-8b7d-32c7bb3cb0ed/0600b049-21d1-41d4-ba88-3a8142850263"
-					(reference "U9")
-					(unit 1)
-				)
+					(reference "U8")
+					(unit 1)
+				)

Commit message: Changed pin headers to vertical
Parts:
- J35, J36: footprint Connector_PinHeader_2.54mm:PinHeader_1x02_P2.54mm_Horizontal -> Connector_PinHeader_2.54mm:PinHeader_1x02_P2.54mm_Vertical
Changed lines of the file:
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@@
 			)
 		)
-		(property "Footprint" "Connector_PinHeader_2.54mm:PinHeader_1x02_P2.54mm_Horizontal"
+		(property "Footprint" "Connector_PinHeader_2.54mm:PinHeader_1x02_P2.54mm_Vertical"
 			(at 83.82 147.32 0)
 			(effects
@@
 			)
 		)
-		(property "Footprint" "Connector_PinHeader_2.54mm:PinHeader_1x02_P2.54mm_Horizontal"
+		(property "Footprint" "Connector_PinHeader_2.54mm:PinHeader_1x02_P2.54mm_Vertical"
 			(at 59.69 147.32 0)
 			(effects

Commit message: Fixed connector footprints; Changed conectors from 2.54 to 1.27
Parts:
- J33: renamed from J35; footprint Connector_PinHeader_2.54mm:PinHeader_1x02_P2.54mm_Vertical -> Connector_PinHeader_1.27mm:PinHeader_1x02_P1.27mm_Vertical
- J34: renamed from J36; footprint Connector_PinHeader_2.54mm:PinHeader_1x02_P2.54mm_Vertical -> Connector_PinHeader_1.27mm:PinHeader_1x02_P1.27mm_Vertical
