File: src/hardware/light_sensor.kicad_sch (KiCad schematic)
At the start: 4 parts, among them J67 Conn_01x02_Pin, J68 Conn_01x02_Pin, U24 LTR-329ALS-01

Commit message: Fixed connector footprints; Changed conectors from 2.54 to 1.27
Parts:
- J65: renamed from J67; footprint Connector_PinHeader_2.54mm:PinHeader_1x02_P2.54mm_Vertical -> Connector_PinHeader_1.27mm:PinHeader_1x02_P1.27mm_Vertical
- J66: renamed from J68; footprint Connector_PinHeader_2.54mm:PinHeader_1x02_P2.54mm_Vertical -> Connector_PinHeader_1.27mm:PinHeader_1x02_P1.27mm_Vertical
Changed lines of the file:
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@@
 		(dnp no)
 		(fields_autoplaced yes)
-		(property "Reference" "#PWR0364"
+		(property "Reference" "#PWR0366"
 			(at 165.1 115.57 0)
 			(effects
@@
 			(project "raywatch"
 				(path "/7b654ee8-2a53-4d39-8b7d-32c7bb3cb0ed/d5a2fc90-5630-482b-949a-d1a5e12221d9"
-					(reference "#PWR0364")
+					(reference "#PWR0366")
 					(unit 1)
 				)
@@
 		(dnp no)
 		(fields_autoplaced yes)
-		(property "Reference" "#PWR0361"
+		(property "Reference" "#PWR0363"
 			(at 105.41 66.04 0)
 			(effects
@@
 			(project "raywatch"
 				(path "/7b654ee8-2a53-4d39-8b7d-32c7bb3cb0ed/d5a2fc90-5630-482b-949a-d1a5e12221d9"
-					(reference "#PWR0361")
+					(reference "#PWR0363")
 					(unit 1)
 				)
@@
 		(dnp no)
 		(fields_autoplaced yes)
-		(property "Reference" "#PWR0363"
+		(property "Reference" "#PWR0365"
 			(at 165.1 100.33 0)
 			(effects
@@
 			(project "raywatch"
 				(path "/7b654ee8-2a53-4d39-8b7d-32c7bb3cb0ed/d5a2fc90-5630-482b-949a-d1a5e12221d9"
-					(reference "#PWR0363")
+					(reference "#PWR0365")
 					(unit 1)
 				)
@@
 		(dnp no)
 		(fields_autoplaced yes)
-		(property "Reference" "J68"
+		(property "Reference" "J66"
 			(at 104.775 72.39 0)
 			(effects
@@
 			)
 		)
-		(property "Footprint" "Connector_PinHeader_2.54mm:PinHeader_1x02_P2.54mm_Vertical"
+		(property "Footprint" "Connector_PinHeader_1.27mm:PinHeader_1x02_P1.27mm_Vertical"
 			(at 104.14 77.47 0)
 			(effects
@@
 			(project "raywatch"
 				(path "/7b654ee8-2a53-4d39-8b7d-32c7bb3cb0ed/d5a2fc90-5630-482b-949a-d1a5e12221d9"
-					(reference "J68")
+					(reference "J66")
 					(unit 1)
 				)
@@
 		(dnp no)
 		(fields_autoplaced yes)
-		(property "Reference" "#PWR0362"
+		(property "Reference" "#PWR0364"
 			(at 115.57 68.58 0)
 			(effects
@@
 			(project "raywatch"
 				(path "/7b654ee8-2a53-4d39-8b7d-32c7bb3cb0ed/d5a2fc90-5630-482b-949a-d1a5e12221d9"
-					(reference "#PWR0362")
+					(reference "#PWR0364")
 					(unit 1)
 				)
@@
 		(dnp no)
 		(fields_autoplaced yes)
-		(property "Reference" "J67"
+		(property "Reference" "J65"
 			(at 104.775 60.96 0)
 			(effects
@@
 			)
 		)
-		(property "Footprint" "Connector_PinHeader_2.54mm:PinHeader_1x02_P2.54mm_Vertical"
+		(property "Footprint" "Connector_PinHeader_1.27mm:PinHeader_1x02_P1.27mm_Vertical"
 			(at 104.14 66.04 0)
 			(effects
@@
 			(project "raywatch"
 				(path "/7b654ee8-2a53-4d39-8b7d-32c7bb3cb0ed/d5a2fc90-5630-482b-949a-d1a5e12221d9"
-					(reference "J67")
-					(unit 1)
-				)
+					(reference "J65")
+					(unit 1)
+				)

Commit message: Fixes; Added TPM PCB
Parts:
- C60: footprint Capacitor_SMD:C_0504_1310Metric -> Capacitor_SMD:C_0402_1005Metric
Changed lines of the file:
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@@
 			)
 		)
-		(property "Footprint" "Capacitor_SMD:C_0504_1310Metric"
+		(property "Footprint" "Capacitor_SMD:C_0402_1005Metric"
 			(at 166.0652 104.14 0)
 			(effects
