File: src/hardware/magnetometer.kicad_sch (KiCad schematic)
At the start: 4 parts, among them U18 MMC34160PJ

Commit message: Changed footprints from 0603 to 0402
Parts:
- C51, C52, C53: footprint Capacitor_SMD:C_0603_1608Metric -> Capacitor_SMD:C_0504_1310Metric
Changed lines of the file:
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@@
 			)
 		)
-		(property "Footprint" "Capacitor_SMD:C_0603_1608Metric"
+		(property "Footprint" "Capacitor_SMD:C_0504_1310Metric"
 			(at 119.0752 102.87 0)
 			(effects
@@
 			)
 		)
-		(property "Footprint" "Capacitor_SMD:C_0603_1608Metric"
+		(property "Footprint" "Capacitor_SMD:C_0504_1310Metric"
 			(at 169.8752 100.33 0)
 			(effects
@@
 			)
 		)
-		(property "Footprint" "Capacitor_SMD:C_0603_1608Metric"
+		(property "Footprint" "Capacitor_SMD:C_0504_1310Metric"
 			(at 181.3052 100.33 0)
 			(effects

Commit message: Replaced global labels with pin headers
Parts:
- added J42, J43, J44: Conn_01x02_Pin, symbol Connector:Conn_01x02_Pin
Connections:
- net +1V8: now also J43.1 (Pin_1)
- net +3V3: now also J42.1 (Pin_1)
- net GND: now also J42.2 (Pin_2), J43.2 (Pin_2)
- net SCL: now also J44.1 (Pin_1)
- net SDA: now also J44.2 (Pin_2)

Commit message: Reannotated schematic
Parts:
- renumbered C51 to C45, C52 to C46, C53 to C47, J42 to J56, J43 to J57, J44 to J58
Changed lines of the file:
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@@
 		(dnp no)
 		(fields_autoplaced yes)
-		(property "Reference" "J43"
+		(property "Reference" "J57"
 			(at 103.505 55.88 0)
 			(effects
@@
 			(project "raywatch"
 				(path "/7b654ee8-2a53-4d39-8b7d-32c7bb3cb0ed/9d8e2113-86ca-4807-a845-38f03d871655"
-					(reference "J43")
+					(reference "J57")
 					(unit 1)
 				)
@@
 		(dnp no)
 		(fields_autoplaced yes)
-		(property "Reference" "C51"
+		(property "Reference" "C45"
 			(at 114.3 97.7899 0)
 			(effects
@@
 			(project "raywatch"
 				(path "/7b654ee8-2a53-4d39-8b7d-32c7bb3cb0ed/9d8e2113-86ca-4807-a845-38f03d871655"
-					(reference "C51")
+					(reference "C45")
 					(unit 1)
 				)
@@
 		(dnp no)
 		(fields_autoplaced yes)
-		(property "Reference" "#PWR0311"
+		(property "Reference" "#PWR0324"
 			(at 168.91 88.9 0)
 			(effects
@@
 			(project "raywatch"
 				(path "/7b654ee8-2a53-4d39-8b7d-32c7bb3cb0ed/9d8e2113-86ca-4807-a845-38f03d871655"
-					(reference "#PWR0311")
+					(reference "#PWR0324")
 					(unit 1)
 				)
@@
 		(dnp no)
 		(fields_autoplaced yes)
-		(property "Reference" "#PWR0309"
+		(property "Reference" "#PWR0322"
 			(at 118.11 109.22 0)
 			(effects
@@
 			(project "raywatch"
 				(path "/7b654ee8-2a53-4d39-8b7d-32c7bb3cb0ed/9d8e2113-86ca-4807-a845-38f03d871655"
-					(reference "#PWR0309")
+					(reference "#PWR0322")
 					(unit 1)
 				)
@@
 		(dnp no)
 		(fields_autoplaced yes)
-		(property "Reference" "#PWR0313"
+		(property "Reference" "#PWR0326"
 			(at 180.34 88.9 0)
 			(effects
@@
 			(project "raywatch"
 				(path "/7b654ee8-2a53-4d39-8b7d-32c7bb3cb0ed/9d8e2113-86ca-4807-a845-38f03d871655"
-					(reference "#PWR0313")
+					(reference "#PWR0326")
 					(unit 1)
 				)
@@
 		(dnp no)
 		(fields_autoplaced yes)
-		(property "Reference" "#PWR0310"
+		(property "Reference" "#PWR0323"
 			(at 153.67 119.38 0)
 			(effects
@@
 			(project "raywatch"
 				(path "/7b654ee8-2a53-4d39-8b7d-32c7bb3cb0ed/9d8e2113-86ca-4807-a845-38f03d871655"
-					(reference "#PWR0310")
+					(reference "#PWR0323")
 					(unit 1)
 				)
@@
 		(dnp no)
 		(fields_autoplaced yes)
-		(property "Reference" "#PWR0312"
+		(property "Reference" "#PWR0325"
 			(at 168.91 106.68 0)
 			(effects
@@
 			(project "raywatch"
 				(path "/7b654ee8-2a53-4d39-8b7d-32c7bb3cb0ed/9d8e2113-86ca-4807-a845-38f03d871655"
-					(reference "#PWR0312")
+					(reference "#PWR0325")
 					(unit 1)
 				)
@@
 		(dnp no)
 		(fields_autoplaced yes)
-		(property "Reference" "J44"
+		(property "Reference" "J58"
 			(at 103.505 67.31 0)
 			(effects
@@
 			(project "raywatch"
 				(path "/7b654ee8-2a53-4d39-8b7d-32c7bb3cb0ed/9d8e2113-86ca-4807-a845-38f03d871655"
-					(reference "J44")
+					(reference "J58")
 					(unit 1)
 				)
@@
 		(dnp no)
 		(fields_autoplaced yes)
-		(property "Reference" "C52"
+		(property "Reference" "C46"
 			(at 172.72 95.2499 0)
 			(effects
@@
 			(project "raywatch"
 				(path "/7b654ee8-2a53-4d39-8b7d-32c7bb3cb0ed/9d8e2113-86ca-4807-a845-38f03d871655"
-					(reference "C52")
+					(reference "C46")
 					(unit 1)
 				)
@@
 		(dnp no)
 		(fields_autoplaced yes)
-		(property "Reference" "#PWR0314"
+		(property "Reference" "#PWR0327"
 			(at 180.34 106.68 0)
 			(effects
@@
 			(project "raywatch"
 				(path "/7b654ee8-2a53-4d39-8b7d-32c7bb3cb0ed/9d8e2113-86ca-4807-a845-38f03d871655"
-					(reference "#PWR0314")
+					(reference "#PWR0327")
 					(unit 1)
 				)
@@
 		(dnp no)
 		(fields_autoplaced yes)
-		(property "Reference" "#PWR0479"
+		(property "Reference" "#PWR0321"
 			(at 114.3 63.5 0)
 			(effects
@@
 			(project "raywatch"
 				(path "/7b654ee8-2a53-4d39-8b7d-32c7bb3cb0ed/9d8e2113-86ca-4807-a845-38f03d871655"
-					(reference "#PWR0479")
+					(reference "#PWR0321")
 					(unit 1)
 				)
@@
 		(dnp no)
 		(fields_autoplaced yes)
-		(property "Reference" "#PWR0477"
+		(property "Reference" "#PWR0320"
 			(at 104.14 60.96 0)
 			(effects
@@
 			(project "raywatch"
 				(path "/7b654ee8-2a53-4d39-8b7d-32c7bb3cb0ed/9d8e2113-86ca-4807-a845-38f03d871655"
-					(reference "#PWR0477")
+					(reference "#PWR0320")
 					(unit 1)
 				)
@@
 		(dnp no)
 		(fields_autoplaced yes)
-		(property "Reference" "#PWR0478"
+		(property "Reference" "#PWR0319"
 			(at 114.3 53.34 0)
 			(effects
@@
 			(project "raywatch"
 				(path "/7b654ee8-2a53-4d39-8b7d-32c7bb3cb0ed/9d8e2113-86ca-4807-a845-38f03d871655"
-					(reference "#PWR0478")
+					(reference "#PWR0319")
 					(unit 1)
 				)
@@
 		(dnp no)
 		(fields_autoplaced yes)
-		(property "Reference" "J42"
+		(property "Reference" "J56"
 			(at 103.505 45.72 0)
 			(effects
@@
 			(project "raywatch"
 				(path "/7b654ee8-2a53-4d39-8b7d-32c7bb3cb0ed/9d8e2113-86ca-4807-a845-38f03d871655"
-					(reference "J42")
+					(reference "J56")
 					(unit 1)
 				)
@@
 		(dnp no)
 		(fields_autoplaced yes)
-		(property "Reference" "C53"
+		(property "Reference" "C47"
 			(at 184.15 95.2499 0)
 			(effects
@@
 			(project "raywatch"
 				(path "/7b654ee8-2a53-4d39-8b7d-32c7bb3cb0ed/9d8e2113-86ca-4807-a845-38f03d871655"
-					(reference "C53")
+					(reference "C47")
 					(unit 1)
 				)
@@
 		(dnp no)
 		(fields_autoplaced yes)
-		(property "Reference" "#PWR0476"
+		(property "Reference" "#PWR0318"
 			(at 104.14 50.8 0)
 			(effects
@@
 			(project "raywatch"
 				(path "/7b654ee8-2a53-4d39-8b7d-32c7bb3cb0ed/9d8e2113-86ca-4807-a845-38f03d871655"
-					(reference "#PWR0476")
-					(unit 1)
-				)
+					(reference "#PWR0318")
+					(unit 1)
+				)

Commit message: Assigned pin header footprints
Parts:
- J56, J57, J58: footprint (none) -> Connector_PinHeader_2.54mm:PinHeader_1x02_P2.54mm_Horizontal
Changed lines of the file:
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@@
 			)
 		)
-		(property "Footprint" ""
+		(property "Footprint" "Connector_PinHeader_2.54mm:PinHeader_1x02_P2.54mm_Horizontal"
 			(at 102.87 60.96 0)
 			(effects
@@
 			)
 		)
-		(property "Footprint" ""
+		(property "Footprint" "Connector_PinHeader_2.54mm:PinHeader_1x02_P2.54mm_Horizontal"
 			(at 102.87 72.39 0)
 			(effects
@@
 			)
 		)
-		(property "Footprint" ""
+		(property "Footprint" "Connector_PinHeader_2.54mm:PinHeader_1x02_P2.54mm_Horizontal"
 			(at 102.87 50.8 0)
 			(effects

Commit message: Reannotate
Parts:
- renumbered U18 to U17
Changed lines of the file:
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@@
 		(dnp no)
 		(fields_autoplaced yes)
-		(property "Reference" "#PWR0324"
+		(property "Reference" "#PWR0325"
 			(at 168.91 88.9 0)
 			(effects
@@
 			(project "raywatch"
 				(path "/7b654ee8-2a53-4d39-8b7d-32c7bb3cb0ed/9d8e2113-86ca-4807-a845-38f03d871655"
-					(reference "#PWR0324")
+					(reference "#PWR0325")
 					(unit 1)
 				)
@@
 		(dnp no)
 		(fields_autoplaced yes)
-		(property "Reference" "#PWR0322"
+		(property "Reference" "#PWR0323"
 			(at 118.11 109.22 0)
 			(effects
@@
 			(project "raywatch"
 				(path "/7b654ee8-2a53-4d39-8b7d-32c7bb3cb0ed/9d8e2113-86ca-4807-a845-38f03d871655"
-					(reference "#PWR0322")
+					(reference "#PWR0323")
 					(unit 1)
 				)
@@
 		(dnp no)
 		(fields_autoplaced yes)
-		(property "Reference" "#PWR0326"
+		(property "Reference" "#PWR0327"
 			(at 180.34 88.9 0)
 			(effects
@@
 			(project "raywatch"
 				(path "/7b654ee8-2a53-4d39-8b7d-32c7bb3cb0ed/9d8e2113-86ca-4807-a845-38f03d871655"
-					(reference "#PWR0326")
+					(reference "#PWR0327")
 					(unit 1)
 				)
@@
 		(dnp no)
 		(fields_autoplaced yes)
-		(property "Reference" "#PWR0323"
+		(property "Reference" "#PWR0324"
 			(at 153.67 119.38 0)
 			(effects
@@
 			(project "raywatch"
 				(path "/7b654ee8-2a53-4d39-8b7d-32c7bb3cb0ed/9d8e2113-86ca-4807-a845-38f03d871655"
-					(reference "#PWR0323")
+					(reference "#PWR0324")
 					(unit 1)
 				)
@@
 		(dnp no)
 		(fields_autoplaced yes)
-		(property "Reference" "#PWR0325"
+		(property "Reference" "#PWR0326"
 			(at 168.91 106.68 0)
 			(effects
@@
 			(project "raywatch"
 				(path "/7b654ee8-2a53-4d39-8b7d-32c7bb3cb0ed/9d8e2113-86ca-4807-a845-38f03d871655"
-					(reference "#PWR0325")
+					(reference "#PWR0326")
 					(unit 1)
 				)
@@
 		(dnp no)
 		(fields_autoplaced yes)
-		(property "Reference" "#PWR0327"
+		(property "Reference" "#PWR0328"
 			(at 180.34 106.68 0)
 			(effects
@@
 			(project "raywatch"
 				(path "/7b654ee8-2a53-4d39-8b7d-32c7bb3cb0ed/9d8e2113-86ca-4807-a845-38f03d871655"
-					(reference "#PWR0327")
+					(reference "#PWR0328")
 					(unit 1)
 				)
@@
 		(dnp no)
 		(fields_autoplaced yes)
-		(property "Reference" "#PWR0321"
+		(property "Reference" "#PWR0322"
 			(at 114.3 63.5 0)
 			(effects
@@
 			(project "raywatch"
 				(path "/7b654ee8-2a53-4d39-8b7d-32c7bb3cb0ed/9d8e2113-86ca-4807-a845-38f03d871655"
-					(reference "#PWR0321")
+					(reference "#PWR0322")
 					(unit 1)
 				)
@@
 		(dnp no)
 		(fields_autoplaced yes)
-		(property "Reference" "#PWR0320"
+		(property "Reference" "#PWR0321"
 			(at 104.14 60.96 0)
 			(effects
@@
 			(project "raywatch"
 				(path "/7b654ee8-2a53-4d39-8b7d-32c7bb3cb0ed/9d8e2113-86ca-4807-a845-38f03d871655"
-					(reference "#PWR0320")
+					(reference "#PWR0321")
 					(unit 1)
 				)
@@
 		(dnp no)
 		(fields_autoplaced yes)
-		(property "Reference" "#PWR0319"
+		(property "Reference" "#PWR0320"
 			(at 114.3 53.34 0)
 			(effects
@@
 			(project "raywatch"
 				(path "/7b654ee8-2a53-4d39-8b7d-32c7bb3cb0ed/9d8e2113-86ca-4807-a845-38f03d871655"
-					(reference "#PWR0319")
+					(reference "#PWR0320")
 					(unit 1)
 				)
@@
 		(dnp no)
 		(fields_autoplaced yes)
-		(property "Reference" "U18"
+		(property "Reference" "U17"
 			(at 138.43 80.01 0)
 			(effects
@@
 			(project "raywatch"
 				(path "/7b654ee8-2a53-4d39-8b7d-32c7bb3cb0ed/9d8e2113-86ca-4807-a845-38f03d871655"
-					(reference "U18")
+					(reference "U17")
 					(unit 1)
 				)
@@
 		(dnp no)
 		(fields_autoplaced yes)
-		(property "Reference" "#PWR0318"
+		(property "Reference" "#PWR0319"
 			(at 104.14 50.8 0)
 			(effects
@@
 			(project "raywatch"
 				(path "/7b654ee8-2a53-4d39-8b7d-32c7bb3cb0ed/9d8e2113-86ca-4807-a845-38f03d871655"
-					(reference "#PWR0318")
-					(unit 1)
-				)
+					(reference "#PWR0319")
+					(unit 1)
+				)

Commit message: Changed pin headers to vertical
Parts:
- J56, J57, J58: footprint Connector_PinHeader_2.54mm:PinHeader_1x02_P2.54mm_Horizontal -> Connector_PinHeader_2.54mm:PinHeader_1x02_P2.54mm_Vertical
Changed lines of the file:
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@@
 			)
 		)
-		(property "Footprint" "Connector_PinHeader_2.54mm:PinHeader_1x02_P2.54mm_Horizontal"
+		(property "Footprint" "Connector_PinHeader_2.54mm:PinHeader_1x02_P2.54mm_Vertical"
 			(at 102.87 60.96 0)
 			(effects
@@
 			)
 		)
-		(property "Footprint" "Connector_PinHeader_2.54mm:PinHeader_1x02_P2.54mm_Horizontal"
+		(property "Footprint" "Connector_PinHeader_2.54mm:PinHeader_1x02_P2.54mm_Vertical"
 			(at 102.87 72.39 0)
 			(effects
@@
 			)
 		)
-		(property "Footprint" "Connector_PinHeader_2.54mm:PinHeader_1x02_P2.54mm_Horizontal"
+		(property "Footprint" "Connector_PinHeader_2.54mm:PinHeader_1x02_P2.54mm_Vertical"
 			(at 102.87 50.8 0)
 			(effects

Commit message: Fixed connector footprints; Changed conectors from 2.54 to 1.27
Parts:
- J54: renamed from J56; footprint Connector_PinHeader_2.54mm:PinHeader_1x02_P2.54mm_Vertical -> Connector_PinHeader_1.27mm:PinHeader_1x02_P1.27mm_Vertical
- J55: renamed from J57; footprint Connector_PinHeader_2.54mm:PinHeader_1x02_P2.54mm_Vertical -> Connector_PinHeader_1.27mm:PinHeader_1x02_P1.27mm_Vertical
- J56: renamed from J58; footprint Connector_PinHeader_2.54mm:PinHeader_1x02_P2.54mm_Vertical -> Connector_PinHeader_1.27mm:PinHeader_1x02_P1.27mm_Vertical
Changed lines of the file:
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@@
 		(dnp no)
 		(fields_autoplaced yes)
-		(property "Reference" "J57"
+		(property "Reference" "J55"
 			(at 103.505 55.88 0)
 			(effects
@@
 			)
 		)
-		(property "Footprint" "Connector_PinHeader_2.54mm:PinHeader_1x02_P2.54mm_Vertical"
+		(property "Footprint" "Connector_PinHeader_1.27mm:PinHeader_1x02_P1.27mm_Vertical"
 			(at 102.87 60.96 0)
 			(effects
@@
 			(project "raywatch"
 				(path "/7b654ee8-2a53-4d39-8b7d-32c7bb3cb0ed/9d8e2113-86ca-4807-a845-38f03d871655"
-					(reference "J57")
+					(reference "J55")
 					(unit 1)
 				)
@@
 		(dnp no)
 		(fields_autoplaced yes)
-		(property "Reference" "#PWR0325"
+		(property "Reference" "#PWR0327"
 			(at 168.91 88.9 0)
 			(effects
@@
 			(project "raywatch"
 				(path "/7b654ee8-2a53-4d39-8b7d-32c7bb3cb0ed/9d8e2113-86ca-4807-a845-38f03d871655"
-					(reference "#PWR0325")
+					(reference "#PWR0327")
 					(unit 1)
 				)
@@
 		(dnp no)
 		(fields_autoplaced yes)
-		(property "Reference" "#PWR0323"
+		(property "Reference" "#PWR0325"
 			(at 118.11 109.22 0)
 			(effects
@@
 			(project "raywatch"
 				(path "/7b654ee8-2a53-4d39-8b7d-32c7bb3cb0ed/9d8e2113-86ca-4807-a845-38f03d871655"
-					(reference "#PWR0323")
+					(reference "#PWR0325")
 					(unit 1)
 				)
@@
 		(dnp no)
 		(fields_autoplaced yes)
-		(property "Reference" "#PWR0327"
+		(property "Reference" "#PWR0329"
 			(at 180.34 88.9 0)
 			(effects
@@
 			(project "raywatch"
 				(path "/7b654ee8-2a53-4d39-8b7d-32c7bb3cb0ed/9d8e2113-86ca-4807-a845-38f03d871655"
-					(reference "#PWR0327")
+					(reference "#PWR0329")
 					(unit 1)
 				)
@@
 		(dnp no)
 		(fields_autoplaced yes)
-		(property "Reference" "#PWR0324"
+		(property "Reference" "#PWR0326"
 			(at 153.67 119.38 0)
 			(effects
@@
 			(project "raywatch"
 				(path "/7b654ee8-2a53-4d39-8b7d-32c7bb3cb0ed/9d8e2113-86ca-4807-a845-38f03d871655"
-					(reference "#PWR0324")
+					(reference "#PWR0326")
 					(unit 1)
 				)
@@
 		(dnp no)
 		(fields_autoplaced yes)
-		(property "Reference" "#PWR0326"
+		(property "Reference" "#PWR0328"
 			(at 168.91 106.68 0)
 			(effects
@@
 			(project "raywatch"
 				(path "/7b654ee8-2a53-4d39-8b7d-32c7bb3cb0ed/9d8e2113-86ca-4807-a845-38f03d871655"
-					(reference "#PWR0326")
+					(reference "#PWR0328")
 					(unit 1)
 				)
@@
 		(dnp no)
 		(fields_autoplaced yes)
-		(property "Reference" "J58"
+		(property "Reference" "J56"
 			(at 103.505 67.31 0)
 			(effects
@@
 			)
 		)
-		(property "Footprint" "Connector_PinHeader_2.54mm:PinHeader_1x02_P2.54mm_Vertical"
+		(property "Footprint" "Connector_PinHeader_1.27mm:PinHeader_1x02_P1.27mm_Vertical"
 			(at 102.87 72.39 0)
 			(effects
@@
 			(project "raywatch"
 				(path "/7b654ee8-2a53-4d39-8b7d-32c7bb3cb0ed/9d8e2113-86ca-4807-a845-38f03d871655"
-					(reference "J58")
+					(reference "J56")
 					(unit 1)
 				)
@@
 		(dnp no)
 		(fields_autoplaced yes)
-		(property "Reference" "#PWR0328"
+		(property "Reference" "#PWR0330"
 			(at 180.34 106.68 0)
 			(effects
@@
 			(project "raywatch"
 				(path "/7b654ee8-2a53-4d39-8b7d-32c7bb3cb0ed/9d8e2113-86ca-4807-a845-38f03d871655"
-					(reference "#PWR0328")
+					(reference "#PWR0330")
 					(unit 1)
 				)
@@
 		(dnp no)
 		(fields_autoplaced yes)
-		(property "Reference" "#PWR0322"
+		(property "Reference" "#PWR0324"
 			(at 114.3 63.5 0)
 			(effects
@@
 			(project "raywatch"
 				(path "/7b654ee8-2a53-4d39-8b7d-32c7bb3cb0ed/9d8e2113-86ca-4807-a845-38f03d871655"
-					(reference "#PWR0322")
+					(reference "#PWR0324")
 					(unit 1)
 				)
@@
 		(dnp no)
 		(fields_autoplaced yes)
-		(property "Reference" "#PWR0321"
+		(property "Reference" "#PWR0323"
 			(at 104.14 60.96 0)
 			(effects
@@
 			(project "raywatch"
 				(path "/7b654ee8-2a53-4d39-8b7d-32c7bb3cb0ed/9d8e2113-86ca-4807-a845-38f03d871655"
-					(reference "#PWR0321")
+					(reference "#PWR0323")
 					(unit 1)
 				)
@@
 		(dnp no)
 		(fields_autoplaced yes)
-		(property "Reference" "#PWR0320"
+		(property "Reference" "#PWR0322"
 			(at 114.3 53.34 0)
 			(effects
@@
 			(project "raywatch"
 				(path "/7b654ee8-2a53-4d39-8b7d-32c7bb3cb0ed/9d8e2113-86ca-4807-a845-38f03d871655"
-					(reference "#PWR0320")
+					(reference "#PWR0322")
 					(unit 1)
 				)
@@
 		(dnp no)
 		(fields_autoplaced yes)
-		(property "Reference" "J56"
+		(property "Reference" "J54"
 			(at 103.505 45.72 0)
 			(effects
@@
 			)
 		)
-		(property "Footprint" "Connector_PinHeader_2.54mm:PinHeader_1x02_P2.54mm_Vertical"
+		(property "Footprint" "Connector_PinHeader_1.27mm:PinHeader_1x02_P1.27mm_Vertical"
 			(at 102.87 50.8 0)
 			(effects
@@
 			(project "raywatch"
 				(path "/7b654ee8-2a53-4d39-8b7d-32c7bb3cb0ed/9d8e2113-86ca-4807-a845-38f03d871655"
-					(reference "J56")
+					(reference "J54")
 					(unit 1)
 				)
@@
 		(dnp no)
 		(fields_autoplaced yes)
-		(property "Reference" "#PWR0319"
+		(property "Reference" "#PWR0321"
 			(at 104.14 50.8 0)
 			(effects
@@
 			(project "raywatch"
 				(path "/7b654ee8-2a53-4d39-8b7d-32c7bb3cb0ed/9d8e2113-86ca-4807-a845-38f03d871655"
-					(reference "#PWR0319")
-					(unit 1)
-				)
+					(reference "#PWR0321")
+					(unit 1)
+				)

Commit message: Fixes; Added TPM PCB
Parts:
- C45, C46, C47: footprint Capacitor_SMD:C_0504_1310Metric -> Capacitor_SMD:C_0402_1005Metric
Changed lines of the file:
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@@
 			)
 		)
-		(property "Footprint" "Capacitor_SMD:C_0504_1310Metric"
+		(property "Footprint" "Capacitor_SMD:C_0402_1005Metric"
 			(at 119.0752 102.87 0)
 			(effects
@@
 			)
 		)
-		(property "Footprint" "Capacitor_SMD:C_0504_1310Metric"
+		(property "Footprint" "Capacitor_SMD:C_0402_1005Metric"
 			(at 169.8752 100.33 0)
 			(effects
@@
 			)
 		)
-		(property "Footprint" "Capacitor_SMD:C_0504_1310Metric"
+		(property "Footprint" "Capacitor_SMD:C_0402_1005Metric"
 			(at 181.3052 100.33 0)
 			(effects
